File: cpu16/kicad/cpu/cpu.kicad_sch (KiCad schematic)
At the start: 300 parts, among them J1 BACKPLANE_2x32, U1 SST39SF010A, U10 74HC138, U100 74HC153, U101 74HC688, U102 74HC688, U103 74HC541, U104 74HC541, U105 74HC157, U106 74HC74, U107 74HC74, U108 74HC74, U109 74HC541, U11 74HC74, U110 74HC541, U111 74HC151, U112 74HC245, U113 74HC245, U114 74HC245, U115 74HC541, U12 74HC74, U121 74HC08, U122 74HC08, U123 74HC08, U124 74HC08, U125 74HC08, U126 74HC08, U127 74HC08, U128 74HC08, U129 74HC08, U13 74HC138, U130 74HC08, U131 74HC08, U132 74HC32, U133 74HC32, U134 74HC32, U136 74HC00, U137 74HC00, U138 74HC00, U139 74HC02, U14 74HC151, U140 74HC02, U141 74HC02, U142 74HC86, U143 74HC86, U144 74HC86, U145 74HC86, U146 74HC86, U147 74HC86, U148 74HC86, U149 74HC86, U15 74HC151, U150 74HC86, U151 74HC04, U152 74HC04, U16 74HC151, U17 74HC138, U18 74HC138, U19 74HC574, U2 74HC574, U20 74HC574, U21 74HC574, U22 74HC574, U23 74HC574, U24 74HC574, U25 74HC574, U26 74HC574, U27 74HC574, U28 74HC574, U29 74HC574, U3 SST39SF010A, U30 74HC574, U31 74HC574, U32 74HC574, U33 74HC574, U34 74HC574, U35 74HC574, U36 74HC574, U37 74HC574, U38 74HC574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

Commit message: CPU16 Faz 9 (1): saat/reset kartı, Flash programlayıcı ve ROM imajları
- Saat ve reset kartı (9 entegre): kristal / yavaş RC osilatör seçimi, 8 durumlu Johnson sayacıyla
  parazitsiz CLK ve WR_WIN, açılış reseti, tek döngü ADIM butonu (eşzamanlı), saat sürücüsü.
  Kapı seviyesi bilgisayar artık yalnızca osilatörü sürer; bütün testler kartla birlikte geçer
- Flash programlayıcı: Arduino Nano yazılımı (Intel HEX, SST komut dizileri, DQ7 sorgulama,
  READ/SUM), yaz.py (pyserial), KiCad şeması ve BOM. Uçtan uca test: yazılımın kendisi derlenip
  kartın kapı seviyesi modeline (2 × 74HC595 + SST39SF010A) bağlanır
- cpu16/roms: mikrokod (4) ve ALU (3) Flash imajları, npm run cpu16 -- roms
- Board: çip başına footprint (ZIF soket), arka panelsiz kart, pasif referans çakışma denetimi

Co-Authored-By: Claude Opus 5.5 (1M context) <noreply@anthropic.com>
Claude-Session: https://claude.ai/code/session_018J8WVuECVRbQJyCbmF6Nsi
Parts:
- C120: renamed from C117; Gorev U121 dekuplaj -> U127 dekuplaj
- C121: renamed from C118; Gorev U122 dekuplaj -> U128 dekuplaj
- C122: renamed from C119; Gorev U123 dekuplaj -> U129 dekuplaj
- C123: renamed from C120; Gorev U124 dekuplaj -> U130 dekuplaj
- C124: renamed from C121; Gorev U125 dekuplaj -> U131 dekuplaj
- C125: renamed from C122; Gorev U126 dekuplaj -> U132 dekuplaj
- C126: renamed from C123; Gorev U127 dekuplaj -> U133 dekuplaj
- C127: renamed from C124; Gorev U128 dekuplaj -> U134 dekuplaj
- C128: renamed from C125; Gorev U129 dekuplaj -> U135 dekuplaj
- C129: renamed from C126; Gorev U130 dekuplaj -> U136 dekuplaj
- C130: renamed from C127; Gorev U131 dekuplaj -> U137 dekuplaj
- C131: renamed from C128; Gorev U132 dekuplaj -> U139 dekuplaj
- C132: renamed from C129; Gorev U133 dekuplaj -> U140 dekuplaj
- C133: renamed from C130; Gorev U134 dekuplaj -> U141 dekuplaj
- C134: renamed from C131; Gorev U136 dekuplaj -> U144 dekuplaj
- C135: renamed from C132; Gorev U137 dekuplaj -> U145 dekuplaj
- C136: renamed from C133; Gorev U138 dekuplaj -> U146 dekuplaj
- C137: renamed from C134; Gorev U139 dekuplaj -> U147 dekuplaj
- C138: renamed from C135; Gorev U140 dekuplaj -> U148 dekuplaj
- C139: renamed from C136; Gorev U141 dekuplaj -> U149 dekuplaj
- C140: renamed from C137; Gorev U142 dekuplaj -> U150 dekuplaj
- C141: renamed from C138; Gorev U143 dekuplaj -> U151 dekuplaj
- C142: renamed from C139; Gorev U144 dekuplaj -> U152 dekuplaj
- C143: renamed from C140; Gorev U145 dekuplaj -> U153 dekuplaj
- C144: renamed from C141; Gorev U146 dekuplaj -> U154 dekuplaj
- C145: renamed from C142; Gorev U147 dekuplaj -> U155 dekuplaj
- C146: renamed from C143; Gorev U148 dekuplaj -> U156 dekuplaj
- C147: renamed from C144; Gorev U149 dekuplaj -> U157 dekuplaj
- C148: renamed from C145; Gorev U150 dekuplaj -> U158 dekuplaj
- C149: renamed from C146; Gorev U151 dekuplaj -> U159 dekuplaj
- C150: renamed from C147; Gorev U152 dekuplaj -> U160 dekuplaj
- renumbered C7 to C10, C97 to C100, C98 to C101, C99 to C102, C100 to C103, C101 to C104, C102 to C105, C103 to C106, C104 to C107, C105 to C108, C106 to C109, C8 to C11, C107 to C110, C108 to C111, C109 to C112, C110 to C113, C111 to C114, C112 to C115, C113 to C116, C114 to C117, C115 to C118, C116 to C119, C9 to C12, C10 to C13, C11 to C14, C12 to C15, C13 to C16, C14 to C17, C15 to C18, C16 to C19, C17 to C20, C18 to C21, C19 to C22, C20 to C23, C21 to C24, C22 to C25, C23 to C26, C24 to C27, C25 to C28, C26 to C29, C27 to C30, C28 to C31, C29 to C32, C30 to C33, C31 to C34, C32 to C35, C33 to C36, C34 to C37, C35 to C38, C36 to C39, C1 to C4, C37 to C40, C38 to C41, C39 to C42, C40 to C43, C41 to C44, C42 to C45, C43 to C46, C44 to C47, C45 to C48, C46 to C49, C2 to C5, C47 to C50, C48 to C51, C49 to C52, C50 to C53, C51 to C54, C52 to C55, C53 to C56, C54 to C57, C55 to C58, C56 to C59, C3 to C6, C57 to C60, C58 to C61, C59 to C62, C60 to C63, C61 to C64, C62 to C65, C63 to C66, C64 to C67, C65 to C68, C66 to C69, C4 to C7, C67 to C70, C68 to C71, C69 to C72, C70 to C73, C71 to C74, C72 to C75, C73 to C76, C74 to C77, C75 to C78, C76 to C79, C5 to C8, C77 to C80, C78 to C81, C79 to C82, C80 to C83, C81 to C84, C82 to C85, C83 to C86, C84 to C87, C85 to C88, C86 to C89, C6 to C9, C87 to C90, C88 to C91, C89 to C92, C90 to C93, C91 to C94, C92 to C95, C93 to C96, C94 to C97, C95 to C98, C96 to C99, U121 to U127, U122 to U128, U123 to U129, U124 to U130, U125 to U131, U126 to U132, U127 to U133, U128 to U134, U129 to U135, U130 to U136, U131 to U137, U132 to U139, U133 to U140, U134 to U141, U136 to U144, U137 to U145, U138 to U146, U139 to U147, U140 to U148, U141 to U149, U142 to U150, U143 to U151, U144 to U152, U145 to U153, U146 to U154, U147 to U155, U148 to U156, U149 to U157, U150 to U158, U151 to U159, U152 to U160

Commit message: Kart başına kararlı referans numaraları; yapıştırıcı kapı ve pasiflerde blok bilgisi
Her kart kendi KiCad projesi olduğu için numaralar kart içinde verilir (cpu U1.., clk U201..,
mem U301..). Deney rehberi bir bloğun hangi kapı birimlerini kullandığını bilsin diye yapıştırıcı
lojik çiplerine birim → blok eşlemesi eklendi.

Co-Authored-By: Claude Opus 5.5 (1M context) <noreply@anthropic.com>
Claude-Session: https://claude.ai/code/session_018J8WVuECVRbQJyCbmF6Nsi
Parts:
- C117: renamed from C120; Gorev U127 dekuplaj -> U116 dekuplaj
- C118: renamed from C121; Gorev U128 dekuplaj -> U117 dekuplaj
- C119: renamed from C122; Gorev U129 dekuplaj -> U118 dekuplaj
- C120: renamed from C123; Gorev U130 dekuplaj -> U119 dekuplaj
- C121: renamed from C124; Gorev U131 dekuplaj -> U120 dekuplaj
- C122: renamed from C125; Gorev U132 dekuplaj -> U121 dekuplaj
- C123: renamed from C126; Gorev U133 dekuplaj -> U122 dekuplaj
- C124: renamed from C127; Gorev U134 dekuplaj -> U123 dekuplaj
- C125: renamed from C128; Gorev U135 dekuplaj -> U124 dekuplaj
- C126: renamed from C129; Gorev U136 dekuplaj -> U125 dekuplaj
- C127: renamed from C130; Gorev U137 dekuplaj -> U126 dekuplaj
- C128: renamed from C131; Gorev U139 dekuplaj -> U127 dekuplaj
- C129: renamed from C132; Gorev U140 dekuplaj -> U128 dekuplaj
- C130: renamed from C133; Gorev U141 dekuplaj -> U129 dekuplaj
- C131: renamed from C134; Gorev U144 dekuplaj -> U130 dekuplaj
- C132: renamed from C135; Gorev U145 dekuplaj -> U131 dekuplaj
- C133: renamed from C136; Gorev U146 dekuplaj -> U132 dekuplaj
- C134: renamed from C137; Gorev U147 dekuplaj -> U133 dekuplaj
- C135: renamed from C138; Gorev U148 dekuplaj -> U134 dekuplaj
- C136: renamed from C139; Gorev U149 dekuplaj -> U135 dekuplaj
- C137: renamed from C140; Gorev U150 dekuplaj -> U136 dekuplaj
- C138: renamed from C141; Gorev U151 dekuplaj -> U137 dekuplaj
- C139: renamed from C142; Gorev U152 dekuplaj -> U138 dekuplaj
- C140: renamed from C143; Gorev U153 dekuplaj -> U139 dekuplaj
- C141: renamed from C144; Gorev U154 dekuplaj -> U140 dekuplaj
- C142: renamed from C145; Gorev U155 dekuplaj -> U141 dekuplaj
- C143: renamed from C146; Gorev U156 dekuplaj -> U142 dekuplaj
- C144: renamed from C147; Gorev U157 dekuplaj -> U143 dekuplaj
- C145: renamed from C148; Gorev U158 dekuplaj -> U144 dekuplaj
- C146: renamed from C149; Gorev U159 dekuplaj -> U145 dekuplaj
- C147: renamed from C150; Gorev U160 dekuplaj -> U146 dekuplaj
- renumbered C4 to C1, C13 to C10, C103 to C100, C104 to C101, C105 to C102, C106 to C103, C107 to C104, C108 to C105, C109 to C106, C110 to C107, C111 to C108, C112 to C109, C14 to C11, C113 to C110, C114 to C111, C115 to C112, C116 to C113, C117 to C114, C118 to C115, C119 to C116, C15 to C12, C16 to C13, C17 to C14, C18 to C15, C19 to C16, C20 to C17, C21 to C18, C22 to C19, C5 to C2, C23 to C20, C24 to C21, C25 to C22, C26 to C23, C27 to C24, C28 to C25, C29 to C26, C30 to C27, C31 to C28, C32 to C29, C6 to C3, C33 to C30, C34 to C31, C35 to C32, C36 to C33, C37 to C34, C38 to C35, C39 to C36, C40 to C37, C41 to C38, C42 to C39, C7 to C4, C43 to C40, C44 to C41, C45 to C42, C46 to C43, C47 to C44, C48 to C45, C49 to C46, C50 to C47, C51 to C48, C52 to C49, C8 to C5, C53 to C50, C54 to C51, C55 to C52, C56 to C53, C57 to C54, C58 to C55, C59 to C56, C60 to C57, C61 to C58, C62 to C59, C9 to C6, C63 to C60, C64 to C61, C65 to C62, C66 to C63, C67 to C64, C68 to C65, C69 to C66, C70 to C67, C71 to C68, C72 to C69, C10 to C7, C73 to C70, C74 to C71, C75 to C72, C76 to C73, C77 to C74, C78 to C75, C79 to C76, C80 to C77, C81 to C78, C82 to C79, C11 to C8, C83 to C80, C84 to C81, C85 to C82, C86 to C83, C87 to C84, C88 to C85, C89 to C86, C90 to C87, C91 to C88, C92 to C89, C12 to C9, C93 to C90, C94 to C91, C95 to C92, C96 to C93, C97 to C94, C98 to C95, C99 to C96, C100 to C97, C101 to C98, C102 to C99, U127 to U116, U128 to U117, U129 to U118, U130 to U119, U131 to U120, U132 to U121, U133 to U122, U134 to U123, U135 to U124, U136 to U125, U137 to U126, U139 to U127, U140 to U128, U141 to U129, U144 to U130, U145 to U131, U146 to U132, U147 to U133, U148 to U134, U149 to U135, U150 to U136, U151 to U137, U152 to U138, U153 to U139, U154 to U140, U155 to U141, U156 to U142, U157 to U143, U158 to U144, U159 to U145, U160 to U146

Commit message: Faz 9: şemadan statik zamanlama analizi; C/V bayrak saati düzeltmesi
- board/zamanlama.ts: saat ağacı, flip-flop'tan flip-flop'a en uzun yollar, yarım/tam periyot,
  kapılı saat kurulum ve tutma kontrolleri; 74HC veri sayfası gecikmeleri (tip / maks) ve yük
  düzeltmesi. npm run cpu16 -- zamanlama [--tip]
- Sonuç: en kötü durumda CPU 1,16 MHz, tipik 2,1 MHz; kritik yol kontrol register'ı → ALU ROM'u
  → 4 × 74HC283 → veriyolu (yarım periyot)
- Analizin bulduğu risk: C/V bayraklarının saat izni ALU ROM'unun SETSCV çıkışından geliyordu;
  ROM adresindeki CFLAG tam o kenarda değiştiği için ROM çıkışındaki bir sıçrama ikinci saat
  darbesi üretebilirdi. Artık dört bayrak aynı saatle yüklenir, SETSCV = 0 iken bir 74HC157
  eski C ve V'yi geri yazar (kapı seviyesi lockstep testleri geçiyor)
- Mikrokod testi: IR yüklenen adımda IR alanlarından seçilen register'a yazılmaz
- Deney rehberleri: otomatik bölümler yeniden üretildi; rehberlerin güncel olduğunu ve elle yazılan
  referansların şemada bulunduğunu denetleyen testler
- KiCad şemaları ve BOM yeniden üretildi

Co-Authored-By: Claude Opus 5.5 (1M context) <noreply@anthropic.com>
Claude-Session: https://claude.ai/code/session_018J8WVuECVRbQJyCbmF6Nsi
Parts:
- removed U116: 74HC08, Package_DIP:DIP-14_W7.62mm, symbol cpu16:74HC08
- added U116: 74HC157, Package_DIP:DIP-16_W7.62mm, symbol cpu16:74HC157
- U117: Gorev yapıştırıcı: HALT durumu, yasadışı komut, çalışma izni, TA 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 -> yapıştırıcı: IRQ ∧ I, INT seçimi, HALT durumu
- U118: Gorev yapıştırıcı: TB saati, MAR saati, IR saati, PC += 2 -> yapıştırıcı: HALT durumu, yasadışı komut, çalışma izni, TA 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
- U119: Gorev yapıştırıcı: toplayıcı B girişi -> yapıştırıcı: TB saati, MAR saati, IR saati, PC += 2
- U123: Gorev yapıştırıcı: taşma (V), SAR işaret biti, NZ saati, C V yükle -> yapıştırıcı: toplayıcı B girişi
- U124: Gorev yapıştırıcı: CV saati, I saati, I girişi, HI koşulu -> yapıştırıcı: taşma (V), SAR işaret biti, NZ saati, I saati
- U125: Gorev yapıştırıcı: GT koşulu, bellek yazma, tek adresli bayt, yaz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 -> yapıştırıcı: I girişi, HI koşulu, GT koşulu, bellek yazma
- U126: Gorev yapıştırıcı: yazma darbesi -> yapıştırıcı: tek adresli bayt, yazma darbesi
- U128: Gorev yapıştırıcı: sağa kaydırmada giren bit, N Z yükle, C V yükl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 -> yapıştırıcı: sağa kaydırmada giren bit, N Z yükle, I yükle
- U129: Gorev yapıştırıcı: I yükle, I girişi, bellek erişimi, yazma darbe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 -> yapıştırıcı: I girişi, bellek erişimi, yazma darbesi
Connections:
- net A0: now also U126.2 (1B), U129.10 (3B); no longer U125.10 (3B), U129.13 (4B)
- net AD1: now also U123.10 (3B), U123.13 (4B), U123.2 (1B), U123.5 (2B); no longer U119.10 (3B), U119.13 (4B), U119.2 (1B), U119.5 (2B)
- net AD4: now also U116.1 (S); no longer U123.13 (4B)
- net AD7: now also U124.4 (2A); no longer U123.4 (2A)
- net BUS4: now also U125.2 (1B); no longer U124.10 (3B)
- net CFLAG: now also U125.4 (2A), U116.2 (1I0); no longer U124.12 (4A)
- net CLKR: now also U118.12 (4A), U119.1 (1A), U119.4 (2A), U119.9 (3A), U124.12 (4A), U124.9 (3A); no longer U117.12 (4A), U118.1 (1A), U118.4 (2A), U118.9 (3A), U123.9 (3A), U124.1 (1A), U124.4 (2A)
- net CLK_I: now also U124.11 (4Y); no longer U124.6 (2Y)
- net CLK_IR: now also U119.8 (3Y); no longer U118.8 (3Y)
- net CLK_MAR: now also U119.6 (2Y); no longer U118.6 (2Y)
- net CLK_NZ: now also U107.11 (2CLK), U107.3 (1CLK), U124.8 (3Y); no longer U123.8 (3Y)
- net CLK_TA: now also U118.11 (4Y); no longer U117.11 (4Y)
- net CLK_TB: now also U119.3 (1Y); no longer U118.3 (1Y)
- net CW17: now also U118.13 (4B); no longer U117.13 (4B)
- net CW18: now also U119.2 (1B); no longer U118.2 (1B)
- net CW20: now also U119.12 (4A); no longer U118.12 (4A)
- net CW21: now also U119.5 (2B); no longer U118.5 (2B)
- net CW22: now also U125.12 (4A); no longer U125.4 (2A)
- net CW23: now also U119.10 (3B); no longer U118.10 (3B)
- net CW24: no longer U123.12 (4A)
- net CW25: now also U125.1 (1A), U128.13 (4B); no longer U124.9 (3A), U128.10 (3B), U129.2 (1B)
- net CW26: now also U128.9 (3A), U129.1 (1A); no longer U128.12 (4A), U129.4 (2A)
- net CW27: now also U128.10 (3B); no longer U128.13 (4B)
- net CW28: now also U126.1 (1A); no longer U125.9 (3A)
- net CW29: now also U118.1 (1A); no longer U117.1 (1A)
- net CW30: now also U118.4 (2A); no longer U117.4 (2A)
- net C_ALU: now also U116.3 (1I1); no longer U105.11 (3I0)
- net DI: now also U129.3 (1Y); no longer U129.6 (2Y)
- net GND: now also U129.12 (4A), U129.13 (4B), U116.10 (3I1), U116.11 (3I0), U116.13 (4I1), U116.14 (4I0), U116.15 (~{E}), U116.8 (GND); no longer U126.10 (3B), U126.4 (2A), U126.5 (2B), U126.9 (3A)
- net HALTED: now also U117.12 (4A)
- net IFLAG: now also U117.2 (1B)
- net INT_HOLD: now also U117.10 (3B)
- net IRQ: now also U117.1 (1A)
- net IS_STEP0: now also U117.4 (2A)
- net I_LD: now also U124.13 (4B), U128.11 (4Y); no longer U124.5 (2B), U129.3 (1Y)
- net LANE_E: now also U126.5 (2B); no longer U125.13 (4B)
- net LANE_OB: now also U126.3 (1Y); no longer U125.8 (3Y)
- net MEMRD: now also U129.4 (2A); no longer U129.9 (3A)
- net MEMW: now also U125.11 (4Y), U126.4 (2A), U126.9 (3A), U129.5 (2B); no longer U125.12 (4A), U125.6 (2Y), U126.1 (1A), U129.10 (3B)
- net MEM_ACC: now also U129.6 (2Y); no longer U129.8 (3Y)
- net N1211: now also U120.3 (1Y); no longer U119.3 (1Y)
- net N1213: now also U120.6 (2Y); no longer U119.6 (2Y)
- net N1215: now also U120.8 (3Y); no longer U119.8 (3Y)
- net N1217: now also U120.11 (4Y); no longer U119.11 (4Y)
- net N1219: now also U121.3 (1Y); no longer U120.3 (1Y)
- net N1221: now also U121.6 (2Y); no longer U120.6 (2Y)
- net N1223: now also U121.8 (3Y); no longer U120.8 (3Y)
- net N1225: now also U121.11 (4Y); no longer U120.11 (4Y)
- net N1227: now also U122.3 (1Y); no longer U121.3 (1Y)
- net N1229: now also U122.6 (2Y); no longer U121.6 (2Y)
- net N1231: now also U122.8 (3Y); no longer U121.8 (3Y)
- net N1233: now also U122.11 (4Y); no longer U121.11 (4Y)
- net N1235: now also U123.3 (1Y); no longer U122.3 (1Y)
- net N1237: now also U123.6 (2Y); no longer U122.6 (2Y)
- net N1239: now also U123.8 (3Y); no longer U122.8 (3Y)
- net N1241: now also U123.11 (4Y); no longer U122.11 (4Y)
- net N1363: now also U124.1 (1A); no longer U123.1 (1A)
- net N1364: now also U124.2 (1B); no longer U123.2 (1B)
- net N1590: now also U124.6 (2Y); no longer U123.6 (2Y)
- net N1779: now also U111.13 (I6), U125.8 (3Y); no longer U111.15 (I4), U124.11 (4Y)
- net N271: now also U117.6 (2Y)
- net N272: now also U117.8 (3Y)
- net N275: now also U117.11 (4Y)
- net N277: now also U118.3 (1Y); no longer U117.3 (1Y)
- net N281: now also U118.6 (2Y); no longer U117.6 (2Y)
- net N284: now also U118.10 (3B); no longer U117.10 (3B)
- net NZ_LD: now also U124.10 (3B); no longer U123.10 (3B)
- net N_EQ_V: now also U125.10 (3B); no longer U125.2 (1B)
- net PC_INC_EN: now also U119.11 (4Y); no longer U118.11 (4Y)
- net RUN: now also U118.8 (3Y); no longer U117.8 (3Y)
- net RUN_R: now also U118.2 (1B), U118.5 (2B), U119.13 (4B), U125.13 (4B); no longer U117.2 (1B), U117.5 (2B), U118.13 (4B), U125.5 (2B)
- net TA15: now also U124.5 (2B); no longer U123.5 (2B)
- net TB0: now also U120.1 (1A); no longer U119.1 (1A)
- net TB1: now also U120.4 (2A); no longer U119.4 (2A)
- net TB10: now also U122.9 (3A); no longer U121.9 (3A)
- net TB11: now also U122.12 (4A); no longer U121.12 (4A)
- net TB12: now also U123.1 (1A); no longer U122.1 (1A)
- net TB13: now also U123.4 (2A); no longer U122.4 (2A)
- net TB14: now also U123.9 (3A); no longer U122.9 (3A)
- net TB15: now also U123.12 (4A); no longer U122.12 (4A)
- net TB2: now also U120.9 (3A); no longer U119.9 (3A)
- net TB3: now also U120.12 (4A); no longer U119.12 (4A)
- net TB4: now also U121.1 (1A); no longer U120.1 (1A)
- net TB5: now also U121.4 (2A); no longer U120.4 (2A)
- net TB6: now also U121.9 (3A); no longer U120.9 (3A)
- net TB7: now also U121.12 (4A); no longer U120.12 (4A)
- net TB8: now also U122.1 (1A); no longer U121.1 (1A)
- net TB9: now also U122.4 (2A); no longer U121.4 (2A)
- net VCC: now also U116.16 (VCC)
- net VFLAG: now also U116.5 (2I0)
- net V_ADD: now also U124.3 (1Y); no longer U123.3 (1Y)
- net V_ALU: now also U116.6 (2I1); no longer U105.14 (4I0)
- net WAKE: now also U117.3 (1Y), U117.5 (2B)
- net WE_E_EN: now also U126.6 (2Y); no longer U125.11 (4Y)
- net WE_O_EN: now also U126.8 (3Y); no longer U126.3 (1Y)
- net ~{BYTE}: now also U129.9 (3A); no longer U129.12 (4A)
- net ~{FAULT}: now also U118.9 (3A); no longer U117.9 (3A)
- net ~{IS_STEP0}: now also U117.9 (3A)
- net ~{WAKE}: now also U117.13 (4B)
- net ~{ZFLAG}: now also U125.5 (2B), U125.9 (3A); no longer U124.13 (4B), U125.1 (1A)
- removed net CLK_CV: U107.11 (2CLK), U107.3 (1CLK), U124.3 (1Y)
- net CV_LD renamed N1766
- net N1766: now also U128.12 (4A); no longer U124.2 (1B)
- removed net N1757: U123.11 (4Y), U128.9 (3A)
- removed net N1767: U128.11 (4Y), U129.1 (1A)
- removed net N1770: U124.8 (3Y), U129.5 (2B)
- net N1777 renamed N1776
- net N1780 renamed N1769
- net N1769: now also U129.2 (1B); no longer U111.13 (I6)
- net N1801 renamed N1800
- net N1814 renamed N1813
- net N1827 renamed N1826
- net N1832 renamed N1831
- net N1835: no longer names the net of U129.11 (4Y)
- net N1835: no longer U126.2 (1B)
- new net C_NEW: U105.11 (3I0), U116.4 (1Y)
- new net N1778: U111.15 (I4), U125.6 (2Y)
- new net N1834: U126.10 (3B), U129.8 (3Y)
- new net V_NEW: U105.14 (4I0), U116.7 (2Y)
- no-connect marks 104 -> 105
