File: cpu16/kicad/cpu/cpu.kicad_sch (KiCad schematic)
At the start: 300 parts, among them J1 BACKPLANE_2x32, U1 SST39SF010A, U10 74HC138, U100 74HC153, U101 74HC688, U102 74HC688, U103 74HC541, U104 74HC541, U105 74HC157, U106 74HC74, U107 74HC74, U108 74HC74, U109 74HC541, U11 74HC74, U110 74HC541, U111 74HC151, U112 74HC245, U113 74HC245, U114 74HC245, U115 74HC541, U12 74HC74, U127 74HC08, U128 74HC08, U129 74HC08, U13 74HC138, U130 74HC08, U131 74HC08, U132 74HC08, U133 74HC08, U134 74HC08, U135 74HC08, U136 74HC08, U137 74HC08, U139 74HC32, U14 74HC151, U140 74HC32, U141 74HC32, U144 74HC00, U145 74HC00, U146 74HC00, U147 74HC02, U148 74HC02, U149 74HC02, U15 74HC151, U150 74HC86, U151 74HC86, U152 74HC86, U153 74HC86, U154 74HC86, U155 74HC86, U156 74HC86, U157 74HC86, U158 74HC86, U159 74HC04, U16 74HC151, U160 74HC04, U17 74HC138, U18 74HC138, U19 74HC574, U2 74HC574, U20 74HC574, U21 74HC574, U22 74HC574, U23 74HC574, U24 74HC574, U25 74HC574, U26 74HC574, U27 74HC574, U28 74HC574, U29 74HC574, U3 SST39SF010A, U30 74HC574, U31 74HC574, U32 74HC574, U33 74HC574, U34 74HC574, U35 74HC574, U36 74HC574, U37 74HC574, U38 74HC574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

Commit message: Anakart: bekleme durumlu saat kartı, bellek ve önbellek kartları (kapı seviyesi)
Saat kartı: ~WAIT (10 kΩ ile 1'e çekili) s7'nin ortasında W flip-flop'una örneklenir;
W = 1 iken CLK ve WR_WIN kapalı kalır, her bekleme tam bir CPU saati (8 OSC) sürer.
TCLK (uzatılmayan OSC/8, Johnson Q1) ve tamponlu OSC arka panele çıkar. ADIM kipinde
bir basış bekleme turları dahil tam bir döngü. 9 → 10 entegre.

Bellek kartı (bellek, 31 entegre): ~IO çözümü, 4 × 74HC273 bank register'ı (reset
0/32/33/34, geri okuma), PA14..PA19, Flash SST39SF010A + RAM AS6C4008 8 bit, TCLK ile
yürüyen bayt sıralayıcı, boş bölge 0xFF, DE/DO çekme dirençleri.

Önbellek kartı (onbellek, 37 entegre): 2 KB doğrudan eşlemeli, 1024 kelimelik satır,
etiket [19:11] + geçerli, 74HC688 karşılaştırma, write-through, yazma gözetleme (RAM:
güncelle, Flash: geçersiz kıl), reset'te sayıcıyla etiket temizleme, CACHE_CTRL, 4 ×
74HC590 isabet/ıskalama sayacı; ana belleğe giden her erişime tam MEM_WAIT = 2 bekleme.

machine-board.ts: buildMachineBoard({ cards }) ve GateMachine (CPU + saat + bellek +
önbellek; ek kartlar için kanca). bus-master.ts: CPU kartı yerine arka paneli süren
düzenek (Machine'in veri yolu izini kartlarda yeniden oynatmak için).

KiCad: bellek (A2) ve onbellek (A1) projeleri, kart klasöründe BOM; arka panel netleri
BACKPLANE'den. npm run cpu16 -- board artık anakartın özetini ve ERC'sini de yazar.

Testler: anakart-bellek.test.ts (BIOS açılışı, monitör komutları, F ile Flash yükleme,
64 bank/gözetleme/sayaç senaryosu, 1 MB harita — her erişimde değer, bekleme, bank,
sayaç), anakart-sistem.test.ts (saat kartı bekleme turları ve ADIM kipi; CPU dahil
tam sistem Machine ile komut komut: RAM'den programlar, sınama programı, BIOS açılışı).

Co-Authored-By: Claude Opus 5.5 (1M context) <noreply@anthropic.com>
Claude-Session: https://claude.ai/code/session_018J8WVuECVRbQJyCbmF6Nsi
Parts:
- C131: Gorev U139 dekuplaj -> U140 dekuplaj
- C132: Gorev U140 dekuplaj -> U141 dekuplaj
- C133: Gorev U141 dekuplaj -> U142 dekuplaj
- C134: Gorev U144 dekuplaj -> U145 dekuplaj
- C135: Gorev U145 dekuplaj -> U146 dekuplaj
- C136: Gorev U146 dekuplaj -> U147 dekuplaj
- C137: Gorev U147 dekuplaj -> U148 dekuplaj
- C138: Gorev U148 dekuplaj -> U149 dekuplaj
- C139: Gorev U149 dekuplaj -> U150 dekuplaj
- C140: Gorev U150 dekuplaj -> U151 dekuplaj
- C141: Gorev U151 dekuplaj -> U152 dekuplaj
- C142: Gorev U152 dekuplaj -> U153 dekuplaj
- C143: Gorev U153 dekuplaj -> U154 dekuplaj
- C144: Gorev U154 dekuplaj -> U155 dekuplaj
- C145: Gorev U155 dekuplaj -> U156 dekuplaj
- C146: Gorev U156 dekuplaj -> U157 dekuplaj
- C147: Gorev U157 dekuplaj -> U158 dekuplaj
- C148: Gorev U158 dekuplaj -> U159 dekuplaj
- C149: Gorev U159 dekuplaj -> U160 dekuplaj
- C150: Gorev U160 dekuplaj -> U161 dekuplaj
- renumbered U139 to U140, U140 to U141, U141 to U142, U144 to U145, U145 to U146, U146 to U147, U147 to U148, U148 to U149, U149 to U150, U150 to U151, U151 to U152, U152 to U153, U153 to U154, U154 to U155, U155 to U156, U156 to U157, U157 to U158, U158 to U159, U159 to U160, U160 to U161
Connections:
- net ~{WAIT}: now reaches J1.46
- net TCLK: now reaches J1.48
- net OSC: now reaches J1.49
- no-connect marks 104 -> 101
