File: cpu16/kicad/cpu/cpu.kicad_sch (KiCad schematic)
At the start: 300 parts, among them J1 BACKPLANE_2x32, U1 SST39SF010A, U10 74HC138, U100 74HC153, U101 74HC688, U102 74HC688, U103 74HC541, U104 74HC541, U105 74HC157, U106 74HC74, U107 74HC74, U108 74HC74, U109 74HC541, U11 74HC74, U110 74HC541, U111 74HC151, U112 74HC245, U113 74HC245, U114 74HC245, U115 74HC541, U116 74HC157, U117 74HC08, U118 74HC08, U119 74HC08, U12 74HC74, U120 74HC08, U121 74HC08, U122 74HC08, U123 74HC08, U124 74HC08, U125 74HC08, U126 74HC08, U127 74HC32, U128 74HC32, U129 74HC32, U13 74HC138, U130 74HC00, U131 74HC00, U132 74HC00, U133 74HC02, U134 74HC02, U135 74HC02, U136 74HC86, U137 74HC86, U138 74HC86, U139 74HC86, U14 74HC151, U140 74HC86, U141 74HC86, U142 74HC86, U143 74HC86, U144 74HC86, U145 74HC04, U146 74HC04, U15 74HC151, U16 74HC151, U17 74HC138, U18 74HC138, U19 74HC574, U2 74HC574, U20 74HC574, U21 74HC574, U22 74HC574, U23 74HC574, U24 74HC574, U25 74HC574, U26 74HC574, U27 74HC574, U28 74HC574, U29 74HC574, U3 SST39SF010A, U30 74HC574, U31 74HC574, U32 74HC574, U33 74HC574, U34 74HC574, U35 74HC574, U36 74HC574, U37 74HC574, U38 74HC574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

Commit message: Kontrol birimi: mikrokod ve ALU ROM'ları yerine 74HC kapı devresi
CPU kartındaki 7 SST39SF010A (4 mikrokod, 3 ALU kod çözme ROM'u) kalktı. Yerine
board/kontrol.ts, cpu16.ucode'dan (tek kaynak) ve aluControl tablosundan çok seviyeli
bir 74HC devresi üretir ve Board API ile gerçek çipler olarak yerleştirir:

- Mikrokod: adım ve komut çözücüleri (74HC138; INT = 1 iken komutlar pasif, f3'e göre
  dallanan komutlara alt çözücü), aynı mikro programı çalıştıran (op, f3, COND)
  atomları, ortak alt kümeli VEYA ağı, sık kullanılan bitler için adım seçici
  (74HC151), adım 8..15 için SWI hattıyla açılan çözücü.
- ALU kod çözme: işlem çözücüleri (3 × 74HC138), işlem bitleri, h ve C terimleri.
- Yeni kapı çipleri: 74HC11, 74HC20, 74HC21, 74HC27, 74HC30 (veri sayfası pin sırası,
  doğruluk tablosu, zamanlama modeli, KiCad sembolü).
- Board: esnek yapıştırıcı kapılar (kartın diğer kapılarından sonra paketlenir, son
  çipi az dolu türü başka türlerin boş birimlerine taşır) ve defer(). Çözücüler eski
  ROM'ların yuvalarına (U1, U3, U5, U7, U10, U68–U71) oturur: kartın diğer bütün
  çiplerinin referansları değişmedi.
- CPU kartı 146 → 194 entegre; en kötü durumda CPU saati 860 → 824 ns (1,21 MHz),
  tipik 470 → 369 ns.
- Denklik testi (tests/kontrol.test.ts): kontrol birimi tek başına bir kartta, gerçek
  çip modelleriyle (LogicSim) 8192 mikrokod adresinin ve 128 ALU adresinin hepsinde
  tabloyla aynı kelimeyi verir.
- roms.ts, cpu16/roms/ ve "roms" komutu kalktı; "kontrol" komutu gömülü mikrokodu
  (micro/cpu16-ucode.ts) yeniler ve devreyi denetler. GateComputer ve GateMachine artık
  mikrokod istemez.
- CPU şeması A0'a sığsın diye dekuplaj kondansatörleri dar sütunlarda; KiCad dosyaları,
  BOM ve deney rehberlerinin otomatik bölümleri yeniden üretildi.

Co-Authored-By: Claude Opus 5.5 (1M context) <noreply@anthropic.com>
Claude-Session: https://claude.ai/code/session_018J8WVuECVRbQJyCbmF6Nsi
Parts:
- removed U1, U3, U5, U69, U7, U70, U71: SST39SF010A, Package_DIP:DIP-32_W15.24mm, symbol cpu16:SST39SF010A
- removed U68: 74HC157, Package_DIP:DIP-16_W7.62mm, symbol cpu16:74HC157
- added C100, C129, C148, C149, C150, C151, C152, C153, C154, C155, C156, C157, C158, C159, C160, C161, C162, C163, C164, C165, C166, C167, C168, C169, C170, C171, C172, C173, C174, C175, C176, C177, C178, C179, C180, C181, C182, C183, C184, C185, C186, C187, C188, C189, C190, C191, C192, C193, C194, C195, C42, C71: C_100N, Capacitor_THT:C_Disc_D5.0mm_W2.5mm_P5.00mm, symbol cpu16:C_100N
- added U1, U3, U5, U68, U69, U7, U70, U71: 74HC138, Package_DIP:DIP-16_W7.62mm, symbol cpu16:74HC138
- added U147, U148, U149, U150, U151, U152, U153, U154, U155, U156: 74HC151, Package_DIP:DIP-16_W7.62mm, symbol cpu16:74HC151
- added U157, U158, U159, U161, U162, U163: 74HC08, Package_DIP:DIP-14_W7.62mm, symbol cpu16:74HC08
- added U164, U166, U167, U168, U169: 74HC32, Package_DIP:DIP-14_W7.62mm, symbol cpu16:74HC32
- added U171, U172, U173, U174: 74HC00, Package_DIP:DIP-14_W7.62mm, symbol cpu16:74HC00
- added U176: 74HC02, Package_DIP:DIP-14_W7.62mm, symbol cpu16:74HC02
- added U177, U178: 74HC04, Package_DIP:DIP-14_W7.62mm, symbol cpu16:74HC04
- added U179, U180, U181, U182, U183, U184, U185: 74HC10, Package_DIP:DIP-14_W7.62mm, symbol cpu16:74HC10
- added U186: 74HC11, Package_DIP:DIP-14_W7.62mm, symbol cpu16:74HC11
- added U187, U188, U189, U190: 74HC21, Package_DIP:DIP-14_W7.62mm, symbol cpu16:74HC21
- added U191, U192, U193, U194: 74HC20, Package_DIP:DIP-14_W7.62mm, symbol cpu16:74HC20
- U10: Gorev adım çözücü (adım 0 algılama) -> adım çözücü: adım 0..7
- U126: Gorev yapıştırıcı: tek adresli bayt, yazma darbesi -> yapıştırıcı: tek adresli bayt, yazma darbesi, ortak alt küme
- U129: Gorev yapıştırıcı: I girişi, bellek erişimi, yazma darbesi -> yapıştırıcı: I girişi, bellek erişimi, yazma darbesi, komut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
- U132: Gorev yapıştırıcı: çift bayt yazma darbesi, tek bayt yazma darbesi -> yapıştırıcı: çift bayt yazma darbesi, tek bayt yazma darbes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
- U135: Gorev yapıştırıcı: Z bayrağı -> yapıştırıcı: Z bayrağı, kesme girişi, CW5, CW6
- U146: Gorev yapıştırıcı: kelime erişimi, bellek okuma (aktif düşük) -> yapıştırıcı: kelime erişimi, bellek okuma (aktif düşük), CW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
- U160: renamed from C42; value C_100N -> 74HC08; footprint Capacitor_THT:C_Disc_D5.0mm_W2.5mm_P5.00mm -> Package_DIP:DIP-14_W7.62mm; symbol cpu16:C_100N -> cpu16:74HC08; Gorev U41 dekuplaj -> yapıştırıcı: ortak alt küme
- U165: renamed from C71; value C_100N -> 74HC32; footprint Capacitor_THT:C_Disc_D5.0mm_W2.5mm_P5.00mm -> Package_DIP:DIP-14_W7.62mm; symbol cpu16:C_100N -> cpu16:74HC32; Gorev U70 dekuplaj -> yapıştırıcı: CW11, CW12, CW13
- U170: renamed from C100; value C_100N -> 74HC00; footprint Capacitor_THT:C_Disc_D5.0mm_W2.5mm_P5.00mm -> Package_DIP:DIP-14_W7.62mm; symbol cpu16:C_100N -> cpu16:74HC00; Gorev U99 dekuplaj -> yapıştırıcı: CW1, CW2, CW3
- U175: renamed from C129; value C_100N -> 74HC02; footprint Capacitor_THT:C_Disc_D5.0mm_W2.5mm_P5.00mm -> Package_DIP:DIP-14_W7.62mm; symbol cpu16:C_100N -> cpu16:74HC02; Gorev U128 dekuplaj -> yapıştırıcı: CW20, CW25, CW26, CW28
Connections:
- net MC0_0 is gone; now on net MK0: U2.2 (D0)
- net MC0_5 is gone; now on net MK5: U2.7 (D5)
- net MC0_6 is gone; now on net MK6: U2.8 (D6)
- net MC1_0 is gone; now on net GND: U4.2 (D0)
- net MC1_1 is gone; now on net GND: U4.3 (D1)
- net MC1_7 is gone; now on net GND: U4.9 (D7)
- net MC2_7 is gone; now on net MK20: U6.9 (D7)
- net AD0: now also U177.12 (6Y)
- net AD1: now also U177.13 (6A), U190.2 (1B), U192.12 (2C), U70.13 (~{Y2})
- net AD10: now also U193.8 (2Y)
- net AD11: now also U185.12 (1Y)
- net AD12: now also U190.6 (1Y)
- net AD13: now also U194.6 (1Y)
- net AD16: now also U178.10 (5Y)
- net AD17: now also U174.3 (1Y)
- net AD18: now also U194.8 (2Y)
- net AD19: now also U174.6 (2Y)
- net AD2: now also U184.8 (3Y)
- net AD20: now also U174.8 (3Y)
- net AD21: now also U185.6 (2Y)
- net AD22: now also U174.11 (4Y)
- net AD23: now also U185.8 (3Y)
- net AD3: now also U192.8 (2Y)
- net AD4: now also U189.8 (2Y)
- net AD5: now also U176.10 (3Y)
- net AD6: now also U176.13 (4Y)
- net AD7: now also U178.4 (2Y)
- net AD8: now also U178.6 (3Y)
- net AD9: now also U193.6 (1Y)
- net AOP0: now also U69.1 (A0), U70.1 (A0), U71.1 (A0)
- net AOP1: now also U69.2 (A1), U70.2 (A1), U71.2 (A1)
- net AOP2: now also U69.3 (A2), U70.3 (A2), U71.3 (A2)
- net AOP3: now also U69.4 (~{E1}), U70.6 (E3), U71.4 (~{E1})
- net AOP4: now also U163.11 (4Y), U178.1 (1A), U69.5 (~{E2}), U70.4 (~{E1}), U71.6 (E3)
- net COND: now also U129.13 (4B), U146.9 (4A)
- net CW10: now also U163.12 (4A)
- net CW11: now also U178.13 (6A)
- net GND: now also U160.7 (GND), U165.7 (GND), U170.7 (GND), U175.7 (GND), C100.2, C129.2, C148.2, C149.2, C150.2, C151.2, C152.2, C153.2, C154.2, C155.2, C156.2, C157.2, C158.2, C159.2, C160.2, C161.2, C162.2, C163.2, C164.2, C165.2, C166.2, C167.2, C168.2, C169.2, C170.2, C171.2, C172.2, C173.2, C174.2, C175.2, C176.2, C177.2, C178.2, C179.2, C180.2, C181.2, C182.2, C183.2, C184.2, C185.2, C186.2, C187.2, C188.2, C189.2, C190.2, C191.2, C192.2, C193.2, C194.2, C195.2, C42.2, C71.2, U1.8 (GND), U147.8 (GND), U148.3 (I1), U148.8 (GND), U149.2 (I2), U149.4 (I0), U149.8 (GND), U150.1 (I3), U150.3 (I1), U150.8 (GND), U151.3 (I1), U151.8 (GND), U152.1 (I3), U152.13 (I6), U152.3 (I1), U152.4 (I0), U152.8 (GND), U153.3 (I1), U153.4 (I0), U153.8 (GND), U154.1 (I3), U154.12 (I7), U154.3 (I1), U154.8 (GND), U155.1 (I3), U155.13 (I6), U155.3 (I1), U155.8 (GND), U156.13 (I6), U156.3 (I1), U156.4 (I0), U156.8 (GND), U157.7 (GND), U158.7 (GND), U159.7 (GND), U161.7 (GND), U162.7 (GND), U163.7 (GND), U164.7 (GND), U166.7 (GND), U167.7 (GND), U168.7 (GND), U169.7 (GND), U171.7 (GND), U172.7 (GND), U173.7 (GND), U174.7 (GND), U176.7 (GND), U177.7 (GND), U178.7 (GND), U179.7 (GND), U180.7 (GND), U181.7 (GND), U182.7 (GND), U183.7 (GND), U184.7 (GND), U185.7 (GND), U186.7 (GND), U187.7 (GND), U188.7 (GND), U189.7 (GND), U190.7 (GND), U191.7 (GND), U192.7 (GND), U193.7 (GND), U194.7 (GND), U3.5 (~{E2}), U3.8 (GND), U5.5 (~{E2}), U5.8 (GND), U68.5 (~{E2}), U68.8 (GND), U69.8 (GND), U7.5 (~{E2}), U7.8 (GND), U70.5 (~{E2}), U70.8 (GND), U71.5 (~{E2}), U71.8 (GND); no longer U126.12 (4A), U126.13 (4B), U129.12 (4A), U129.13 (4B), U132.10 (3B), U132.12 (4A), U132.13 (4B), U132.9 (3A), U135.11 (4A), U135.12 (4B), U135.5 (2A), U135.8 (3A), U135.9 (3B), U146.11 (5A), U146.13 (6A), U146.5 (3A), U146.9 (4A), U160.2, U165.2, U170.2, U175.2
- net INT: now also U135.5 (2A), U175.3 (1B), U1.5 (~{E2}), U147.12 (I7), U147.3 (I1), U149.13 (I6), U150.4 (I0), U151.4 (I0), U152.14 (I5), U152.2 (I2), U154.15 (I4), U154.4 (I0), U3.4 (~{E1})
- net IR0: now also U182.3 (2A), U5.1 (A0), U7.1 (A0)
- net IR1: now also U182.4 (2B), U5.2 (A1), U7.2 (A1)
- net IR12: now also U1.1 (A0), U3.1 (A0)
- net IR13: now also U1.2 (A1), U3.2 (A1)
- net IR14: now also U1.3 (A2), U3.3 (A2)
- net IR15: now also U1.4 (~{E1}), U3.6 (E3)
- net IR2: now also U182.5 (2C), U5.3 (A2), U7.3 (A2)
- net IR8: now also U169.12 (4A), U178.9 (4A)
- net STEP0: now also U147.11 (S0), U148.11 (S0), U149.11 (S0), U150.11 (S0), U151.11 (S0), U152.11 (S0), U153.11 (S0), U154.11 (S0), U155.11 (S0), U156.11 (S0), U68.1 (A0)
- net STEP1: now also U147.10 (S1), U148.10 (S1), U149.10 (S1), U150.10 (S1), U151.10 (S1), U152.10 (S1), U153.10 (S1), U154.10 (S1), U155.10 (S1), U156.10 (S1), U68.2 (A1)
- net STEP2: now also U147.9 (S2), U148.9 (S2), U149.9 (S2), U150.9 (S2), U151.9 (S2), U152.9 (S2), U153.9 (S2), U154.9 (S2), U155.9 (S2), U156.9 (S2), U68.3 (A2)
- net STEP3: now also U147.7 (~{E}), U148.7 (~{E}), U149.7 (~{E}), U150.7 (~{E}), U151.7 (~{E}), U152.7 (~{E}), U153.7 (~{E}), U154.7 (~{E}), U155.7 (~{E}), U156.7 (~{E}), U68.6 (E3)
- net VCC: now also U160.14 (VCC), U165.14 (VCC), U170.14 (VCC), U175.14 (VCC), C100.1, C129.1, C148.1, C149.1, C150.1, C151.1, C152.1, C153.1, C154.1, C155.1, C156.1, C157.1, C158.1, C159.1, C160.1, C161.1, C162.1, C163.1, C164.1, C165.1, C166.1, C167.1, C168.1, C169.1, C170.1, C171.1, C172.1, C173.1, C174.1, C175.1, C176.1, C177.1, C178.1, C179.1, C180.1, C181.1, C182.1, C183.1, C184.1, C185.1, C186.1, C187.1, C188.1, C189.1, C190.1, C191.1, C192.1, C193.1, C194.1, C195.1, C42.1, C71.1, U1.16 (VCC), U1.6 (E3), U147.16 (VCC), U147.4 (I0), U148.16 (VCC), U149.16 (VCC), U149.3 (I1), U150.16 (VCC), U151.16 (VCC), U152.16 (VCC), U153.16 (VCC), U154.16 (VCC), U155.16 (VCC), U156.16 (VCC), U157.14 (VCC), U158.14 (VCC), U159.14 (VCC), U161.14 (VCC), U162.14 (VCC), U163.14 (VCC), U164.14 (VCC), U166.14 (VCC), U167.14 (VCC), U168.14 (VCC), U169.14 (VCC), U171.14 (VCC), U172.14 (VCC), U173.14 (VCC), U174.14 (VCC), U176.14 (VCC), U177.14 (VCC), U178.14 (VCC), U179.14 (VCC), U179.5 (2C), U180.14 (VCC), U181.14 (VCC), U182.14 (VCC), U183.14 (VCC), U184.14 (VCC), U185.14 (VCC), U186.14 (VCC), U187.14 (VCC), U187.4 (1C), U187.5 (1D), U188.14 (VCC), U189.14 (VCC), U190.14 (VCC), U191.14 (VCC), U191.2 (1B), U191.4 (1C), U191.5 (1D), U192.14 (VCC), U193.14 (VCC), U194.14 (VCC), U3.16 (VCC), U5.16 (VCC), U5.6 (E3), U68.16 (VCC), U69.16 (VCC), U69.6 (E3), U7.16 (VCC), U7.6 (E3), U70.16 (VCC), U71.16 (VCC); no longer U160.1, U165.1, U170.1, U175.1
- net MK5: now reaches U135.10 (3Y)
- net MK6: now reaches U135.13 (4Y)
- net ~{INT}: now reaches U135.4 (2Y)
- net ~{INT}: now also U132.12 (4A), U160.10 (3B), U165.10 (3B), U170.1 (1A), U148.4 (I0), U155.4 (I0), U157.12 (4A), U166.10 (3B), U167.13 (4B), U169.2 (1B), U171.4 (2A), U172.10 (3B), U173.4 (2A), U179.4 (2B), U181.4 (2B), U191.12 (2C)
- net ~{ADIM5}: now reaches U10.10 (~{Y5})
- net ~{ADIM5}: now also U175.11 (4A), U167.4 (2A), U168.1 (1A)
- net ~{ADIM4}: now reaches U10.11 (~{Y4})
- net ~{ADIM4}: now also U165.1 (1A), U175.5 (2A), U164.9 (3A), U167.1 (1A), U168.9 (3A)
- net ~{ADIM3}: now reaches U10.12 (~{Y3})
- net ~{ADIM3}: now also U135.11 (4A), U165.12 (4A), U165.4 (2A), U162.9 (3A), U164.12 (4A), U164.4 (2A), U166.1 (1A), U166.12 (4A), U168.4 (2A)
- net ~{ADIM2}: now reaches U10.13 (~{Y2})
- net ~{ADIM2}: now also U135.8 (3A), U175.8 (3A), U168.12 (4A), U176.2 (1A), U176.5 (2A)
- net ~{ADIM1}: now reaches U10.14 (~{Y1})
- net ~{ADIM1}: now also U175.2 (1A), U162.1 (1A), U166.9 (3A)
- net ~{ADIM7}: now reaches U10.7 (~{Y7})
- net ~{ADIM7}: now also U162.2 (1B), U167.9 (3A)
- net ~{ADIM6}: now reaches U10.9 (~{Y6})
- net ~{ADIM6}: now also U162.10 (3B), U169.1 (1A)
- net ~{KOP9_C0}: now reaches U129.11 (4Y)
- net ~{KOP9_C0}: now also U187.1 (1A)
- net kb1: now reaches U126.11 (4Y)
- net kb1: now also U157.4 (2A)
- net ~{CFLAG}: now reaches U107.6 (~{1Q})
- net ~{CFLAG}: now also U169.4 (2A), U176.11 (4A), U176.8 (3A)
- net kb15: now reaches U132.11 (4Y)
- net kb15: now also U148.2 (I2)
- net MK0: now reaches U132.8 (3Y)
- net kb27: now reaches U146.10 (5Y)
- net kb27: now also U148.13 (I6), U149.12 (I7), U151.14 (I5), U155.14 (I5), U156.12 (I7)
- net kb32: now reaches U146.12 (6Y)
- net kb32: now also U149.15 (I4), U153.13 (I6), U154.14 (I5)
- net kb13: now reaches U146.6 (3Y)
- net kb13: now also U147.13 (I6), U148.12 (I7), U150.12 (I7), U151.12 (I7), U152.12 (I7), U153.12 (I7), U154.13 (I6), U155.12 (I7)
- net ~{COND}: now reaches U146.8 (4Y)
- net ~{COND}: now also U164.2 (1B)
- net IS_STEP0 renamed ADIM0
- net MC0_1 renamed MK1
- net MK1: now also U170.6 (2Y)
- net MC0_2 renamed MK2
- net MK2: now also U170.8 (3Y)
- net MC0_3 renamed MK3
- net MK3: now also U150.5 (Y)
- net MC0_4 renamed MK4
- net MK4: now also U151.5 (Y)
- net MC0_7 renamed MK7
- net MK7: now also U152.5 (Y)
- net MC1_2 renamed MK10
- net MK10: now also U171.11 (4Y)
- net MC1_3 renamed MK11
- net MK11: now also U172.3 (1Y)
- net MC1_4 renamed MK12
- net MK12: now also U172.6 (2Y)
- net MC1_5 renamed MK13
- net MK13: now also U181.8 (3Y)
- net MC1_6 renamed MK14
- net MK14: now also U182.12 (1Y)
- net MC2_0 renamed MK16
- net MK16: now also U153.5 (Y)
- net MC2_1 renamed MK17
- net MK17: now also U154.5 (Y)
- net MC2_2 renamed MK18
- net MK18: now also U173.3 (1Y)
- net MC2_3 renamed MK19
- net MK19: now also U192.6 (1Y)
- net MC2_4 renamed MK20
- net MK20: now also U175.1 (1Y)
- net MC2_5 renamed MK21
- net MK21: now also U155.5 (Y)
- net MC2_6 renamed MK22
- net MK22: now also U183.6 (2Y)
- net MC3_0 renamed MK24
- net MK24: now also U173.8 (3Y)
- net MC3_1 renamed MK25
- net MK25: now also U175.4 (2Y)
- net MC3_2 renamed MK26
- net MK26: now also U175.10 (3Y)
- net MC3_3 renamed MK27
- net MK27: now also U183.8 (3Y)
- net MC3_4 renamed MK28
- net MK28: now also U175.13 (4Y)
- net MC3_5 renamed MK29
- net MK29: now also U176.1 (1Y)
- net MC3_6 renamed MK30
- net MK30: now also U176.4 (2Y)
- net MC3_7 renamed MK31
- net MK31: now also U173.11 (4Y)
- net N1211 renamed N1406
- net N1213 renamed N1408
- net N1215 renamed N1410
- net N1217 renamed N1412
- net N1219 renamed N1414
- net N1221 renamed N1416
- net N1223 renamed N1418
- net N1225 renamed N1420
- net N1227 renamed N1422
- net N1229 renamed N1424
- net N1231 renamed N1426
- net N1233 renamed N1428
- net N1235 renamed N1430
- net N1237 renamed N1432
- net N1239 renamed N1434
- net N1241 renamed N1436
- net N1363 renamed N1558
- net N1364 renamed N1559
- net N1590 renamed N1785
- net N1766 renamed N1961
- net N1769 renamed N1964
- net N1776 renamed N1971
- net N1778 renamed N1973
- net N1779 renamed N1974
- net N1800 renamed N1995
- net N1813 renamed N2008
- net N1826 renamed N2021
- net N1831 renamed N2026
- net N1834 renamed N2029
- net N271 renamed N468
- net N272 renamed N469
- net N275 renamed N472
- net N277 renamed N474
- net N281 renamed N478
- net N284 renamed N481
- net ~{IS_STEP0} renamed ~{ADIM0}
- new net KOP13: U179.1 (1A), U191.6 (1Y)
- new net ak10: U169.11 (4Y), U193.13 (2D)
- new net ak12: U163.8 (3Y), U190.5 (1D), U194.5 (1D)
- new net ak13: U186.8 (3Y), U190.1 (1A)
- new net ak19: U174.12 (4A), U190.8 (2Y)
- new net ak2: U162.11 (4Y), U169.5 (2B), U190.4 (1C)
- new net ak3: U169.6 (2Y), U192.13 (2D)
- new net ak4: U163.3 (1Y), U163.5 (2B), U174.2 (1B), U185.5 (2C), U193.4 (1C)
- new net ak5: U163.6 (2Y), U174.4 (2A), U185.10 (3B), U185.13 (1C), U189.13 (2D)
- new net ak9: U169.8 (3Y), U174.13 (4B), U174.5 (2B), U185.11 (3C), U193.5 (1D), U194.13 (2D)
- new net kb0: U157.9 (3A), U187.6 (1Y)
- new net kb10: U147.15 (I4), U179.6 (2Y)
- new net kb11: U158.8 (3Y), U161.1 (1A), U171.9 (3A), U179.11 (3C), U181.5 (2C), U182.11 (3C), U183.1 (1A), U188.4 (1C)
- new net kb12: U147.14 (I5), U177.9 (4A), U179.8 (3Y)
- new net kb14: U132.13 (4B), U158.11 (4Y), U161.4 (2A), U167.2 (1B), U184.2 (1B), U188.5 (1D)
- new net kb16: U148.1 (I3), U170.3 (1Y)
- new net kb17: U159.3 (1Y), U159.5 (2B), U162.4 (2A), U171.10 (3B), U188.12 (2C)
- new net kb18: U159.6 (2Y), U180.10 (3B), U180.2 (1B), U184.13 (1C)
- new net kb19: U159.8 (3Y), U160.4 (2A), U175.12 (4B), U183.13 (1C)
- new net kb2: U179.12 (1Y), U187.10 (2B)
- new net kb20: U159.11 (4Y), U160.2 (1B), U183.2 (1B)
- new net kb21: U160.3 (1Y), U160.5 (2B), U186.13 (1C)
- new net kb22: U160.6 (2Y), U180.11 (3C), U180.13 (1C), U184.5 (2C)
- new net kb23: U180.1 (1A), U188.6 (1Y)
- new net kb24: U148.15 (I4), U180.12 (1Y)
- new net kb25: U146.11 (5A), U160.8 (3Y), U167.10 (3B), U170.13 (4B), U180.5 (2C)
- new net kb26: U148.14 (I5), U180.6 (2Y)
- new net kb28: U160.11 (4Y), U161.2 (1B), U173.5 (2B), U191.13 (2D)
- new net kb29: U161.3 (1Y), U161.5 (2B), U162.5 (2B), U171.5 (2B)
- new net kb3: U157.2 (1B), U176.6 (2B), U187.8 (2Y)
- new net kb30: U161.6 (2Y), U166.2 (1B), U180.9 (3A)
- new net kb31: U149.1 (I3), U180.8 (3Y)
- new net kb33: U149.14 (I5), U181.12 (1Y)
- new net kb34: U161.8 (3Y), U170.10 (3B)
- new net kb35: U161.11 (4Y), U188.9 (2A)
- new net kb36: U150.2 (I2), U188.8 (2Y)
- new net kb37: U150.15 (I4), U151.15 (I4), U181.6 (2Y)
- new net kb38: U150.14 (I5), U170.11 (4Y)
- new net kb39: U150.13 (I6), U151.13 (I6), U171.3 (1Y)
- new net kb4: U157.3 (1Y), U157.5 (2B)
- new net kb40: U151.2 (I2), U171.6 (2Y)
- new net kb41: U151.1 (I3), U177.2 (1Y)
- new net kb42: U152.15 (I4), U171.8 (3Y)
- new net kb43: U164.6 (2Y), U171.12 (4A)
- new net kb44: U164.8 (3Y), U171.13 (4B)
- new net kb45: U164.11 (4Y), U172.1 (1A)
- new net kb46: U165.3 (1Y), U172.2 (1B)
- new net kb47: U165.5 (2B), U186.12 (1Y)
- new net kb48: U165.6 (2Y), U172.4 (2A)
- new net kb49: U162.3 (1Y), U165.9 (3A)
- new net kb5: U157.10 (3B), U157.6 (2Y), U188.13 (2D)
- new net kb50: U165.8 (3Y), U181.9 (3A), U182.1 (1A)
- new net kb51: U162.6 (2Y), U165.13 (4B)
- new net kb52: U165.11 (4Y), U181.10 (3B)
- new net kb53: U166.3 (1Y), U182.2 (1B)
- new net kb54: U153.2 (I2), U172.8 (3Y)
- new net kb55: U153.1 (I3), U156.1 (I3), U177.4 (2Y)
- new net kb56: U177.5 (3A), U182.6 (2Y)
- new net kb57: U166.5 (2B), U177.6 (3Y)
- new net kb58: U166.6 (2Y), U182.10 (3B)
- new net kb59: U182.9 (3A), U189.6 (1Y)
- new net kb6: U157.13 (4B), U157.8 (3Y), U158.5 (2B), U177.11 (5A)
- new net kb60: U153.15 (I4), U182.8 (3Y)
- new net kb61: U153.14 (I5), U191.8 (2Y)
- new net kb62: U166.8 (3Y), U173.1 (1A)
- new net kb63: U166.13 (4B), U172.11 (4Y)
- new net kb64: U166.11 (4Y), U173.2 (1B)
- new net kb65: U167.3 (1Y), U192.1 (1A)
- new net kb66: U167.6 (2Y), U192.2 (1B)
- new net kb67: U167.8 (3Y), U192.4 (1C)
- new net kb68: U155.2 (I2), U173.6 (2Y)
- new net kb69: U155.15 (I4), U183.12 (1Y)
- new net kb7: U147.2 (I2), U154.2 (I2), U157.11 (4Y), U172.13 (4B)
- new net kb70: U162.8 (3Y), U167.12 (4A)
- new net kb71: U167.11 (4Y), U183.3 (2A)
- new net kb72: U168.2 (1B), U177.8 (4Y)
- new net kb73: U168.3 (1Y), U183.4 (2B)
- new net kb74: U168.6 (2Y), U173.9 (3A)
- new net kb75: U168.10 (3B), U186.6 (2Y)
- new net kb76: U168.8 (3Y), U173.10 (3B)
- new net kb77: U168.11 (4Y), U183.9 (3A)
- new net kb78: U169.3 (1Y), U183.10 (3B)
- new net kb79: U156.2 (I2), U177.10 (5Y)
- new net kb8: U158.3 (1Y), U158.4 (2A), U168.5 (2B), U170.2 (1B), U172.12 (4A), U177.3 (2A)
- new net kb80: U156.15 (I4), U184.12 (1Y)
- new net kb81: U156.14 (I5), U184.6 (2Y)
- new net kb9: U147.1 (I3), U158.6 (2Y)
- new net ~{ADIM8_A}: U161.9 (3A), U170.5 (2B), U183.11 (3C), U183.5 (2C), U68.15 (~{Y0})
- new net ~{ADIM9_A}: U132.10 (3B), U161.10 (3B), U172.5 (2B), U173.13 (4B), U181.11 (3C), U182.13 (1C), U192.5 (1D), U68.14 (~{Y1})
- new net ~{AIS0}: U186.9 (3A), U69.15 (~{Y0})
- new net ~{AIS11}: U163.9 (3A), U70.12 (~{Y3})
- new net ~{AIS12}: U194.1 (1A), U70.11 (~{Y4})
- new net ~{AIS13}: U178.3 (2A), U194.2 (1B), U70.10 (~{Y5})
- new net ~{AIS14}: U163.10 (3B), U176.9 (3B), U70.9 (~{Y6})
- new net ~{AIS15}: U176.12 (4B), U194.4 (1C), U70.7 (~{Y7})
- new net ~{AIS17}: U174.10 (3B), U185.1 (1A), U185.4 (2B), U185.9 (3A), U190.13 (2D), U193.2 (1B), U71.14 (~{Y1})
- new net ~{AIS18}: U169.10 (3B), U169.13 (4B), U185.2 (1B), U71.13 (~{Y2})
- new net ~{AIS1}: U162.12 (4A), U69.14 (~{Y1})
- new net ~{AIS2}: U184.9 (3A), U186.10 (3B), U192.9 (2A), U69.13 (~{Y2})
- new net ~{AIS3}: U162.13 (4B), U184.10 (3B), U69.12 (~{Y3})
- new net ~{AIS4}: U163.4 (2A), U69.11 (~{Y4})
- new net ~{AIS5}: U163.1 (1A), U190.9 (2A), U193.9 (2A), U194.9 (2A), U69.10 (~{Y5})
- new net ~{AIS6}: U174.1 (1A), U185.3 (2A), U189.10 (2B), U190.10 (2B), U193.1 (1A), U193.10 (2B), U194.10 (2B), U69.9 (~{Y6})
- new net ~{AIS7}: U184.11 (3C), U186.11 (3C), U192.10 (2B), U69.7 (~{Y7})
- new net ~{AIS8}: U163.2 (1B), U70.15 (~{Y0})
- new net ~{AIS9}: U174.9 (3A), U178.11 (5A), U178.5 (3A), U189.12 (2C), U190.12 (2C), U193.12 (2C), U194.12 (2C), U70.14 (~{Y1})
- new net ~{ALU_IR}: U163.13 (4B), U178.12 (6Y)
- new net ~{AOP4}: U178.2 (1Y), U189.9 (2A)
- new net ~{IR8}: U169.9 (3A), U178.8 (4Y)
- new net ~{KOP0}: U1.15 (~{Y0}), U165.2 (1B), U166.4 (2A), U177.1 (1A), U184.1 (1A), U186.3 (2A), U188.1 (1A)
- new net ~{KOP10}: U135.9 (3B), U158.12 (4A), U161.13 (4B), U172.9 (3A), U186.1 (1A), U3.13 (~{Y2})
- new net ~{KOP11}: U160.1 (1A), U167.5 (2B), U179.3 (2A), U180.3 (2A), U189.4 (1C), U3.12 (~{Y3})
- new net ~{KOP12}: U159.2 (1B), U186.2 (1B), U186.5 (2C), U3.11 (~{Y4})
- new net ~{KOP13_F0}: U158.9 (3A), U170.12 (4A), U179.2 (1B), U184.3 (2A), U5.15 (~{Y0})
- new net ~{KOP13_F1}: U160.12 (4A), U179.13 (1C), U181.13 (1C), U181.3 (2A), U184.4 (2B), U188.2 (1B), U189.5 (1D), U5.14 (~{Y1})
- new net ~{KOP13}: U191.1 (1A), U3.10 (~{Y5}), U5.4 (~{E1})
- new net ~{KOP14_F0}: U187.2 (1B), U188.10 (2B), U7.15 (~{Y0})
- new net ~{KOP14_F1}: U126.12 (4A), U176.3 (1B), U7.14 (~{Y1})
- new net ~{KOP14_F2}: U126.13 (4B), U175.9 (3B), U7.13 (~{Y2})
- new net ~{KOP14_F3}: U157.1 (1A), U168.13 (4B), U7.12 (~{Y3})
- new net ~{KOP14_F4}: U146.13 (6A), U160.13 (4B), U160.9 (3A), U171.1 (1A), U175.6 (2B), U7.11 (~{Y4})
- new net ~{KOP14_F5}: U146.5 (3A), U158.10 (3B), U171.2 (1B), U180.4 (2B), U68.4 (~{E1}), U7.10 (~{Y5})
- new net ~{KOP14_F6}: U135.12 (4B), U158.2 (1B), U164.5 (2B), U7.9 (~{Y6})
- new net ~{KOP14_F7}: U187.12 (2C), U7.7 (~{Y7})
- new net ~{KOP14}: U3.9 (~{Y6}), U7.4 (~{E1})
- new net ~{KOP15}: U187.13 (2D), U3.7 (~{Y7})
- new net ~{KOP1}: U1.14 (~{Y1}), U158.1 (1A), U164.13 (4B)
- new net ~{KOP2}: U1.13 (~{Y2}), U187.9 (2A)
- new net ~{KOP3}: U1.12 (~{Y3}), U159.4 (2A), U186.4 (2B), U189.1 (1A)
- new net ~{KOP4}: U1.11 (~{Y4}), U159.1 (1A), U164.10 (3B), U189.2 (1B)
- new net ~{KOP5}: U1.10 (~{Y5}), U159.12 (4A), U181.1 (1A), U191.9 (2A)
- new net ~{KOP6}: U1.9 (~{Y6}), U159.13 (4B), U179.9 (3A)
- new net ~{KOP7}: U1.7 (~{Y7}), U159.9 (3A), U181.2 (1B), U191.10 (2B)
- new net ~{KOP8}: U159.10 (3B), U179.10 (3B), U3.15 (~{Y0})
- new net ~{KOP9_C1}: U158.13 (4B), U164.3 (1Y)
- new net ~{KOP9}: U129.12 (4A), U161.12 (4A), U164.1 (1A), U3.14 (~{Y1})
- new net ~{MK0_0}: U132.9 (3A), U147.6 (~{Y})
- new net ~{MK1_0}: U148.6 (~{Y}), U170.4 (2A)
- new net ~{MK2_0}: U149.6 (~{Y}), U170.9 (3A)
- new net ~{MK31_0}: U156.6 (~{Y}), U173.12 (4A)
- no-connect marks 102 -> 108

Commit message: CPU kartı: hata ayıklama LED'leri ve çubuk göstergeler
James Sharman'ın ve Ben Eater'ın breadboard bilgisayarlarındaki gibi, CPU
kartında ne olduğunu gösteren LED'ler (şema = kod, çip eklenmedi):

- 39 durum LED'i (D3–D41, her biri 1 kΩ ile, R3–R41): r0–r7 okuma/yazma
  (~ROE, ~WSEL), veriyolu sürücüsü (~SRC_REG/ALU/PC/MEM/IMM/FLAGS), MEMRD,
  MEMW, TA/TB/MAR/IR yükleme, PC yükleme ve artırma, N/Z/C/V/I bayrakları,
  STEP0–3. Aktif düşük sinyallerde LED VCC'den sinyale bağlı (çıkış 0 iken
  yanar); Board.led() aktifDusuk seçeneği aldı.
- 10 çubuk gösterge (DS1–DS10, DISP_BAR_10, DIP-20) ve önlerinde 8×1 kΩ
  bağımsız direnç dizileri (RN3–RN12, RN_1K_ISO_8, DIP-16): BUS, PC, MAR
  adresi, IR ve ALU sonucu, bayt başına bir gösterge (1. segment bit 0).
- Renkler LED_RENK_KURALLARI'ndan: okuma yeşil, yazma/yükleme turuncu,
  veriyolu sürücüsü beyaz, bayraklar mavi, mikro adım ve çubuklar sarı;
  kırmızı yalnız hata (HALTED, FAULT).
- Yeni parçalar Board.sonaErtele() ile en sona eklenir: mevcut ref'ler ve
  öbür kartların adsız netleri değişmez (yalnız CPU kartının breadboard
  parmak izi değişir).
- 3D: çubuk gösterge gövdesi, bacakları ve segment başına yanma (PCB ve
  breadboard görünümü); aktif düşük LED net 0 iken yanar; bilgi panelinde
  LED, direnç, dizi ve çubuk açıklamaları.
- Yerleşim: göstergeler bloklarının altında; CPU kartı 438×508 mm.
- KiCad: CPU şeması A0'a sığsın diye sıkı çip yerleşimi (denseChips);
  şema, BOM ve sembol kütüphanesi yeniden üretildi; ERC temiz.
- Güç bütçesi: 1 kΩ'luk LED ≈ 3 mA, çubuk gösterge ≈ 24 mA; CPU kartının
  kurulum bütçesi ≈ 0,21 A → ≈ 0,57 A; üretim belgesindeki makine
  toplamı ≈ 1 A olarak kalır.
- Belgeler: led-ve-direnc (renk kuralı, aktif düşük bağlama, çubuk okuma,
  anahtar girişiyle RN3/RN4 uyarısı), kartlar, parcalar, uretim, 3d-gorunum,
  deney 04–07, mimari çizimleri, README sayıları (593 pasif).

Co-Authored-By: Claude Opus 5.5 (1M context) <noreply@anthropic.com>
Claude-Session: https://claude.ai/code/session_0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
Parts:
- added D10, D11, D12, D13, D14, D15, D16, D17, D18, D19, D20, D21, D22, D23, D24, D25, D26, D27, D28, D29, D3, D30, D31, D32, D33, D34, D35, D36, D37, D38, D39, D4, D40, D41, D5, D6, D7, D8, D9: LED, LED_THT:LED_D3.0mm, symbol cpu16:LED
- added DS1, DS10, DS2, DS3, DS4, DS5, DS6, DS7, DS8, DS9: DISP_BAR_10, Display:HDSP-4830, symbol cpu16:DISP_BAR_10
- added R10, R11, R12, R13, R14, R15, R16, R17, R18, R19, R20, R21, R22, R23, R24, R25, R26, R27, R28, R29, R3, R30, R31, R32, R33, R34, R35, R36, R37, R38, R39, R4, R40, R41, R5, R6, R7, R8, R9: R_1K, Resistor_THT:R_Axial_DIN0207_L6.3mm_D2.5mm_P7.62mm_Horizontal, symbol cpu16:R_1K
- added RN10, RN11, RN12, RN3, RN4, RN5, RN6, RN7, RN8, RN9: RN_1K_ISO_8, Package_DIP:DIP-16_W7.62mm, symbol cpu16:RN_1K_ISO_8
Connections:
- net A0: now also RN7.1 (R1A)
- net A1: now also RN7.2 (R2A)
- net A10: now also RN8.3 (R3A)
- net A11: now also RN8.4 (R4A)
- net A12: now also RN8.5 (R5A)
- net A13: now also RN8.6 (R6A)
- net A14: now also RN8.7 (R7A)
- net A15: now also RN8.8 (R8A)
- net A2: now also RN7.3 (R3A)
- net A3: now also RN7.4 (R4A)
- net A4: now also RN7.5 (R5A)
- net A5: now also RN7.6 (R6A)
- net A6: now also RN7.7 (R7A)
- net A7: now also RN7.8 (R8A)
- net A8: now also RN8.1 (R1A)
- net A9: now also RN8.2 (R2A)
- net BUS0: now also RN3.1 (R1A)
- net BUS1: now also RN3.2 (R2A)
- net BUS10: now also RN4.3 (R3A)
- net BUS11: now also RN4.4 (R4A)
- net BUS12: now also RN4.5 (R5A)
- net BUS13: now also RN4.6 (R6A)
- net BUS14: now also RN4.7 (R7A)
- net BUS15: now also RN4.8 (R8A)
- net BUS2: now also RN3.3 (R3A)
- net BUS3: now also RN3.4 (R4A)
- net BUS4: now also RN3.5 (R5A)
- net BUS5: now also RN3.6 (R6A)
- net BUS6: now also RN3.7 (R7A)
- net BUS7: now also RN3.8 (R8A)
- net BUS8: now also RN4.1 (R1A)
- net BUS9: now also RN4.2 (R2A)
- net CFLAG: now also R35.1
- net CW17: now also R27.1
- net CW18: now also R28.1
- net CW21: now also R29.1
- net CW23: now also R30.1
- net GND: now also D25.2 (K), D26.2 (K), D27.2 (K), D28.2 (K), D29.2 (K), D30.2 (K), D32.2 (K), D33.2 (K), D34.2 (K), D35.2 (K), D36.2 (K), D37.2 (K), D38.2 (K), D39.2 (K), D40.2 (K), D41.2 (K), DS1.13 (K8), DS1.14 (K7), DS1.15 (K6), DS1.16 (K5), DS1.17 (K4), DS1.18 (K3), DS1.19 (K2), DS1.20 (K1), DS10.13 (K8), DS10.14 (K7), DS10.15 (K6), DS10.16 (K5), DS10.17 (K4), DS10.18 (K3), DS10.19 (K2), DS10.20 (K1), DS2.13 (K8), DS2.14 (K7), DS2.15 (K6), DS2.16 (K5), DS2.17 (K4), DS2.18 (K3), DS2.19 (K2), DS2.20 (K1), DS3.13 (K8), DS3.14 (K7), DS3.15 (K6), DS3.16 (K5), DS3.17 (K4), DS3.18 (K3), DS3.19 (K2), DS4.13 (K8), DS4.14 (K7), DS4.15 (K6), DS4.16 (K5), DS4.17 (K4), DS4.18 (K3), DS4.19 (K2), DS4.20 (K1), DS5.13 (K8), DS5.14 (K7), DS5.15 (K6), DS5.16 (K5), DS5.17 (K4), DS5.18 (K3), DS5.19 (K2), DS5.20 (K1), DS6.13 (K8), DS6.14 (K7), DS6.15 (K6), DS6.16 (K5), DS6.17 (K4), DS6.18 (K3), DS6.19 (K2), DS6.20 (K1), DS7.13 (K8), DS7.14 (K7), DS7.15 (K6), DS7.16 (K5), DS7.17 (K4), DS7.18 (K3), DS7.19 (K2), DS7.20 (K1), DS8.13 (K8), DS8.14 (K7), DS8.15 (K6), DS8.16 (K5), DS8.17 (K4), DS8.18 (K3), DS8.19 (K2), DS8.20 (K1), DS9.13 (K8), DS9.14 (K7), DS9.15 (K6), DS9.16 (K5), DS9.17 (K4), DS9.18 (K3), DS9.19 (K2), DS9.20 (K1)
- net IFLAG: now also R37.1
- net IR0: now also RN9.1 (R1A)
- net IR1: now also RN9.2 (R2A)
- net IR10: now also RN10.3 (R3A)
- net IR11: now also RN10.4 (R4A)
- net IR12: now also RN10.5 (R5A)
- net IR13: now also RN10.6 (R6A)
- net IR14: now also RN10.7 (R7A)
- net IR15: now also RN10.8 (R8A)
- net IR2: now also RN9.3 (R3A)
- net IR3: now also RN9.4 (R4A)
- net IR4: now also RN9.5 (R5A)
- net IR5: now also RN9.6 (R6A)
- net IR6: now also RN9.7 (R7A)
- net IR7: now also RN9.8 (R8A)
- net IR8: now also RN10.1 (R1A)
- net IR9: now also RN10.2 (R2A)
- net MEMRD: now also R25.1
- net MEMW: now also R26.1
- net NFLAG: now also R33.1
- net PC1: now also RN5.2 (R2A)
- net PC10: now also RN6.3 (R3A)
- net PC11: now also RN6.4 (R4A)
- net PC12: now also RN6.5 (R5A)
- net PC13: now also RN6.6 (R6A)
- net PC14: now also RN6.7 (R7A)
- net PC15: now also RN6.8 (R8A)
- net PC2: now also RN5.3 (R3A)
- net PC3: now also RN5.4 (R4A)
- net PC4: now also RN5.5 (R5A)
- net PC5: now also RN5.6 (R6A)
- net PC6: now also RN5.7 (R7A)
- net PC7: now also RN5.8 (R8A)
- net PC8: now also RN6.1 (R1A)
- net PC9: now also RN6.2 (R2A)
- net PC_INC_EN: now also R32.1
- net RES0: now also RN11.1 (R1A)
- net RES1: now also RN11.2 (R2A)
- net RES10: now also RN12.3 (R3A)
- net RES11: now also RN12.4 (R4A)
- net RES12: now also RN12.5 (R5A)
- net RES13: now also RN12.6 (R6A)
- net RES14: now also RN12.7 (R7A)
- net RES15: now also RN12.8 (R8A)
- net RES2: now also RN11.3 (R3A)
- net RES3: now also RN11.4 (R4A)
- net RES4: now also RN11.5 (R5A)
- net RES5: now also RN11.6 (R6A)
- net RES6: now also RN11.7 (R7A)
- net RES7: now also RN11.8 (R8A)
- net RES8: now also RN12.1 (R1A)
- net RES9: now also RN12.2 (R2A)
- net STEP0: now also R38.1
- net STEP1: now also R39.1
- net STEP2: now also R40.1
- net STEP3: now also R41.1
- net VCC: now also R10.1, R11.1, R12.1, R13.1, R14.1, R15.1, R16.1, R17.1, R18.1, R19.1, R20.1, R21.1, R22.1, R23.1, R24.1, R3.1, R31.1, R4.1, R5.1, R6.1, R7.1, R8.1, R9.1
- net VFLAG: now also R36.1
- net ZFLAG: now also R34.1
- net ~{PC_LOAD}: now also D31.2 (K)
- net ~{ROE0}: now also D3.2 (K)
- net ~{ROE1}: now also D5.2 (K)
- net ~{ROE2}: now also D7.2 (K)
- net ~{ROE3}: now also D9.2 (K)
- net ~{ROE4}: now also D11.2 (K)
- net ~{ROE5}: now also D13.2 (K)
- net ~{ROE6}: now also D15.2 (K)
- net ~{ROE7}: now also D17.2 (K)
- net ~{SRC_ALU}: now also D20.2 (K)
- net ~{SRC_FLAGS}: now also D24.2 (K)
- net ~{SRC_IMM}: now also D23.2 (K)
- net ~{SRC_MEM}: now also D22.2 (K)
- net ~{SRC_PC}: now also D21.2 (K)
- net ~{SRC_REG}: now also D19.2 (K)
- net ~{WSEL0}: now also D4.2 (K)
- net ~{WSEL1}: now also D6.2 (K)
- net ~{WSEL2}: now also D8.2 (K)
- net ~{WSEL3}: now also D10.2 (K)
- net ~{WSEL4}: now also D12.2 (K)
- net ~{WSEL5}: now also D14.2 (K)
- net ~{WSEL6}: now also D16.2 (K)
- net ~{WSEL7}: now also D18.2 (K)
- new net BAR_A0: DS5.1 (A1), RN7.16 (R1B)
- new net BAR_A1: DS5.2 (A2), RN7.15 (R2B)
- new net BAR_A10: DS6.3 (A3), RN8.14 (R3B)
- new net BAR_A11: DS6.4 (A4), RN8.13 (R4B)
- new net BAR_A12: DS6.5 (A5), RN8.12 (R5B)
- new net BAR_A13: DS6.6 (A6), RN8.11 (R6B)
- new net BAR_A14: DS6.7 (A7), RN8.10 (R7B)
- new net BAR_A15: DS6.8 (A8), RN8.9 (R8B)
- new net BAR_A2: DS5.3 (A3), RN7.14 (R3B)
- new net BAR_A3: DS5.4 (A4), RN7.13 (R4B)
- new net BAR_A4: DS5.5 (A5), RN7.12 (R5B)
- new net BAR_A5: DS5.6 (A6), RN7.11 (R6B)
- new net BAR_A6: DS5.7 (A7), RN7.10 (R7B)
- new net BAR_A7: DS5.8 (A8), RN7.9 (R8B)
- new net BAR_A8: DS6.1 (A1), RN8.16 (R1B)
- new net BAR_A9: DS6.2 (A2), RN8.15 (R2B)
- new net BAR_BUS0: DS1.1 (A1), RN3.16 (R1B)
- new net BAR_BUS1: DS1.2 (A2), RN3.15 (R2B)
- new net BAR_BUS10: DS2.3 (A3), RN4.14 (R3B)
- new net BAR_BUS11: DS2.4 (A4), RN4.13 (R4B)
- new net BAR_BUS12: DS2.5 (A5), RN4.12 (R5B)
- new net BAR_BUS13: DS2.6 (A6), RN4.11 (R6B)
- new net BAR_BUS14: DS2.7 (A7), RN4.10 (R7B)
- new net BAR_BUS15: DS2.8 (A8), RN4.9 (R8B)
- new net BAR_BUS2: DS1.3 (A3), RN3.14 (R3B)
- new net BAR_BUS3: DS1.4 (A4), RN3.13 (R4B)
- new net BAR_BUS4: DS1.5 (A5), RN3.12 (R5B)
- new net BAR_BUS5: DS1.6 (A6), RN3.11 (R6B)
- new net BAR_BUS6: DS1.7 (A7), RN3.10 (R7B)
- new net BAR_BUS7: DS1.8 (A8), RN3.9 (R8B)
- new net BAR_BUS8: DS2.1 (A1), RN4.16 (R1B)
- new net BAR_BUS9: DS2.2 (A2), RN4.15 (R2B)
- new net BAR_IR0: DS7.1 (A1), RN9.16 (R1B)
- new net BAR_IR1: DS7.2 (A2), RN9.15 (R2B)
- new net BAR_IR10: DS8.3 (A3), RN10.14 (R3B)
- new net BAR_IR11: DS8.4 (A4), RN10.13 (R4B)
- new net BAR_IR12: DS8.5 (A5), RN10.12 (R5B)
- new net BAR_IR13: DS8.6 (A6), RN10.11 (R6B)
- new net BAR_IR14: DS8.7 (A7), RN10.10 (R7B)
- new net BAR_IR15: DS8.8 (A8), RN10.9 (R8B)
- new net BAR_IR2: DS7.3 (A3), RN9.14 (R3B)
- new net BAR_IR3: DS7.4 (A4), RN9.13 (R4B)
- new net BAR_IR4: DS7.5 (A5), RN9.12 (R5B)
- new net BAR_IR5: DS7.6 (A6), RN9.11 (R6B)
- new net BAR_IR6: DS7.7 (A7), RN9.10 (R7B)
- new net BAR_IR7: DS7.8 (A8), RN9.9 (R8B)
- new net BAR_IR8: DS8.1 (A1), RN10.16 (R1B)
- new net BAR_IR9: DS8.2 (A2), RN10.15 (R2B)
- new net BAR_PC1: DS3.2 (A2), RN5.15 (R2B)
- new net BAR_PC10: DS4.3 (A3), RN6.14 (R3B)
- new net BAR_PC11: DS4.4 (A4), RN6.13 (R4B)
- new net BAR_PC12: DS4.5 (A5), RN6.12 (R5B)
- new net BAR_PC13: DS4.6 (A6), RN6.11 (R6B)
- new net BAR_PC14: DS4.7 (A7), RN6.10 (R7B)
- new net BAR_PC15: DS4.8 (A8), RN6.9 (R8B)
- new net BAR_PC2: DS3.3 (A3), RN5.14 (R3B)
- new net BAR_PC3: DS3.4 (A4), RN5.13 (R4B)
- new net BAR_PC4: DS3.5 (A5), RN5.12 (R5B)
- new net BAR_PC5: DS3.6 (A6), RN5.11 (R6B)
- new net BAR_PC6: DS3.7 (A7), RN5.10 (R7B)
- new net BAR_PC7: DS3.8 (A8), RN5.9 (R8B)
- new net BAR_PC8: DS4.1 (A1), RN6.16 (R1B)
- new net BAR_PC9: DS4.2 (A2), RN6.15 (R2B)
- new net BAR_RES0: DS9.1 (A1), RN11.16 (R1B)
- new net BAR_RES1: DS9.2 (A2), RN11.15 (R2B)
- new net BAR_RES10: DS10.3 (A3), RN12.14 (R3B)
- new net BAR_RES11: DS10.4 (A4), RN12.13 (R4B)
- new net BAR_RES12: DS10.5 (A5), RN12.12 (R5B)
- new net BAR_RES13: DS10.6 (A6), RN12.11 (R6B)
- new net BAR_RES14: DS10.7 (A7), RN12.10 (R7B)
- new net BAR_RES15: DS10.8 (A8), RN12.9 (R8B)
- new net BAR_RES2: DS9.3 (A3), RN11.14 (R3B)
- new net BAR_RES3: DS9.4 (A4), RN11.13 (R4B)
- new net BAR_RES4: DS9.5 (A5), RN11.12 (R5B)
- new net BAR_RES5: DS9.6 (A6), RN11.11 (R6B)
- new net BAR_RES6: DS9.7 (A7), RN11.10 (R7B)
- new net BAR_RES7: DS9.8 (A8), RN11.9 (R8B)
- new net BAR_RES8: DS10.1 (A1), RN12.16 (R1B)
- new net BAR_RES9: DS10.2 (A2), RN12.15 (R2B)
- new net LED_CFLAG: D35.1 (A), R35.2
- new net LED_IFLAG: D37.1 (A), R37.2
- new net LED_IR_L: D30.1 (A), R30.2
- new net LED_MAR_L: D29.1 (A), R29.2
- new net LED_MEMRD: D25.1 (A), R25.2
- new net LED_MEMW: D26.1 (A), R26.2
- new net LED_NFLAG: D33.1 (A), R33.2
- new net LED_PC_INC: D32.1 (A), R32.2
- new net LED_PC_L: D31.1 (A), R31.2
- new net LED_ROE0: D3.1 (A), R3.2
- new net LED_ROE1: D5.1 (A), R5.2
- new net LED_ROE2: D7.1 (A), R7.2
- new net LED_ROE3: D9.1 (A), R9.2
- new net LED_ROE4: D11.1 (A), R11.2
- new net LED_ROE5: D13.1 (A), R13.2
- new net LED_ROE6: D15.1 (A), R15.2
- new net LED_ROE7: D17.1 (A), R17.2
- new net LED_SRC_ALU: D20.1 (A), R20.2
- new net LED_SRC_FLAGS: D24.1 (A), R24.2
- new net LED_SRC_IMM: D23.1 (A), R23.2
- new net LED_SRC_MEM: D22.1 (A), R22.2
- new net LED_SRC_PC: D21.1 (A), R21.2
- new net LED_SRC_REG: D19.1 (A), R19.2
- new net LED_STEP0: D38.1 (A), R38.2
- new net LED_STEP1: D39.1 (A), R39.2
- new net LED_STEP2: D40.1 (A), R40.2
- new net LED_STEP3: D41.1 (A), R41.2
- new net LED_TA_L: D27.1 (A), R27.2
- new net LED_TB_L: D28.1 (A), R28.2
- new net LED_VFLAG: D36.1 (A), R36.2
- new net LED_WSEL0: D4.1 (A), R4.2
- new net LED_WSEL1: D6.1 (A), R6.2
- new net LED_WSEL2: D8.1 (A), R8.2
- new net LED_WSEL3: D10.1 (A), R10.2
- new net LED_WSEL4: D12.1 (A), R12.2
- new net LED_WSEL5: D14.1 (A), R14.2
- new net LED_WSEL6: D16.1 (A), R16.2
- new net LED_WSEL7: D18.1 (A), R18.2
- new net LED_ZFLAG: D34.1 (A), R34.2
- no-connect marks 108 -> 152
Other:
- moved on the sheet: C1, C10, C100, C101, C102, C103, C104, C105, C106, C107, C108, C109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
