File: cpu16/kicad/cpu/cpu.kicad_sch (KiCad schematic)
At the start: 494 parts, among them J1 BACKPLANE_2x32, U1 74HC138, U10 74HC138, U100 74HC153, U101 74HC688, U102 74HC688, U103 74HC541, U104 74HC541, U105 74HC157, U106 74HC74, U107 74HC74, U108 74HC74, U109 74HC541, U11 74HC74, U110 74HC541, U111 74HC151, U112 74HC245, U113 74HC245, U114 74HC245, U115 74HC541, U116 74HC157, U117 74HC08, U118 74HC08, U119 74HC08, U12 74HC74, U120 74HC08, U121 74HC08, U122 74HC08, U123 74HC08, U124 74HC08, U125 74HC08, U126 74HC08, U127 74HC32, U128 74HC32, U129 74HC32, U13 74HC138, U130 74HC00, U131 74HC00, U132 74HC00, U133 74HC02, U134 74HC02, U135 74HC02, U136 74HC86, U137 74HC86, U138 74HC86, U139 74HC86, U14 74HC151, U140 74HC86, U141 74HC86, U142 74HC86, U143 74HC86, U144 74HC86, U145 74HC04, U146 74HC04, U147 74HC151, U148 74HC151, U149 74HC151, U15 74HC151, U150 74HC151, U151 74HC151, U152 74HC151, U153 74HC151, U154 74HC151, U155 74HC151, U156 74HC151, U157 74HC08, U158 74HC08, U159 74HC08, U16 74HC151, U160 74HC08, U161 74HC08, U162 74HC08, U163 74HC08, U164 74HC32, U165 74HC32, U166 74HC32, U167 74HC32, U168 74HC32, U169 74HC32, U17 74HC138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

Commit message: CPU kartı: register içeriği çubuk göstergeleri (74HC541 tamponlarla)
Sekiz register'ın değeri her an görünsün diye (James Sharman'ın
bilgisayarındaki gibi) register'ların 74HC574'leri artık veriyolunu
doğrudan sürmez:

- 574'lerin ~OE'si GND'de, çıkışları R{r}Q0..15 hatlarında; veriyolunu
  register başına iki 74HC541 sürer (~OE1 = ~ROEr, ~OE2 = GND).
- Her register'ın içeriği iki çubuk göstergede (DS11–DS26, önlerinde
  RN13–RN28, 8 × 1 kΩ). Bu göstergeler veriyolunu yüklemez, anahtar
  girişiyle de takılı kalabilir.
- 16 yeni çip kartın en sonunda: U195–U199, sonra yeni taşma diliminden
  U901–U911 (CARD_REF_TASMA; kondansatörleri C196–C199, C901–C912).
  Öbür çiplerin referansları değişmez.
- Board.bacakTasi(): 574'lerin bacakları sonaErtele() içinde yeni netlere
  taşınır; böylece öbür kartların adsız netleri ve breadboard parmak
  izleri değişmez (yalnız CPU kartınınki değişir).
- Yerleşim: çubuk göstergenin direnç dizisi göstergesiyle aynı satırda
  kalır; CPU kartı 438×557 mm.
- Zamanlama: --anakart ve --anakart --tip sonuçları değişmedi (CLK
  956 / 448 ns; CPU + saat 824 / 369 ns).
- Sayılar: CPU kartı 194 → 210 entegre, bilgisayar 444 → 460 entegre,
  593 → 641 pasif. CPU kartının kurulum güç bütçesi ≈ 0,57 → 0,97 A
  (en kötü durum, bütün bitler 1); üretim tablosu ≈ 1,4 A.
- Bölüm metinleri, kartlar, mikromimari, led-ve-direnc, uretim,
  parcalar, Deney 4, README'ler, KiCad şeması, BOM ve mimari çizimleri
  güncellendi; ERC temiz.

Bu değişiklik ayrı tutuldu: geri alınınca 541'ler, DS11–DS26 ve
RN13–RN28 kalkar, 574'ler yine veriyolunu sürer.

Co-Authored-By: Claude Opus 5.5 (1M context) <noreply@anthropic.com>
Claude-Session: https://claude.ai/code/session_018J8WVuECVRbQJyCbmF6Nsi
Parts:
- removed C120, C143, C194, C74, C97: C_100N, Capacitor_THT:C_Disc_D5.0mm_W2.5mm_P5.00mm, symbol cpu16:C_100N
- removed D8: LED, LED_THT:LED_D3.0mm, symbol cpu16:LED
- removed DS10: DISP_BAR_10, Display:HDSP-4830, symbol cpu16:DISP_BAR_10
- added C103, C196, C197, C198, C199, C21, C62, C901, C902, C903, C904, C905, C907, C908, C909, C910, C911, C912: C_100N, Capacitor_THT:C_Disc_D5.0mm_W2.5mm_P5.00mm, symbol cpu16:C_100N
- added D2, D7: LED, LED_THT:LED_D3.0mm, symbol cpu16:LED
- added DS11, DS12, DS13, DS14, DS15, DS16, DS17, DS18, DS19, DS20, DS21, DS22, DS23, DS24, DS25, DS26, DS4, DS9: DISP_BAR_10, Display:HDSP-4830, symbol cpu16:DISP_BAR_10
- added R16, R39, R4: R_1K, Resistor_THT:R_Axial_DIN0207_L6.3mm_D2.5mm_P7.62mm_Horizontal, symbol cpu16:R_1K
- added RN13, RN14, RN15, RN16, RN17, RN18, RN19, RN20, RN21, RN22, RN23, RN24, RN25, RN26, RN27, RN28: RN_1K_ISO_8, Package_DIP:DIP-16_W7.62mm, symbol cpu16:RN_1K_ISO_8
- added RN2: RN_10K_8, Resistor_THT:R_Array_SIP9, symbol cpu16:RN_10K_8
- added U195, U196, U198, U199, U901, U902, U904, U905, U906, U907, U909, U910, U911: 74HC541, Package_DIP:DIP-20_W7.62mm, symbol cpu16:74HC541
- C120: renamed from D7; value LED -> C_100N; footprint LED_THT:LED_D3.0mm -> Capacitor_THT:C_Disc_D5.0mm_W2.5mm_P5.00mm; symbol cpu16:LED -> cpu16:C_100N; Gorev ROE2 LED'i: r2 okuma (~ROE2 = 0, r2 veriyolunu sürüyor) -> U119 dekuplaj
- C143: renamed from DS9; value DISP_BAR_10 -> C_100N; footprint Display:HDSP-4830 -> Capacitor_THT:C_Disc_D5.0mm_W2.5mm_P5.00mm; symbol cpu16:DISP_BAR_10 -> cpu16:C_100N; Gorev ALU sonucu RES0–7: çubuk gösterge -> U142 dekuplaj
- C194: renamed from RN2; value RN_10K_8 -> C_100N; footprint Resistor_THT:R_Array_SIP9 -> Capacitor_THT:C_Disc_D5.0mm_W2.5mm_P5.00mm; symbol cpu16:RN_10K_8 -> cpu16:C_100N; Gorev iç veriyolu: sürülmeyince 0 -> U193 dekuplaj
- C74: renamed from D2; value LED -> C_100N; footprint LED_THT:LED_D3.0mm -> Capacitor_THT:C_Disc_D5.0mm_W2.5mm_P5.00mm; symbol cpu16:LED -> cpu16:C_100N; Gorev FAULT LED'i -> U73 dekuplaj
- C906: renamed from R4; value R_1K -> C_100N; footprint Resistor_THT:R_Axial_DIN0207_L6.3mm_D2.5mm_P7.62mm_Horizontal -> Capacitor_THT:C_Disc_D5.0mm_W2.5mm_P5.00mm; symbol cpu16:R_1K -> cpu16:C_100N; Gorev WSEL0 LED direnci -> U905 dekuplaj
- C97: renamed from DS4; value DISP_BAR_10 -> C_100N; footprint Display:HDSP-4830 -> Capacitor_THT:C_Disc_D5.0mm_W2.5mm_P5.00mm; symbol cpu16:DISP_BAR_10 -> cpu16:C_100N; Gorev PC8–15: çubuk gösterge -> U96 dekuplaj
- D8: renamed from R16; value R_1K -> LED; footprint Resistor_THT:R_Axial_DIN0207_L6.3mm_D2.5mm_P7.62mm_Horizontal -> LED_THT:LED_D3.0mm; symbol cpu16:R_1K -> cpu16:LED; Gorev WSEL6 LED direnci -> WSEL2 LED'i: r2 yazma (~WSEL2 = 0, yükselen kenarda r2 veri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
- DS10: renamed from R39; value R_1K -> DISP_BAR_10; footprint Resistor_THT:R_Axial_DIN0207_L6.3mm_D2.5mm_P7.62mm_Horizontal -> Display:HDSP-4830; symbol cpu16:R_1K -> cpu16:DISP_BAR_10; Gorev STEP1 LED direnci -> ALU sonucu RES8–15: çubuk gösterge
- U197: renamed from C21; value C_100N -> 74HC541; footprint Capacitor_THT:C_Disc_D5.0mm_W2.5mm_P5.00mm -> Package_DIP:DIP-20_W7.62mm; symbol cpu16:C_100N -> cpu16:74HC541; Gorev U20 dekuplaj -> r1 düşük bayt → veriyolu
- U903: renamed from C62; value C_100N -> 74HC541; footprint Capacitor_THT:C_Disc_D5.0mm_W2.5mm_P5.00mm -> Package_DIP:DIP-20_W7.62mm; symbol cpu16:C_100N -> cpu16:74HC541; Gorev U61 dekuplaj -> r3 yüksek bayt → veriyolu
- U908: renamed from C103; value C_100N -> 74HC541; footprint Capacitor_THT:C_Disc_D5.0mm_W2.5mm_P5.00mm -> Package_DIP:DIP-20_W7.62mm; symbol cpu16:C_100N -> cpu16:74HC541; Gorev U102 dekuplaj -> r6 (SP) düşük bayt → veriyolu
Connections:
- net BAR_PC10: now also DS4.3 (A3); no longer C97.3 (A3)
- net BAR_PC11: now also DS4.4 (A4); no longer C97.4 (A4)
- net BAR_PC12: now also DS4.5 (A5); no longer C97.5 (A5)
- net BAR_PC13: now also DS4.6 (A6); no longer C97.6 (A6)
- net BAR_PC14: now also DS4.7 (A7); no longer C97.7 (A7)
- net BAR_PC15: now also DS4.8 (A8); no longer C97.8 (A8)
- net BAR_PC8: now also DS4.1 (A1); no longer C97.1 (A1)
- net BAR_PC9: now also DS4.2 (A2); no longer C97.2 (A2)
- net BAR_RES0: now also DS9.1 (A1); no longer C143.1 (A1)
- net BAR_RES1: now also DS9.2 (A2); no longer C143.2 (A2)
- net BAR_RES10: now also DS10.3 (A3)
- net BAR_RES11: now also DS10.4 (A4)
- net BAR_RES12: now also DS10.5 (A5)
- net BAR_RES13: now also DS10.6 (A6)
- net BAR_RES14: now also DS10.7 (A7)
- net BAR_RES15: now also DS10.8 (A8)
- net BAR_RES2: now also DS9.3 (A3); no longer C143.3 (A3)
- net BAR_RES3: now also DS9.4 (A4); no longer C143.4 (A4)
- net BAR_RES4: now also DS9.5 (A5); no longer C143.5 (A5)
- net BAR_RES5: now also DS9.6 (A6); no longer C143.6 (A6)
- net BAR_RES6: now also DS9.7 (A7); no longer C143.7 (A7)
- net BAR_RES7: now also DS9.8 (A8); no longer C143.8 (A8)
- net BAR_RES8: now also DS10.1 (A1)
- net BAR_RES9: now also DS10.2 (A2)
- net BUS0: now also U197.18 (Y0), U908.18 (Y0), U195.18 (Y0), U199.18 (Y0), U902.18 (Y0), U904.18 (Y0), U906.18 (Y0), U910.18 (Y0); no longer U19.19 (Q0), U21.19 (Q0), U23.19 (Q0), U25.19 (Q0), U27.19 (Q0), U29.19 (Q0), U31.19 (Q0), U33.19 (Q0)
- net BUS1: now also U197.17 (Y1), U908.17 (Y1), U195.17 (Y1), U199.17 (Y1), U902.17 (Y1), U904.17 (Y1), U906.17 (Y1), U910.17 (Y1); no longer U19.18 (Q1), U21.18 (Q1), U23.18 (Q1), U25.18 (Q1), U27.18 (Q1), U29.18 (Q1), U31.18 (Q1), U33.18 (Q1)
- net BUS10: now also U903.16 (Y2), RN2.4 (R3), U196.16 (Y2), U198.16 (Y2), U901.16 (Y2), U905.16 (Y2), U907.16 (Y2), U909.16 (Y2), U911.16 (Y2); no longer C194.4 (R3), U20.17 (Q2), U22.17 (Q2), U24.17 (Q2), U26.17 (Q2), U28.17 (Q2), U30.17 (Q2), U32.17 (Q2), U34.17 (Q2)
- net BUS11: now also U903.15 (Y3), RN2.5 (R4), U196.15 (Y3), U198.15 (Y3), U901.15 (Y3), U905.15 (Y3), U907.15 (Y3), U909.15 (Y3), U911.15 (Y3); no longer C194.5 (R4), U20.16 (Q3), U22.16 (Q3), U24.16 (Q3), U26.16 (Q3), U28.16 (Q3), U30.16 (Q3), U32.16 (Q3), U34.16 (Q3)
- net BUS12: now also U903.14 (Y4), RN2.6 (R5), U196.14 (Y4), U198.14 (Y4), U901.14 (Y4), U905.14 (Y4), U907.14 (Y4), U909.14 (Y4), U911.14 (Y4); no longer C194.6 (R5), U20.15 (Q4), U22.15 (Q4), U24.15 (Q4), U26.15 (Q4), U28.15 (Q4), U30.15 (Q4), U32.15 (Q4), U34.15 (Q4)
- net BUS13: now also U903.13 (Y5), RN2.7 (R6), U196.13 (Y5), U198.13 (Y5), U901.13 (Y5), U905.13 (Y5), U907.13 (Y5), U909.13 (Y5), U911.13 (Y5); no longer C194.7 (R6), U20.14 (Q5), U22.14 (Q5), U24.14 (Q5), U26.14 (Q5), U28.14 (Q5), U30.14 (Q5), U32.14 (Q5), U34.14 (Q5)
- net BUS14: now also U903.12 (Y6), RN2.8 (R7), U196.12 (Y6), U198.12 (Y6), U901.12 (Y6), U905.12 (Y6), U907.12 (Y6), U909.12 (Y6), U911.12 (Y6); no longer C194.8 (R7), U20.13 (Q6), U22.13 (Q6), U24.13 (Q6), U26.13 (Q6), U28.13 (Q6), U30.13 (Q6), U32.13 (Q6), U34.13 (Q6)
- net BUS15: now also U903.11 (Y7), RN2.9 (R8), U196.11 (Y7), U198.11 (Y7), U901.11 (Y7), U905.11 (Y7), U907.11 (Y7), U909.11 (Y7), U911.11 (Y7); no longer C194.9 (R8), U20.12 (Q7), U22.12 (Q7), U24.12 (Q7), U26.12 (Q7), U28.12 (Q7), U30.12 (Q7), U32.12 (Q7), U34.12 (Q7)
- net BUS2: now also U197.16 (Y2), U908.16 (Y2), U195.16 (Y2), U199.16 (Y2), U902.16 (Y2), U904.16 (Y2), U906.16 (Y2), U910.16 (Y2); no longer U19.17 (Q2), U21.17 (Q2), U23.17 (Q2), U25.17 (Q2), U27.17 (Q2), U29.17 (Q2), U31.17 (Q2), U33.17 (Q2)
- net BUS3: now also U197.15 (Y3), U908.15 (Y3), U195.15 (Y3), U199.15 (Y3), U902.15 (Y3), U904.15 (Y3), U906.15 (Y3), U910.15 (Y3); no longer U19.16 (Q3), U21.16 (Q3), U23.16 (Q3), U25.16 (Q3), U27.16 (Q3), U29.16 (Q3), U31.16 (Q3), U33.16 (Q3)
- net BUS4: now also U197.14 (Y4), U908.14 (Y4), U195.14 (Y4), U199.14 (Y4), U902.14 (Y4), U904.14 (Y4), U906.14 (Y4), U910.14 (Y4); no longer U19.15 (Q4), U21.15 (Q4), U23.15 (Q4), U25.15 (Q4), U27.15 (Q4), U29.15 (Q4), U31.15 (Q4), U33.15 (Q4)
- net BUS5: now also U197.13 (Y5), U908.13 (Y5), U195.13 (Y5), U199.13 (Y5), U902.13 (Y5), U904.13 (Y5), U906.13 (Y5), U910.13 (Y5); no longer U19.14 (Q5), U21.14 (Q5), U23.14 (Q5), U25.14 (Q5), U27.14 (Q5), U29.14 (Q5), U31.14 (Q5), U33.14 (Q5)
- net BUS6: now also U197.12 (Y6), U908.12 (Y6), U195.12 (Y6), U199.12 (Y6), U902.12 (Y6), U904.12 (Y6), U906.12 (Y6), U910.12 (Y6); no longer U19.13 (Q6), U21.13 (Q6), U23.13 (Q6), U25.13 (Q6), U27.13 (Q6), U29.13 (Q6), U31.13 (Q6), U33.13 (Q6)
- net BUS7: now also U197.11 (Y7), U908.11 (Y7), U195.11 (Y7), U199.11 (Y7), U902.11 (Y7), U904.11 (Y7), U906.11 (Y7), U910.11 (Y7); no longer U19.12 (Q7), U21.12 (Q7), U23.12 (Q7), U25.12 (Q7), U27.12 (Q7), U29.12 (Q7), U31.12 (Q7), U33.12 (Q7)
- net BUS8: now also U903.18 (Y0), RN2.2 (R1), U196.18 (Y0), U198.18 (Y0), U901.18 (Y0), U905.18 (Y0), U907.18 (Y0), U909.18 (Y0), U911.18 (Y0); no longer C194.2 (R1), U20.19 (Q0), U22.19 (Q0), U24.19 (Q0), U26.19 (Q0), U28.19 (Q0), U30.19 (Q0), U32.19 (Q0), U34.19 (Q0)
- net BUS9: now also U903.17 (Y1), RN2.3 (R2), U196.17 (Y1), U198.17 (Y1), U901.17 (Y1), U905.17 (Y1), U907.17 (Y1), U909.17 (Y1), U911.17 (Y1); no longer C194.3 (R2), U20.18 (Q1), U22.18 (Q1), U24.18 (Q1), U26.18 (Q1), U28.18 (Q1), U30.18 (Q1), U32.18 (Q1), U34.18 (Q1)
- net GND: now also C120.2, C143.2, C194.2, C906.2, C97.2, DS10.13 (K8), DS10.14 (K7), DS10.15 (K6), DS10.16 (K5), DS10.17 (K4), DS10.18 (K3), DS10.19 (K2), DS10.20 (K1), U19.1 (~{OE}), U197.10 (GND), U197.19 (~{OE2}), U20.1 (~{OE}), U21.1 (~{OE}), U22.1 (~{OE}), U23.1 (~{OE}), U24.1 (~{OE}), U25.1 (~{OE}), U26.1 (~{OE}), U27.1 (~{OE}), U28.1 (~{OE}), U29.1 (~{OE}), U30.1 (~{OE}), U31.1 (~{OE}), U32.1 (~{OE}), U33.1 (~{OE}), U34.1 (~{OE}), U903.10 (GND), U903.19 (~{OE2}), U908.10 (GND), U908.19 (~{OE2}), C103.2, C196.2, C197.2, C198.2, C199.2, C21.2, C62.2, C901.2, C902.2, C903.2, C904.2, C905.2, C907.2, C908.2, C909.2, C910.2, C911.2, C912.2, D2.2 (K), DS11.13 (K8), DS11.14 (K7), DS11.15 (K6), DS11.16 (K5), DS11.17 (K4), DS11.18 (K3), DS11.19 (K2), DS11.20 (K1), DS12.13 (K8), DS12.14 (K7), DS12.15 (K6), DS12.16 (K5), DS12.17 (K4), DS12.18 (K3), DS12.19 (K2), DS12.20 (K1), DS13.13 (K8), DS13.14 (K7), DS13.15 (K6), DS13.16 (K5), DS13.17 (K4), DS13.18 (K3), DS13.19 (K2), DS13.20 (K1), DS14.13 (K8), DS14.14 (K7), DS14.15 (K6), DS14.16 (K5), DS14.17 (K4), DS14.18 (K3), DS14.19 (K2), DS14.20 (K1), DS15.13 (K8), DS15.14 (K7), DS15.15 (K6), DS15.16 (K5), DS15.17 (K4), DS15.18 (K3), DS15.19 (K2), DS15.20 (K1), DS16.13 (K8), DS16.14 (K7), DS16.15 (K6), DS16.16 (K5), DS16.17 (K4), DS16.18 (K3), DS16.19 (K2), DS16.20 (K1), DS17.13 (K8), DS17.14 (K7), DS17.15 (K6), DS17.16 (K5), DS17.17 (K4), DS17.18 (K3), DS17.19 (K2), DS17.20 (K1), DS18.13 (K8), DS18.14 (K7), DS18.15 (K6), DS18.16 (K5), DS18.17 (K4), DS18.18 (K3), DS18.19 (K2), DS18.20 (K1), DS19.13 (K8), DS19.14 (K7), DS19.15 (K6), DS19.16 (K5), DS19.17 (K4), DS19.18 (K3), DS19.19 (K2), DS19.20 (K1), DS20.13 (K8), DS20.14 (K7), DS20.15 (K6), DS20.16 (K5), DS20.17 (K4), DS20.18 (K3), DS20.19 (K2), DS20.20 (K1), DS21.13 (K8), DS21.14 (K7), DS21.15 (K6), DS21.16 (K5), DS21.17 (K4), DS21.18 (K3), DS21.19 (K2), DS21.20 (K1), DS22.13 (K8), DS22.14 (K7), DS22.15 (K6), DS22.16 (K5), DS22.17 (K4), DS22.18 (K3), DS22.19 (K2), DS22.20 (K1), DS23.13 (K8), DS23.14 (K7), DS23.15 (K6), DS23.16 (K5), DS23.17 (K4), DS23.18 (K3), DS23.19 (K2), DS23.20 (K1), DS24.13 (K8), DS24.14 (K7), DS24.15 (K6), DS24.16 (K5), DS24.17 (K4), DS24.18 (K3), DS24.19 (K2), DS24.20 (K1), DS25.13 (K8), DS25.14 (K7), DS25.15 (K6), DS25.16 (K5), DS25.17 (K4), DS25.18 (K3), DS25.19 (K2), DS25.20 (K1), DS26.13 (K8), DS26.14 (K7), DS26.15 (K6), DS26.16 (K5), DS26.17 (K4), DS26.18 (K3), DS26.19 (K2), DS26.20 (K1), DS4.13 (K8), DS4.14 (K7), DS4.15 (K6), DS4.16 (K5), DS4.17 (K4), DS4.18 (K3), DS4.19 (K2), DS4.20 (K1), DS9.13 (K8), DS9.14 (K7), DS9.15 (K6), DS9.16 (K5), DS9.17 (K4), DS9.18 (K3), DS9.19 (K2), DS9.20 (K1), RN2.1 (COM), U195.10 (GND), U195.19 (~{OE2}), U196.10 (GND), U196.19 (~{OE2}), U198.10 (GND), U198.19 (~{OE2}), U199.10 (GND), U199.19 (~{OE2}), U901.10 (GND), U901.19 (~{OE2}), U902.10 (GND), U902.19 (~{OE2}), U904.10 (GND), U904.19 (~{OE2}), U905.10 (GND), U905.19 (~{OE2}), U906.10 (GND), U906.19 (~{OE2}), U907.10 (GND), U907.19 (~{OE2}), U909.10 (GND), U909.19 (~{OE2}), U910.10 (GND), U910.19 (~{OE2}), U911.10 (GND), U911.19 (~{OE2}); no longer C143.13 (K8), C143.14 (K7), C143.15 (K6), C143.16 (K5), C143.17 (K4), C143.18 (K3), C143.19 (K2), C143.20 (K1), C194.1 (COM), C97.13 (K8), C97.14 (K7), C97.15 (K6), C97.16 (K5), C97.17 (K4), C97.18 (K3), C97.19 (K2), C97.20 (K1), U197.2, U903.2, U908.2
- net LED_FAULT: now also D2.1 (A); no longer C74.1 (A)
- net LED_ROE2: now also D7.1 (A); no longer C120.1 (A)
- net LED_STEP1: now also R39.2; no longer DS10.2
- net LED_WSEL0: now also R4.2; no longer C906.2
- net LED_WSEL2: now also D8.1 (A)
- net LED_WSEL6: now also R16.2; no longer D8.2
- net STEP1: now also R39.1; no longer DS10.1
- net VCC: now also C120.1, C143.1, C194.1, C74.1, C97.1, U197.20 (VCC), U903.20 (VCC), U908.20 (VCC), C103.1, C196.1, C197.1, C198.1, C199.1, C21.1, C62.1, C901.1, C902.1, C903.1, C904.1, C905.1, C907.1, C908.1, C909.1, C910.1, C911.1, C912.1, R16.1, R4.1, U195.20 (VCC), U196.20 (VCC), U198.20 (VCC), U199.20 (VCC), U901.20 (VCC), U902.20 (VCC), U904.20 (VCC), U905.20 (VCC), U906.20 (VCC), U907.20 (VCC), U909.20 (VCC), U910.20 (VCC), U911.20 (VCC); no longer D8.1, U197.1, U903.1, U908.1
- net ~{ROE0}: now also U195.1 (~{OE1}), U196.1 (~{OE1}); no longer U19.1 (~{OE}), U20.1 (~{OE})
- net ~{ROE1}: now also U197.1 (~{OE1}), U198.1 (~{OE1}); no longer U21.1 (~{OE}), U22.1 (~{OE})
- net ~{ROE2}: now also D7.2 (K), U199.1 (~{OE1}), U901.1 (~{OE1}); no longer C120.2 (K), U23.1 (~{OE}), U24.1 (~{OE})
- net ~{ROE3}: now also U903.1 (~{OE1}), U902.1 (~{OE1}); no longer U25.1 (~{OE}), U26.1 (~{OE})
- net ~{ROE4}: now also U904.1 (~{OE1}), U905.1 (~{OE1}); no longer U27.1 (~{OE}), U28.1 (~{OE})
- net ~{ROE5}: now also U906.1 (~{OE1}), U907.1 (~{OE1}); no longer U29.1 (~{OE}), U30.1 (~{OE})
- net ~{ROE6}: now also U908.1 (~{OE1}), U909.1 (~{OE1}); no longer U31.1 (~{OE}), U32.1 (~{OE})
- net ~{ROE7}: now also U910.1 (~{OE1}), U911.1 (~{OE1}); no longer U33.1 (~{OE}), U34.1 (~{OE})
- net ~{WSEL2}: now also D8.2 (K)
- new net BAR_R0Q0: DS11.1 (A1), RN13.16 (R1B)
- new net BAR_R0Q1: DS11.2 (A2), RN13.15 (R2B)
- new net BAR_R0Q10: DS12.3 (A3), RN14.14 (R3B)
- new net BAR_R0Q11: DS12.4 (A4), RN14.13 (R4B)
- new net BAR_R0Q12: DS12.5 (A5), RN14.12 (R5B)
- new net BAR_R0Q13: DS12.6 (A6), RN14.11 (R6B)
- new net BAR_R0Q14: DS12.7 (A7), RN14.10 (R7B)
- new net BAR_R0Q15: DS12.8 (A8), RN14.9 (R8B)
- new net BAR_R0Q2: DS11.3 (A3), RN13.14 (R3B)
- new net BAR_R0Q3: DS11.4 (A4), RN13.13 (R4B)
- new net BAR_R0Q4: DS11.5 (A5), RN13.12 (R5B)
- new net BAR_R0Q5: DS11.6 (A6), RN13.11 (R6B)
- new net BAR_R0Q6: DS11.7 (A7), RN13.10 (R7B)
- new net BAR_R0Q7: DS11.8 (A8), RN13.9 (R8B)
- new net BAR_R0Q8: DS12.1 (A1), RN14.16 (R1B)
- new net BAR_R0Q9: DS12.2 (A2), RN14.15 (R2B)
- new net BAR_R1Q0: DS13.1 (A1), RN15.16 (R1B)
- new net BAR_R1Q1: DS13.2 (A2), RN15.15 (R2B)
- new net BAR_R1Q10: DS14.3 (A3), RN16.14 (R3B)
- new net BAR_R1Q11: DS14.4 (A4), RN16.13 (R4B)
- new net BAR_R1Q12: DS14.5 (A5), RN16.12 (R5B)
- new net BAR_R1Q13: DS14.6 (A6), RN16.11 (R6B)
- new net BAR_R1Q14: DS14.7 (A7), RN16.10 (R7B)
- new net BAR_R1Q15: DS14.8 (A8), RN16.9 (R8B)
- new net BAR_R1Q2: DS13.3 (A3), RN15.14 (R3B)
- new net BAR_R1Q3: DS13.4 (A4), RN15.13 (R4B)
- new net BAR_R1Q4: DS13.5 (A5), RN15.12 (R5B)
- new net BAR_R1Q5: DS13.6 (A6), RN15.11 (R6B)
- new net BAR_R1Q6: DS13.7 (A7), RN15.10 (R7B)
- new net BAR_R1Q7: DS13.8 (A8), RN15.9 (R8B)
- new net BAR_R1Q8: DS14.1 (A1), RN16.16 (R1B)
- new net BAR_R1Q9: DS14.2 (A2), RN16.15 (R2B)
- new net BAR_R2Q0: DS15.1 (A1), RN17.16 (R1B)
- new net BAR_R2Q1: DS15.2 (A2), RN17.15 (R2B)
- new net BAR_R2Q10: DS16.3 (A3), RN18.14 (R3B)
- new net BAR_R2Q11: DS16.4 (A4), RN18.13 (R4B)
- new net BAR_R2Q12: DS16.5 (A5), RN18.12 (R5B)
- new net BAR_R2Q13: DS16.6 (A6), RN18.11 (R6B)
- new net BAR_R2Q14: DS16.7 (A7), RN18.10 (R7B)
- new net BAR_R2Q15: DS16.8 (A8), RN18.9 (R8B)
- new net BAR_R2Q2: DS15.3 (A3), RN17.14 (R3B)
- new net BAR_R2Q3: DS15.4 (A4), RN17.13 (R4B)
- new net BAR_R2Q4: DS15.5 (A5), RN17.12 (R5B)
- new net BAR_R2Q5: DS15.6 (A6), RN17.11 (R6B)
- new net BAR_R2Q6: DS15.7 (A7), RN17.10 (R7B)
- new net BAR_R2Q7: DS15.8 (A8), RN17.9 (R8B)
- new net BAR_R2Q8: DS16.1 (A1), RN18.16 (R1B)
- new net BAR_R2Q9: DS16.2 (A2), RN18.15 (R2B)
- new net BAR_R3Q0: DS17.1 (A1), RN19.16 (R1B)
- new net BAR_R3Q1: DS17.2 (A2), RN19.15 (R2B)
- new net BAR_R3Q10: DS18.3 (A3), RN20.14 (R3B)
- new net BAR_R3Q11: DS18.4 (A4), RN20.13 (R4B)
- new net BAR_R3Q12: DS18.5 (A5), RN20.12 (R5B)
- new net BAR_R3Q13: DS18.6 (A6), RN20.11 (R6B)
- new net BAR_R3Q14: DS18.7 (A7), RN20.10 (R7B)
- new net BAR_R3Q15: DS18.8 (A8), RN20.9 (R8B)
- new net BAR_R3Q2: DS17.3 (A3), RN19.14 (R3B)
- new net BAR_R3Q3: DS17.4 (A4), RN19.13 (R4B)
- new net BAR_R3Q4: DS17.5 (A5), RN19.12 (R5B)
- new net BAR_R3Q5: DS17.6 (A6), RN19.11 (R6B)
- new net BAR_R3Q6: DS17.7 (A7), RN19.10 (R7B)
- new net BAR_R3Q7: DS17.8 (A8), RN19.9 (R8B)
- new net BAR_R3Q8: DS18.1 (A1), RN20.16 (R1B)
- new net BAR_R3Q9: DS18.2 (A2), RN20.15 (R2B)
- new net BAR_R4Q0: DS19.1 (A1), RN21.16 (R1B)
- new net BAR_R4Q1: DS19.2 (A2), RN21.15 (R2B)
- new net BAR_R4Q10: DS20.3 (A3), RN22.14 (R3B)
- new net BAR_R4Q11: DS20.4 (A4), RN22.13 (R4B)
- new net BAR_R4Q12: DS20.5 (A5), RN22.12 (R5B)
- new net BAR_R4Q13: DS20.6 (A6), RN22.11 (R6B)
- new net BAR_R4Q14: DS20.7 (A7), RN22.10 (R7B)
- new net BAR_R4Q15: DS20.8 (A8), RN22.9 (R8B)
- new net BAR_R4Q2: DS19.3 (A3), RN21.14 (R3B)
- new net BAR_R4Q3: DS19.4 (A4), RN21.13 (R4B)
- new net BAR_R4Q4: DS19.5 (A5), RN21.12 (R5B)
- new net BAR_R4Q5: DS19.6 (A6), RN21.11 (R6B)
- new net BAR_R4Q6: DS19.7 (A7), RN21.10 (R7B)
- new net BAR_R4Q7: DS19.8 (A8), RN21.9 (R8B)
- new net BAR_R4Q8: DS20.1 (A1), RN22.16 (R1B)
- new net BAR_R4Q9: DS20.2 (A2), RN22.15 (R2B)
- new net BAR_R5Q0: DS21.1 (A1), RN23.16 (R1B)
- new net BAR_R5Q1: DS21.2 (A2), RN23.15 (R2B)
- new net BAR_R5Q10: DS22.3 (A3), RN24.14 (R3B)
- new net BAR_R5Q11: DS22.4 (A4), RN24.13 (R4B)
- new net BAR_R5Q12: DS22.5 (A5), RN24.12 (R5B)
- new net BAR_R5Q13: DS22.6 (A6), RN24.11 (R6B)
- new net BAR_R5Q14: DS22.7 (A7), RN24.10 (R7B)
- new net BAR_R5Q15: DS22.8 (A8), RN24.9 (R8B)
- new net BAR_R5Q2: DS21.3 (A3), RN23.14 (R3B)
- new net BAR_R5Q3: DS21.4 (A4), RN23.13 (R4B)
- new net BAR_R5Q4: DS21.5 (A5), RN23.12 (R5B)
- new net BAR_R5Q5: DS21.6 (A6), RN23.11 (R6B)
- new net BAR_R5Q6: DS21.7 (A7), RN23.10 (R7B)
- new net BAR_R5Q7: DS21.8 (A8), RN23.9 (R8B)
- new net BAR_R5Q8: DS22.1 (A1), RN24.16 (R1B)
- new net BAR_R5Q9: DS22.2 (A2), RN24.15 (R2B)
- new net BAR_R6Q0: DS23.1 (A1), RN25.16 (R1B)
- new net BAR_R6Q1: DS23.2 (A2), RN25.15 (R2B)
- new net BAR_R6Q10: DS24.3 (A3), RN26.14 (R3B)
- new net BAR_R6Q11: DS24.4 (A4), RN26.13 (R4B)
- new net BAR_R6Q12: DS24.5 (A5), RN26.12 (R5B)
- new net BAR_R6Q13: DS24.6 (A6), RN26.11 (R6B)
- new net BAR_R6Q14: DS24.7 (A7), RN26.10 (R7B)
- new net BAR_R6Q15: DS24.8 (A8), RN26.9 (R8B)
- new net BAR_R6Q2: DS23.3 (A3), RN25.14 (R3B)
- new net BAR_R6Q3: DS23.4 (A4), RN25.13 (R4B)
- new net BAR_R6Q4: DS23.5 (A5), RN25.12 (R5B)
- new net BAR_R6Q5: DS23.6 (A6), RN25.11 (R6B)
- new net BAR_R6Q6: DS23.7 (A7), RN25.10 (R7B)
- new net BAR_R6Q7: DS23.8 (A8), RN25.9 (R8B)
- new net BAR_R6Q8: DS24.1 (A1), RN26.16 (R1B)
- new net BAR_R6Q9: DS24.2 (A2), RN26.15 (R2B)
- new net BAR_R7Q0: DS25.1 (A1), RN27.16 (R1B)
- new net BAR_R7Q1: DS25.2 (A2), RN27.15 (R2B)
- new net BAR_R7Q10: DS26.3 (A3), RN28.14 (R3B)
- new net BAR_R7Q11: DS26.4 (A4), RN28.13 (R4B)
- new net BAR_R7Q12: DS26.5 (A5), RN28.12 (R5B)
- new net BAR_R7Q13: DS26.6 (A6), RN28.11 (R6B)
- new net BAR_R7Q14: DS26.7 (A7), RN28.10 (R7B)
- new net BAR_R7Q15: DS26.8 (A8), RN28.9 (R8B)
- new net BAR_R7Q2: DS25.3 (A3), RN27.14 (R3B)
- new net BAR_R7Q3: DS25.4 (A4), RN27.13 (R4B)
- new net BAR_R7Q4: DS25.5 (A5), RN27.12 (R5B)
- new net BAR_R7Q5: DS25.6 (A6), RN27.11 (R6B)
- new net BAR_R7Q6: DS25.7 (A7), RN27.10 (R7B)
- new net BAR_R7Q7: DS25.8 (A8), RN27.9 (R8B)
- new net BAR_R7Q8: DS26.1 (A1), RN28.16 (R1B)
- new net BAR_R7Q9: DS26.2 (A2), RN28.15 (R2B)
- new net R0Q0: RN13.1 (R1A), U19.19 (Q0), U195.2 (A0)
- new net R0Q1: RN13.2 (R2A), U19.18 (Q1), U195.3 (A1)
- new net R0Q10: RN14.3 (R3A), U196.4 (A2), U20.17 (Q2)
- new net R0Q11: RN14.4 (R4A), U196.5 (A3), U20.16 (Q3)
- new net R0Q12: RN14.5 (R5A), U196.6 (A4), U20.15 (Q4)
- new net R0Q13: RN14.6 (R6A), U196.7 (A5), U20.14 (Q5)
- new net R0Q14: RN14.7 (R7A), U196.8 (A6), U20.13 (Q6)
- new net R0Q15: RN14.8 (R8A), U196.9 (A7), U20.12 (Q7)
- new net R0Q2: RN13.3 (R3A), U19.17 (Q2), U195.4 (A2)
- new net R0Q3: RN13.4 (R4A), U19.16 (Q3), U195.5 (A3)
- new net R0Q4: RN13.5 (R5A), U19.15 (Q4), U195.6 (A4)
- new net R0Q5: RN13.6 (R6A), U19.14 (Q5), U195.7 (A5)
- new net R0Q6: RN13.7 (R7A), U19.13 (Q6), U195.8 (A6)
- new net R0Q7: RN13.8 (R8A), U19.12 (Q7), U195.9 (A7)
- new net R0Q8: RN14.1 (R1A), U196.2 (A0), U20.19 (Q0)
- new net R0Q9: RN14.2 (R2A), U196.3 (A1), U20.18 (Q1)
- new net R1Q0: RN15.1 (R1A), U197.2 (A0), U21.19 (Q0)
- new net R1Q1: RN15.2 (R2A), U197.3 (A1), U21.18 (Q1)
- new net R1Q10: RN16.3 (R3A), U198.4 (A2), U22.17 (Q2)
- new net R1Q11: RN16.4 (R4A), U198.5 (A3), U22.16 (Q3)
- new net R1Q12: RN16.5 (R5A), U198.6 (A4), U22.15 (Q4)
- new net R1Q13: RN16.6 (R6A), U198.7 (A5), U22.14 (Q5)
- new net R1Q14: RN16.7 (R7A), U198.8 (A6), U22.13 (Q6)
- new net R1Q15: RN16.8 (R8A), U198.9 (A7), U22.12 (Q7)
- new net R1Q2: RN15.3 (R3A), U197.4 (A2), U21.17 (Q2)
- new net R1Q3: RN15.4 (R4A), U197.5 (A3), U21.16 (Q3)
- new net R1Q4: RN15.5 (R5A), U197.6 (A4), U21.15 (Q4)
- new net R1Q5: RN15.6 (R6A), U197.7 (A5), U21.14 (Q5)
- new net R1Q6: RN15.7 (R7A), U197.8 (A6), U21.13 (Q6)
- new net R1Q7: RN15.8 (R8A), U197.9 (A7), U21.12 (Q7)
- new net R1Q8: RN16.1 (R1A), U198.2 (A0), U22.19 (Q0)
- new net R1Q9: RN16.2 (R2A), U198.3 (A1), U22.18 (Q1)
- new net R2Q0: RN17.1 (R1A), U199.2 (A0), U23.19 (Q0)
- new net R2Q1: RN17.2 (R2A), U199.3 (A1), U23.18 (Q1)
- new net R2Q10: RN18.3 (R3A), U24.17 (Q2), U901.4 (A2)
- new net R2Q11: RN18.4 (R4A), U24.16 (Q3), U901.5 (A3)
- new net R2Q12: RN18.5 (R5A), U24.15 (Q4), U901.6 (A4)
- new net R2Q13: RN18.6 (R6A), U24.14 (Q5), U901.7 (A5)
- new net R2Q14: RN18.7 (R7A), U24.13 (Q6), U901.8 (A6)
- new net R2Q15: RN18.8 (R8A), U24.12 (Q7), U901.9 (A7)
- new net R2Q2: RN17.3 (R3A), U199.4 (A2), U23.17 (Q2)
- new net R2Q3: RN17.4 (R4A), U199.5 (A3), U23.16 (Q3)
- new net R2Q4: RN17.5 (R5A), U199.6 (A4), U23.15 (Q4)
- new net R2Q5: RN17.6 (R6A), U199.7 (A5), U23.14 (Q5)
- new net R2Q6: RN17.7 (R7A), U199.8 (A6), U23.13 (Q6)
- new net R2Q7: RN17.8 (R8A), U199.9 (A7), U23.12 (Q7)
- new net R2Q8: RN18.1 (R1A), U24.19 (Q0), U901.2 (A0)
- new net R2Q9: RN18.2 (R2A), U24.18 (Q1), U901.3 (A1)
- new net R3Q0: RN19.1 (R1A), U25.19 (Q0), U902.2 (A0)
- new net R3Q1: RN19.2 (R2A), U25.18 (Q1), U902.3 (A1)
- new net R3Q10: RN20.3 (R3A), U26.17 (Q2), U903.4 (A2)
- new net R3Q11: RN20.4 (R4A), U26.16 (Q3), U903.5 (A3)
- new net R3Q12: RN20.5 (R5A), U26.15 (Q4), U903.6 (A4)
- new net R3Q13: RN20.6 (R6A), U26.14 (Q5), U903.7 (A5)
- new net R3Q14: RN20.7 (R7A), U26.13 (Q6), U903.8 (A6)
- new net R3Q15: RN20.8 (R8A), U26.12 (Q7), U903.9 (A7)
- new net R3Q2: RN19.3 (R3A), U25.17 (Q2), U902.4 (A2)
- new net R3Q3: RN19.4 (R4A), U25.16 (Q3), U902.5 (A3)
- new net R3Q4: RN19.5 (R5A), U25.15 (Q4), U902.6 (A4)
- new net R3Q5: RN19.6 (R6A), U25.14 (Q5), U902.7 (A5)
- new net R3Q6: RN19.7 (R7A), U25.13 (Q6), U902.8 (A6)
- new net R3Q7: RN19.8 (R8A), U25.12 (Q7), U902.9 (A7)
- new net R3Q8: RN20.1 (R1A), U26.19 (Q0), U903.2 (A0)
- new net R3Q9: RN20.2 (R2A), U26.18 (Q1), U903.3 (A1)
- new net R4Q0: RN21.1 (R1A), U27.19 (Q0), U904.2 (A0)
- new net R4Q1: RN21.2 (R2A), U27.18 (Q1), U904.3 (A1)
- new net R4Q10: RN22.3 (R3A), U28.17 (Q2), U905.4 (A2)
- new net R4Q11: RN22.4 (R4A), U28.16 (Q3), U905.5 (A3)
- new net R4Q12: RN22.5 (R5A), U28.15 (Q4), U905.6 (A4)
- new net R4Q13: RN22.6 (R6A), U28.14 (Q5), U905.7 (A5)
- new net R4Q14: RN22.7 (R7A), U28.13 (Q6), U905.8 (A6)
- new net R4Q15: RN22.8 (R8A), U28.12 (Q7), U905.9 (A7)
- new net R4Q2: RN21.3 (R3A), U27.17 (Q2), U904.4 (A2)
- new net R4Q3: RN21.4 (R4A), U27.16 (Q3), U904.5 (A3)
- new net R4Q4: RN21.5 (R5A), U27.15 (Q4), U904.6 (A4)
- new net R4Q5: RN21.6 (R6A), U27.14 (Q5), U904.7 (A5)
- new net R4Q6: RN21.7 (R7A), U27.13 (Q6), U904.8 (A6)
- new net R4Q7: RN21.8 (R8A), U27.12 (Q7), U904.9 (A7)
- new net R4Q8: RN22.1 (R1A), U28.19 (Q0), U905.2 (A0)
- new net R4Q9: RN22.2 (R2A), U28.18 (Q1), U905.3 (A1)
- new net R5Q0: RN23.1 (R1A), U29.19 (Q0), U906.2 (A0)
- new net R5Q1: RN23.2 (R2A), U29.18 (Q1), U906.3 (A1)
- new net R5Q10: RN24.3 (R3A), U30.17 (Q2), U907.4 (A2)
- new net R5Q11: RN24.4 (R4A), U30.16 (Q3), U907.5 (A3)
- new net R5Q12: RN24.5 (R5A), U30.15 (Q4), U907.6 (A4)
- new net R5Q13: RN24.6 (R6A), U30.14 (Q5), U907.7 (A5)
- new net R5Q14: RN24.7 (R7A), U30.13 (Q6), U907.8 (A6)
- new net R5Q15: RN24.8 (R8A), U30.12 (Q7), U907.9 (A7)
- new net R5Q2: RN23.3 (R3A), U29.17 (Q2), U906.4 (A2)
- new net R5Q3: RN23.4 (R4A), U29.16 (Q3), U906.5 (A3)
- new net R5Q4: RN23.5 (R5A), U29.15 (Q4), U906.6 (A4)
- new net R5Q5: RN23.6 (R6A), U29.14 (Q5), U906.7 (A5)
- new net R5Q6: RN23.7 (R7A), U29.13 (Q6), U906.8 (A6)
- new net R5Q7: RN23.8 (R8A), U29.12 (Q7), U906.9 (A7)
- new net R5Q8: RN24.1 (R1A), U30.19 (Q0), U907.2 (A0)
- new net R5Q9: RN24.2 (R2A), U30.18 (Q1), U907.3 (A1)
- new net R6Q0: RN25.1 (R1A), U31.19 (Q0), U908.2 (A0)
- new net R6Q1: RN25.2 (R2A), U31.18 (Q1), U908.3 (A1)
- new net R6Q10: RN26.3 (R3A), U32.17 (Q2), U909.4 (A2)
- new net R6Q11: RN26.4 (R4A), U32.16 (Q3), U909.5 (A3)
- new net R6Q12: RN26.5 (R5A), U32.15 (Q4), U909.6 (A4)
- new net R6Q13: RN26.6 (R6A), U32.14 (Q5), U909.7 (A5)
- new net R6Q14: RN26.7 (R7A), U32.13 (Q6), U909.8 (A6)
- new net R6Q15: RN26.8 (R8A), U32.12 (Q7), U909.9 (A7)
- new net R6Q2: RN25.3 (R3A), U31.17 (Q2), U908.4 (A2)
- new net R6Q3: RN25.4 (R4A), U31.16 (Q3), U908.5 (A3)
- new net R6Q4: RN25.5 (R5A), U31.15 (Q4), U908.6 (A4)
- new net R6Q5: RN25.6 (R6A), U31.14 (Q5), U908.7 (A5)
- new net R6Q6: RN25.7 (R7A), U31.13 (Q6), U908.8 (A6)
- new net R6Q7: RN25.8 (R8A), U31.12 (Q7), U908.9 (A7)
- new net R6Q8: RN26.1 (R1A), U32.19 (Q0), U909.2 (A0)
- new net R6Q9: RN26.2 (R2A), U32.18 (Q1), U909.3 (A1)
- new net R7Q0: RN27.1 (R1A), U33.19 (Q0), U910.2 (A0)
- new net R7Q1: RN27.2 (R2A), U33.18 (Q1), U910.3 (A1)
- new net R7Q10: RN28.3 (R3A), U34.17 (Q2), U911.4 (A2)
- new net R7Q11: RN28.4 (R4A), U34.16 (Q3), U911.5 (A3)
- new net R7Q12: RN28.5 (R5A), U34.15 (Q4), U911.6 (A4)
- new net R7Q13: RN28.6 (R6A), U34.14 (Q5), U911.7 (A5)
- new net R7Q14: RN28.7 (R7A), U34.13 (Q6), U911.8 (A6)
- new net R7Q15: RN28.8 (R8A), U34.12 (Q7), U911.9 (A7)
- new net R7Q2: RN27.3 (R3A), U33.17 (Q2), U910.4 (A2)
- new net R7Q3: RN27.4 (R4A), U33.16 (Q3), U910.5 (A3)
- new net R7Q4: RN27.5 (R5A), U33.15 (Q4), U910.6 (A4)
- new net R7Q5: RN27.6 (R6A), U33.14 (Q5), U910.7 (A5)
- new net R7Q6: RN27.7 (R7A), U33.13 (Q6), U910.8 (A6)
- new net R7Q7: RN27.8 (R8A), U33.12 (Q7), U910.9 (A7)
- new net R7Q8: RN28.1 (R1A), U34.19 (Q0), U911.2 (A0)
- new net R7Q9: RN28.2 (R2A), U34.18 (Q1), U911.3 (A1)
- no-connect marks 152 -> 216
Other:
- moved on the sheet: C120, C74, C906, D8
