File: cpu16/kicad/clk/clk.kicad_sch (KiCad schematic)
At the start: 34 parts, among them J3 BACKPLANE_2x32, SW1 SW_PUSH, SW2 SW_PUSH, SW3 SW_SPDT, SW4 SW_SPDT, U121 74HC14, U122 74HC157, U123 74HC175, U124 74HC74, U125 74HC74, U126 74HC541, U138 74HC08, U143 74HC32, U162 74HC04, X1 OSC_CAN

Commit message: Anakart: bekleme durumlu saat kartı, bellek ve önbellek kartları (kapı seviyesi)
Saat kartı: ~WAIT (10 kΩ ile 1'e çekili) s7'nin ortasında W flip-flop'una örneklenir;
W = 1 iken CLK ve WR_WIN kapalı kalır, her bekleme tam bir CPU saati (8 OSC) sürer.
TCLK (uzatılmayan OSC/8, Johnson Q1) ve tamponlu OSC arka panele çıkar. ADIM kipinde
bir basış bekleme turları dahil tam bir döngü. 9 → 10 entegre.

Bellek kartı (bellek, 31 entegre): ~IO çözümü, 4 × 74HC273 bank register'ı (reset
0/32/33/34, geri okuma), PA14..PA19, Flash SST39SF010A + RAM AS6C4008 8 bit, TCLK ile
yürüyen bayt sıralayıcı, boş bölge 0xFF, DE/DO çekme dirençleri.

Önbellek kartı (onbellek, 37 entegre): 2 KB doğrudan eşlemeli, 1024 kelimelik satır,
etiket [19:11] + geçerli, 74HC688 karşılaştırma, write-through, yazma gözetleme (RAM:
güncelle, Flash: geçersiz kıl), reset'te sayıcıyla etiket temizleme, CACHE_CTRL, 4 ×
74HC590 isabet/ıskalama sayacı; ana belleğe giden her erişime tam MEM_WAIT = 2 bekleme.

machine-board.ts: buildMachineBoard({ cards }) ve GateMachine (CPU + saat + bellek +
önbellek; ek kartlar için kanca). bus-master.ts: CPU kartı yerine arka paneli süren
düzenek (Machine'in veri yolu izini kartlarda yeniden oynatmak için).

KiCad: bellek (A2) ve onbellek (A1) projeleri, kart klasöründe BOM; arka panel netleri
BACKPLANE'den. npm run cpu16 -- board artık anakartın özetini ve ERC'sini de yazar.

Testler: anakart-bellek.test.ts (BIOS açılışı, monitör komutları, F ile Flash yükleme,
64 bank/gözetleme/sayaç senaryosu, 1 MB harita — her erişimde değer, bekleme, bank,
sayaç), anakart-sistem.test.ts (saat kartı bekleme turları ve ADIM kipi; CPU dahil
tam sistem Machine ile komut komut: RAM'den programlar, sınama programı, BIOS açılışı).

Co-Authored-By: Claude Opus 5.5 (1M context) <noreply@anthropic.com>
Claude-Session: https://claude.ai/code/session_018J8WVuECVRbQJyCbmF6Nsi
Parts:
- removed R6: R_330, Resistor_THT:R_Axial_DIN0207_L6.3mm_D2.5mm_P7.62mm_Horizontal, symbol cpu16:R_330
- added C169: C_100N, Capacitor_THT:C_Disc_D5.0mm_W2.5mm_P5.00mm, symbol cpu16:C_100N
- added R6: R_10K, Resistor_THT:R_Axial_DIN0207_L6.3mm_D2.5mm_P7.62mm_Horizontal, symbol cpu16:R_10K
- added R7: R_330, Resistor_THT:R_Axial_DIN0207_L6.3mm_D2.5mm_P7.62mm_Horizontal, symbol cpu16:R_330
- added U163: 74HC04, Package_DIP:DIP-14_W7.62mm, symbol cpu16:74HC04
- C167: Gorev U143 dekuplaj -> U139 dekuplaj
- C168: Gorev U162 dekuplaj -> U144 dekuplaj
- U123: Gorev Johnson sayacı: osilatör / 8 → CLK ve yazma penceresi -> Johnson sayacı: osilatör / 8 → CLK, yazma penceresi, TCLK
- U125: Gorev GO: adım kipinde bir tam döngü boyunca saat izni -> GO: adım kipinde bir tam döngü boyunca saat izni; W: beklem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
- U126: Gorev arka panel saat ve reset sürücüsü -> arka panel saat, TCLK, OSC ve reset sürücüsü
- U138: Gorev yapıştırıcı: yazma penceresi (s5, s6), basış anı (bir osilatör periyodu), GO tut, kapılı osilatör -> yapıştırıcı: yazma penceresi (s5, s6), basış anı (bir osilatör periyodu), GO tut, sayaç s7'de
- U139: renamed from U143; value 74HC32 -> 74HC08; symbol cpu16:74HC32 -> cpu16:74HC08; Gorev yapıştırıcı: sayaç s0'da değil, GO sonraki, saat izni -> yapıştırıcı: ~WAIT örnekleme kenarı: s7'nin ortası, bekleme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
- U144: renamed from U162; value 74HC04 -> 74HC32; symbol cpu16:74HC04 -> cpu16:74HC32; Gorev yapıştırıcı: osilatör tersi (eşzamanlama) -> yapıştırıcı: sayaç s0'da değil, GO tut (s0 değil ya da bekl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
Connections:
- net AUTO: now also U144.12 (4A); no longer U139.9 (3A)
- net CLK: now also R7.1
- net GND: now also C169.2, U163.11 (5A), U163.13 (6A), U163.5 (3A), U163.7 (GND), U163.9 (4A); no longer U125.11 (2CLK), U125.12 (2D), U126.5 (A3), U126.6 (A4), U139.12 (4A), U139.13 (4B), U144.11 (5A), U144.13 (6A), U144.3 (2A), U144.5 (3A), U144.9 (4A)
- net GO: now also U144.13 (4B); no longer U139.10 (3B)
- net GO_NEXT: now also U144.8 (3Y); no longer U139.6 (2Y)
- net JCLK: now also U139.4 (2A); no longer U126.2 (A0)
- net JQ0: now also U144.1 (1A); no longer U139.1 (1A)
- net JQ1: now also U126.5 (A3)
- net JQ3: now also U138.13 (4B), U144.2 (1B); no longer U139.2 (1B)
- net JWR: now also U139.9 (3A); no longer U126.3 (A1)
- net LED_CLK: now also R7.2
- net OSC_G: now also U139.11 (4Y); no longer U138.11 (4Y)
- net OSC_RUN: now also U139.13 (4B), U144.11 (4Y); no longer U138.13 (4B), U139.8 (3Y)
- net OSC_SRC: now also U126.6 (A4), U139.12 (4A), U163.1 (1A); no longer U138.12 (4A), U144.1 (1A)
- net PRESS: now also U144.9 (3A); no longer U139.4 (2A)
- net VCC: now also C169.1, R6.1, U163.14 (VCC); no longer U125.13 (~{2CLR})
- net ~{IS_S0}: now also U144.3 (1Y), U144.4 (2A); no longer U138.10 (3B), U139.3 (1Y)
- net ~{OSC_SRC}: now also U139.1 (1A), U163.2 (1Y); no longer U144.2 (1Y)
- net ~{RST}: now also U125.13 (~{2CLR})
- net ~{WST}: now reaches U125.8 (~{2Q})
- net ~{WST}: now also U139.10 (3B), U139.5 (2B)
- net WST: now reaches U125.9 (2Q)
- net WST: now also U144.5 (2B)
- net OSC: now reaches U126.14 (Y4)
- net OSC: now also J3.49
- net TCLK: now reaches U126.15 (Y3)
- net TCLK: now also J3.48
- net ~{WAIT}: now reaches J3.46
- net ~{WAIT}: now also R6.2, U163.3 (2A)
- net ~{JQ2}: now reaches U123.11 (~{Q2})
- net ~{JQ2}: now also U138.12 (4A)
- net N1938: now reaches U144.10 (3B)
- net N1938: now also U138.8 (3Y)
- net GO_HOLD: now reaches U144.6 (2Y)
- net GO_HOLD: now also U138.10 (3B)
- removed net N1936: U138.8 (3Y), U139.5 (2B)
- new net CLK_G: U126.2 (A0), U139.6 (2Y)
- new net JS7: U138.11 (4Y), U139.2 (1B)
- new net WAITREQ: U125.12 (2D), U163.4 (2Y)
- new net WAIT_CK: U125.11 (2CLK), U139.3 (1Y)
- new net WR_G: U126.3 (A1), U139.8 (3Y)
- no-connect marks 39 -> 29
Other:
- moved on the sheet: U144
