File: cpu16/kicad/clk/clk.kicad_sch (KiCad schematic)
At the start: 37 parts, among them J201 BACKPLANE_2x32, SW201 SW_PUSH, SW202 SW_PUSH, SW203 SW_SPDT, SW204 SW_SPDT, U201 74HC14, U202 74HC157, U203 74HC175, U204 74HC74, U205 74HC74, U206 74HC541, U207 74HC08, U208 74HC08, U209 74HC32, U210 74HC04, X201 OSC_CAN

Commit message: Kontrol birimi: mikrokod ve ALU ROM'ları yerine 74HC kapı devresi
CPU kartındaki 7 SST39SF010A (4 mikrokod, 3 ALU kod çözme ROM'u) kalktı. Yerine
board/kontrol.ts, cpu16.ucode'dan (tek kaynak) ve aluControl tablosundan çok seviyeli
bir 74HC devresi üretir ve Board API ile gerçek çipler olarak yerleştirir:

- Mikrokod: adım ve komut çözücüleri (74HC138; INT = 1 iken komutlar pasif, f3'e göre
  dallanan komutlara alt çözücü), aynı mikro programı çalıştıran (op, f3, COND)
  atomları, ortak alt kümeli VEYA ağı, sık kullanılan bitler için adım seçici
  (74HC151), adım 8..15 için SWI hattıyla açılan çözücü.
- ALU kod çözme: işlem çözücüleri (3 × 74HC138), işlem bitleri, h ve C terimleri.
- Yeni kapı çipleri: 74HC11, 74HC20, 74HC21, 74HC27, 74HC30 (veri sayfası pin sırası,
  doğruluk tablosu, zamanlama modeli, KiCad sembolü).
- Board: esnek yapıştırıcı kapılar (kartın diğer kapılarından sonra paketlenir, son
  çipi az dolu türü başka türlerin boş birimlerine taşır) ve defer(). Çözücüler eski
  ROM'ların yuvalarına (U1, U3, U5, U7, U10, U68–U71) oturur: kartın diğer bütün
  çiplerinin referansları değişmedi.
- CPU kartı 146 → 194 entegre; en kötü durumda CPU saati 860 → 824 ns (1,21 MHz),
  tipik 470 → 369 ns.
- Denklik testi (tests/kontrol.test.ts): kontrol birimi tek başına bir kartta, gerçek
  çip modelleriyle (LogicSim) 8192 mikrokod adresinin ve 128 ALU adresinin hepsinde
  tabloyla aynı kelimeyi verir.
- roms.ts, cpu16/roms/ ve "roms" komutu kalktı; "kontrol" komutu gömülü mikrokodu
  (micro/cpu16-ucode.ts) yeniler ve devreyi denetler. GateComputer ve GateMachine artık
  mikrokod istemez.
- CPU şeması A0'a sığsın diye dekuplaj kondansatörleri dar sütunlarda; KiCad dosyaları,
  BOM ve deney rehberlerinin otomatik bölümleri yeniden üretildi.

Co-Authored-By: Claude Opus 5.5 (1M context) <noreply@anthropic.com>
Claude-Session: https://claude.ai/code/session_018J8WVuECVRbQJyCbmF6Nsi
Connections:
- net N1949 renamed N2144
Changed lines of the file:
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@@
   (label "JWR" (at 134.62 231.14 0) (fields_autoplaced) (effects (font (size 1.27 1.27)) (justify left bottom)))
   (label "PRESS" (at 134.62 233.68 0) (fields_autoplaced) (effects (font (size 1.27 1.27)) (justify left bottom)))
-  (label "N1949" (at 134.62 236.22 0) (fields_autoplaced) (effects (font (size 1.27 1.27)) (justify left bottom)))
+  (label "N2144" (at 134.62 236.22 0) (fields_autoplaced) (effects (font (size 1.27 1.27)) (justify left bottom)))
   (label "JS7" (at 134.62 238.76 0) (fields_autoplaced) (effects (font (size 1.27 1.27)) (justify left bottom)))
   (label "GND" (at 124.46 256.54 270) (fields_autoplaced) (effects (font (size 1.27 1.27)) (justify right bottom)))
@@
   (label "WST" (at 185.42 104.14 180) (fields_autoplaced) (effects (font (size 1.27 1.27)) (justify right bottom)))
   (label "PRESS" (at 185.42 106.68 180) (fields_autoplaced) (effects (font (size 1.27 1.27)) (justify right bottom)))
-  (label "N1949" (at 185.42 109.22 180) (fields_autoplaced) (effects (font (size 1.27 1.27)) (justify right bottom)))
+  (label "N2144" (at 185.42 109.22 180) (fields_autoplaced) (effects (font (size 1.27 1.27)) (justify right bottom)))
   (label "AUTO" (at 185.42 111.76 180) (fields_autoplaced) (effects (font (size 1.27 1.27)) (justify right bottom)))
   (label "GO" (at 185.42 114.3 180) (fields_autoplaced) (effects (font (size 1.27 1.27)) (justify right bottom)))
