File: cpu16/kicad/bellek/bellek.kicad_sch (KiCad schematic)
At the start: 67 parts, among them J401 BACKPLANE_2x32, U401 74HC688, U402 74HC688, U403 74HC139, U404 74HC273, U405 74HC273, U406 74HC273, U407 74HC273, U408 74HC153, U409 74HC153, U410 74HC153, U411 74HC541, U412 74HC541, U413 74HC541, U414 74HC541, U415 74HC74, U416 74HC74, U417 74HC574, U418 74HC245, U419 74HC245, U420 SST39SF010A, U421 AS6C4008, U422 74HC08, U423 74HC08, U424 74HC32, U425 74HC32, U426 74HC00, U427 74HC00, U428 74HC02, U429 74HC04, U430 74HC04, U431 74HC04

Commit message: Kontrol birimi: mikrokod ve ALU ROM'ları yerine 74HC kapı devresi
CPU kartındaki 7 SST39SF010A (4 mikrokod, 3 ALU kod çözme ROM'u) kalktı. Yerine
board/kontrol.ts, cpu16.ucode'dan (tek kaynak) ve aluControl tablosundan çok seviyeli
bir 74HC devresi üretir ve Board API ile gerçek çipler olarak yerleştirir:

- Mikrokod: adım ve komut çözücüleri (74HC138; INT = 1 iken komutlar pasif, f3'e göre
  dallanan komutlara alt çözücü), aynı mikro programı çalıştıran (op, f3, COND)
  atomları, ortak alt kümeli VEYA ağı, sık kullanılan bitler için adım seçici
  (74HC151), adım 8..15 için SWI hattıyla açılan çözücü.
- ALU kod çözme: işlem çözücüleri (3 × 74HC138), işlem bitleri, h ve C terimleri.
- Yeni kapı çipleri: 74HC11, 74HC20, 74HC21, 74HC27, 74HC30 (veri sayfası pin sırası,
  doğruluk tablosu, zamanlama modeli, KiCad sembolü).
- Board: esnek yapıştırıcı kapılar (kartın diğer kapılarından sonra paketlenir, son
  çipi az dolu türü başka türlerin boş birimlerine taşır) ve defer(). Çözücüler eski
  ROM'ların yuvalarına (U1, U3, U5, U7, U10, U68–U71) oturur: kartın diğer bütün
  çiplerinin referansları değişmedi.
- CPU kartı 146 → 194 entegre; en kötü durumda CPU saati 860 → 824 ns (1,21 MHz),
  tipik 470 → 369 ns.
- Denklik testi (tests/kontrol.test.ts): kontrol birimi tek başına bir kartta, gerçek
  çip modelleriyle (LogicSim) 8192 mikrokod adresinin ve 128 ALU adresinin hepsinde
  tabloyla aynı kelimeyi verir.
- roms.ts, cpu16/roms/ ve "roms" komutu kalktı; "kontrol" komutu gömülü mikrokodu
  (micro/cpu16-ucode.ts) yeniler ve devreyi denetler. GateComputer ve GateMachine artık
  mikrokod istemez.
- CPU şeması A0'a sığsın diye dekuplaj kondansatörleri dar sütunlarda; KiCad dosyaları,
  BOM ve deney rehberlerinin otomatik bölümleri yeniden üretildi.

Co-Authored-By: Claude Opus 5.5 (1M context) <noreply@anthropic.com>
Claude-Session: https://claude.ai/code/session_018J8WVuECVRbQJyCbmF6Nsi
Connections:
- net N2101 renamed N2296
Changed lines of the file:
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@@
   (label "GND" (at 325.12 154.94 180) (fields_autoplaced) (effects (font (size 1.27 1.27)) (justify right bottom)))
   (label "GND" (at 325.12 157.48 180) (fields_autoplaced) (effects (font (size 1.27 1.27)) (justify right bottom)))
-  (label "N2101" (at 345.44 139.7 0) (fields_autoplaced) (effects (font (size 1.27 1.27)) (justify left bottom)))
+  (label "N2296" (at 345.44 139.7 0) (fields_autoplaced) (effects (font (size 1.27 1.27)) (justify left bottom)))
   (no_connect (at 345.44 142.24))
   (no_connect (at 345.44 144.78))
@@
   (label "VCC" (at 335.28 177.8 90) (fields_autoplaced) (effects (font (size 1.27 1.27)) (justify left bottom)))
   (label "M_SODD" (at 325.12 226.06 180) (fields_autoplaced) (effects (font (size 1.27 1.27)) (justify right bottom)))
-  (label "N2101" (at 325.12 228.6 180) (fields_autoplaced) (effects (font (size 1.27 1.27)) (justify right bottom)))
+  (label "N2296" (at 325.12 228.6 180) (fields_autoplaced) (effects (font (size 1.27 1.27)) (justify right bottom)))
   (label "GND" (at 325.12 231.14 180) (fields_autoplaced) (effects (font (size 1.27 1.27)) (justify right bottom)))
   (label "GND" (at 325.12 233.68 180) (fields_autoplaced) (effects (font (size 1.27 1.27)) (justify right bottom)))
