File: cpu16/kicad/bellek/bellek.kicad_sch (KiCad schematic)
At the start: 67 parts, among them J401 BACKPLANE_2x32, U401 74HC688, U402 74HC688, U403 74HC139, U404 74HC273, U405 74HC273, U406 74HC273, U407 74HC273, U408 74HC153, U409 74HC153, U410 74HC153, U411 74HC541, U412 74HC541, U413 74HC541, U414 74HC541, U415 74HC74, U416 74HC74, U417 74HC574, U418 74HC245, U419 74HC245, U420 SST39SF010A, U421 AS6C4008, U422 74HC08, U423 74HC08, U424 74HC32, U425 74HC32, U426 74HC00, U427 74HC00, U428 74HC02, U429 74HC04, U430 74HC04, U431 74HC04

Commit message: Anakart yalnız yaygın parçalarla: 28C256 + 4 × 62256, kendin yap bellek kartı
AFU kararı: bilgisayar yalnız yaygın 7400 serisi lojikle ve iki bellek
çipiyle (62256, 28C256) kurulur.

Bellek kartı (31 → 34 entegre):
- SST39SF010A yerine 28C256 (32 KB, fiziksel 0x00000–0x07FFF, bank 0–1)
- AS6C4008 yerine 4 × 62256 (128 KB, 0x80000–0x9FFFF, bank 32–39)
- çip seçimi tek 74HC138; geri kalan bölgeler boş (0xFF, yazma yok sayılır)

Nadir parçalar çıktı:
- önbellek sayaçları 74HC590 → 74HC161 × 8 + 74HC541 × 4 (37 → 46)
- zamanlayıcı 74HC193 → 74HC161 (tümleyeni yukarı sayar)
- kesme öncelik kodlayıcısı 74HC148 → kapılar
- video adres sayacı (VADDR) 74HC193 → 74HC161 × 4 + yükleme bayrakları
- karakter ROM'u 28C256; yavaşlığı font register'ıyla bir aşamalık boru
  hattında karşılanır (V_H2 en kötü 262 ns, font yolu 199 ns ≤ 317,8);
  resim Machine ile aynı (video 69 → 73 entegre)
- 74HC166 kalır: 74HC165'in eşzamansız yüklemesi piksel saatine sığmaz

Kendin yap bellek kartı (kyb, 22 entegre): FF40–FF4F, 16 bayt, her bayt
bir 74HC574; 74HC138 çözücüler ve 74HC245 veri yolu tamponları. Machine
aygıtı, KiCad klasörü, kapı seviyesi kart Machine ile döngü döngüsüne aynı.

Machine'de At28c256 modeli (sayfa yazma, tBLC, yazma döngüsü, DATA
yoklaması, toggle biti, SDP); kapı seviyesi kartlar aynı modeli kullanır.
BIOS: F komutu korumalı sayfa yazmasıyla yalnız bank 1'e, I komutu yazma
korumasını gösterir, T bank 32–39'u sınar. Deney 8 programı 8 bank sayar,
boş bölgeleri denetler; Deney 14 programı ve testi eklendi.

Co-Authored-By: Claude Opus 5.5 (1M context) <noreply@anthropic.com>
Claude-Session: https://claude.ai/code/session_018J8WVuECVRbQJyCbmF6Nsi
Parts:
- removed U420: SST39SF010A, Package_DIP:DIP-32_W15.24mm_Socket, symbol cpu16:SST39SF010A
- removed U421: AS6C4008, Package_DIP:DIP-32_W15.24mm, symbol cpu16:AS6C4008
- removed U422, U423: 74HC08, Package_DIP:DIP-14_W7.62mm, symbol cpu16:74HC08
- removed U424, U425: 74HC32, Package_DIP:DIP-14_W7.62mm, symbol cpu16:74HC32
- removed U426, U427: 74HC00, Package_DIP:DIP-14_W7.62mm, symbol cpu16:74HC00
- removed U428: 74HC02, Package_DIP:DIP-14_W7.62mm, symbol cpu16:74HC02
- removed U429, U430, U431: 74HC04, Package_DIP:DIP-14_W7.62mm, symbol cpu16:74HC04
- added C412, C433, C434, C435: C_100N, Capacitor_THT:C_Disc_D5.0mm_W2.5mm_P5.00mm, symbol cpu16:C_100N
- added U420: 28C256, Package_DIP:DIP-28_W15.24mm_Socket, symbol cpu16:28C256
- added U421, U422, U423, U424: 62256, Package_DIP:DIP-28_W15.24mm, symbol cpu16:62256
- added U425: 74HC138, Package_DIP:DIP-16_W7.62mm, symbol cpu16:74HC138
- added U426, U427: 74HC08, Package_DIP:DIP-14_W7.62mm, symbol cpu16:74HC08
- added U428, U429: 74HC32, Package_DIP:DIP-14_W7.62mm, symbol cpu16:74HC32
- added U430: 74HC00, Package_DIP:DIP-14_W7.62mm, symbol cpu16:74HC00
- added U432, U433, U434: 74HC04, Package_DIP:DIP-14_W7.62mm, symbol cpu16:74HC04
- U403: Gorev bank register seçimi (FF10/11, FF12/13); Flash seçimi (PA19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 -> bank register seçimi (FF10/11, FF12/13)
- U431: renamed from C412; value C_100N -> 74HC02; footprint Capacitor_THT:C_Disc_D5.0mm_W2.5mm_P5.00mm -> Package_DIP:DIP-14_W7.62mm; symbol cpu16:C_100N -> cpu16:74HC02; Gorev U411 dekuplaj -> yapıştırıcı: çift bayt yazma penceresi [2, 6), bellek çiple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
Connections:
- net ~{LOWSEL} is gone; now on net VCC: U403.15 (~{2E})
- net A1: now also U420.9 (A1), U421.9 (A1), U422.9 (A1), U423.9 (A1), U424.9 (A1)
- net A10: now also U420.21 (A10), U421.21 (A10), U422.21 (A10), U423.21 (A10), U424.21 (A10)
- net A11: now also U420.23 (A11), U421.23 (A11), U422.23 (A11), U423.23 (A11), U424.23 (A11)
- net A12: now also U420.2 (A12), U421.2 (A12), U422.2 (A12), U423.2 (A12), U424.2 (A12)
- net A13: now also U420.26 (A13), U421.26 (A13), U422.26 (A13), U423.26 (A13), U424.26 (A13)
- net A2: now also U420.8 (A2), U421.8 (A2), U422.8 (A2), U423.8 (A2), U424.8 (A2)
- net A3: now also U420.7 (A3), U421.7 (A3), U422.7 (A3), U423.7 (A3), U424.7 (A3)
- net A4: now also U420.6 (A4), U421.6 (A4), U422.6 (A4), U423.6 (A4), U424.6 (A4)
- net A5: now also U420.5 (A5), U421.5 (A5), U422.5 (A5), U423.5 (A5), U424.5 (A5)
- net A6: now also U420.4 (A6), U421.4 (A6), U422.4 (A6), U423.4 (A6), U424.4 (A6)
- net A7: now also U420.3 (A7), U421.3 (A7), U422.3 (A7), U423.3 (A7), U424.3 (A7)
- net A8: now also U420.25 (A8), U421.25 (A8), U422.25 (A8), U423.25 (A8), U424.25 (A8)
- net A9: now also U420.24 (A9), U421.24 (A9), U422.24 (A9), U423.24 (A9), U424.24 (A9)
- net BANK0_CP: now also U428.3 (1Y)
- net BANK1_5: now also U432.4 (2Y)
- net BANK1_CP: now also U428.6 (2Y)
- net BANK2_0: now also U432.8 (4Y)
- net BANK2_5: now also U432.12 (6Y)
- net BANK2_CP: now also U428.8 (3Y)
- net BANK3_1: now also U433.4 (2Y)
- net BANK3_5: now also U433.8 (4Y)
- net BANK3_CP: now also U428.11 (4Y)
- net BSEL: now also U420.10 (A0), U421.10 (A0), U422.10 (A0), U423.10 (A0), U424.10 (A0), U426.13 (4B), U426.2 (1B)
- net DE0: now also U432.5 (3A)
- net DE5: now also U432.11 (5A)
- net DO1: now also U433.1 (1A)
- net DO5: now also U432.1 (1A), U433.5 (3A)
- net GND: now also U403.13 (2A1), U403.14 (2A0), U431.11 (4A), U431.12 (4B), U431.7 (GND), U431.8 (3A), U431.9 (3B), C412.2, C433.2, C434.2, C435.2, U420.14 (GND), U421.14 (GND), U422.14 (GND), U423.14 (GND), U424.14 (GND), U425.8 (GND), U426.7 (GND), U427.10 (3B), U427.12 (4A), U427.13 (4B), U427.7 (GND), U427.9 (3A), U428.7 (GND), U429.10 (3B), U429.12 (4A), U429.13 (4B), U429.4 (2A), U429.5 (2B), U429.7 (GND), U429.9 (3A), U430.12 (4A), U430.13 (4B), U430.7 (GND), U432.7 (GND), U433.7 (GND), U434.11 (5A), U434.13 (6A), U434.3 (2A), U434.5 (3A), U434.7 (GND), U434.9 (4A); no longer U431.2
- net MD0: now also U420.11 (IO0), U421.11 (IO0), U422.11 (IO0), U423.11 (IO0), U424.11 (IO0)
- net MD1: now also U420.12 (IO1), U421.12 (IO1), U422.12 (IO1), U423.12 (IO1), U424.12 (IO1)
- net MD2: now also U420.13 (IO2), U421.13 (IO2), U422.13 (IO2), U423.13 (IO2), U424.13 (IO2)
- net MD3: now also U420.15 (IO3), U421.15 (IO3), U422.15 (IO3), U423.15 (IO3), U424.15 (IO3)
- net MD4: now also U420.16 (IO4), U421.16 (IO4), U422.16 (IO4), U423.16 (IO4), U424.16 (IO4)
- net MD5: now also U420.17 (IO5), U421.17 (IO5), U422.17 (IO5), U423.17 (IO5), U424.17 (IO5)
- net MD6: now also U420.18 (IO6), U421.18 (IO6), U422.18 (IO6), U423.18 (IO6), U424.18 (IO6)
- net MD7: now also U420.19 (IO7), U421.19 (IO7), U422.19 (IO7), U423.19 (IO7), U424.19 (IO7)
- net M_EWIN: now also U431.1 (1Y), U426.10 (3B)
- net M_EWR: now also U431.5 (2A), U426.8 (3Y)
- net M_LCP: now also U427.6 (2Y)
- net M_MRD: now also U429.1 (1A), U430.2 (1B), U434.2 (1Y)
- net M_OWIN: now also U426.11 (4Y), U427.1 (1A)
- net M_OWR: now also U431.6 (2B), U427.3 (1Y)
- net M_SA: now also U431.3 (1B), U426.1 (1A)
- net M_SODD: now also U426.3 (1Y), U430.1 (1A), U430.9 (3A)
- net M_WAITING: now also U433.10 (5Y)
- net M_WEL_E: now also U426.4 (2A)
- net M_WEL_O: now also U427.2 (1B), U429.2 (1B)
- net M_WEM: now also U426.6 (2Y), U426.9 (3A), U430.4 (2A)
- net PA14: now also U420.1 (A14), U421.1 (A14), U422.1 (A14), U423.1 (A14), U424.1 (A14)
- net PA15: now also U425.1 (A0)
- net PA16: now also U425.2 (A1)
- net PA17: now also U425.4 (~{E1}); no longer U403.14 (2A0)
- net PA18: now also U425.5 (~{E2}); no longer U403.13 (2A1)
- net PA19: now also U425.3 (A2)
- net TCLK: now also U431.2 (1A), U426.12 (4A), U427.4 (2A), U433.13 (6A)
- net VCC: now also U431.14 (VCC), C412.1, C433.1, C434.1, C435.1, U420.28 (VCC), U421.28 (VCC), U422.28 (VCC), U423.28 (VCC), U424.28 (VCC), U425.16 (VCC), U426.14 (VCC), U427.14 (VCC), U428.14 (VCC), U429.14 (VCC), U430.14 (VCC), U432.14 (VCC), U433.14 (VCC), U434.14 (VCC); no longer U431.1
- net ~{BANK1_5}: now also U432.3 (2A)
- net ~{BANK1_D5}: now also U432.2 (1Y)
- net ~{BANK2_0}: now also U432.9 (4A)
- net ~{BANK2_5}: now also U432.13 (6A)
- net ~{BANK2_D0}: now also U432.6 (3Y)
- net ~{BANK2_D5}: now also U432.10 (5Y)
- net ~{BANK3_1}: now also U433.3 (2A)
- net ~{BANK3_5}: now also U433.9 (4A)
- net ~{BANK3_D1}: now also U433.2 (1Y)
- net ~{BANK3_D5}: now also U433.6 (3Y)
- net ~{BSEL01}: now also U428.2 (1B), U428.5 (2B)
- net ~{BSEL23}: now also U428.10 (3B), U428.13 (4B)
- net ~{BSEL}: now also U427.5 (2B), U430.5 (2B)
- net ~{IO}: now also U425.6 (E3), U426.5 (2B)
- net ~{MRD}: now also U420.22 (~{OE}), U421.22 (~{OE}), U422.22 (~{OE}), U423.22 (~{OE}), U424.22 (~{OE}), U434.1 (1A)
- net ~{MWE_E}: now also U428.1 (1A), U428.9 (3A)
- net ~{MWE_O}: now also U428.12 (4A), U428.4 (2A)
- net ~{MWR}: now also U431.4 (2Y), U420.27 (~{WE}), U421.27 (~{WE}), U422.27 (~{WE}), U423.27 (~{WE}), U424.27 (~{WE})
- net ~{M_EVEN_OE}: now also U430.6 (2Y)
- net ~{M_ODD_OE}: now also U430.8 (3Y)
- net ~{M_RDDRV}: now also U430.3 (1Y)
- net ~{M_TCLK}: now also U433.12 (6Y)
- net ~{WAIT}: now also U433.11 (5A)
- net ~{CE_FLASH}: no longer names the net of U403.12 (~{2Y0})
- new net N2098: U429.3 (1Y), U430.10 (3B)
- new net ~{CE_RAM0}: U421.20 (~{CE}), U425.11 (~{Y4})
- new net ~{CE_RAM1}: U422.20 (~{CE}), U425.10 (~{Y5})
- new net ~{CE_RAM2}: U423.20 (~{CE}), U425.9 (~{Y6})
- new net ~{CE_RAM3}: U424.20 (~{CE}), U425.7 (~{Y7})
- new net ~{CE_ROM}: U420.20 (~{CE}), U425.15 (~{Y0})
- no-connect marks 37 -> 38
Other:
- title: CPU16 — Bellek kartı (Flash 128 KB + RAM 512 KB, bank register'ları) -> CPU16 — Bellek kartı (EEPROM 32 KB + RAM 128 KB, bank register'ları)
- moved on the sheet: U405, U406, U407, U408, U409, U410, U411, U412, U413, U414, U415, U416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
