File: cpu16/kicad/gc/gc.kicad_sch (KiCad schematic)
At the start: 137 parts, among them J601 CONN_CH340, J602 CONN_PS2, J603 BACKPLANE_2x32, U601 74HC138, U602 74HC138, U603 74HC138, U604 74HC138, U605 74HC74, U606 74HC14, U607 74HC165, U608 74HC161, U609 74HC161, U610 74HC161, U611 74HC74, U612 74HC74, U613 74HC161, U614 74HC161, U615 74HC161, U616 74HC595, U617 74HC161, U618 74HC595, U619 74HC05, U620 74HC161, U621 74HC161, U622 74HC161, U623 74HC574, U624 74HC574, U625 74HC541, U626 74HC541, U627 74HC175, U628 74HC541, U629 74HC541, U630 74HC74, U631 74HC74, U632 74HC193, U633 74HC193, U634 74HC193, U635 74HC193, U636 74HC688, U637 74HC688, U638 74HC175, U639 74HC148, U640 74HC541, U641 74HC541, U642 74HC541, U643 74HC541, U644 74HC541, U645 74HC74, U646 74HC08, U647 74HC08, U648 74HC08, U649 74HC08, U650 74HC08, U651 74HC08, U652 74HC08, U653 74HC08, U654 74HC32, U655 74HC32, U656 74HC32, U657 74HC32, U658 74HC00, U659 74HC00, U660 74HC00, U661 74HC02, U662 74HC02, U663 74HC04, U664 74HC04, U665 74HC04

Commit message: Kontrol birimi: mikrokod ve ALU ROM'ları yerine 74HC kapı devresi
CPU kartındaki 7 SST39SF010A (4 mikrokod, 3 ALU kod çözme ROM'u) kalktı. Yerine
board/kontrol.ts, cpu16.ucode'dan (tek kaynak) ve aluControl tablosundan çok seviyeli
bir 74HC devresi üretir ve Board API ile gerçek çipler olarak yerleştirir:

- Mikrokod: adım ve komut çözücüleri (74HC138; INT = 1 iken komutlar pasif, f3'e göre
  dallanan komutlara alt çözücü), aynı mikro programı çalıştıran (op, f3, COND)
  atomları, ortak alt kümeli VEYA ağı, sık kullanılan bitler için adım seçici
  (74HC151), adım 8..15 için SWI hattıyla açılan çözücü.
- ALU kod çözme: işlem çözücüleri (3 × 74HC138), işlem bitleri, h ve C terimleri.
- Yeni kapı çipleri: 74HC11, 74HC20, 74HC21, 74HC27, 74HC30 (veri sayfası pin sırası,
  doğruluk tablosu, zamanlama modeli, KiCad sembolü).
- Board: esnek yapıştırıcı kapılar (kartın diğer kapılarından sonra paketlenir, son
  çipi az dolu türü başka türlerin boş birimlerine taşır) ve defer(). Çözücüler eski
  ROM'ların yuvalarına (U1, U3, U5, U7, U10, U68–U71) oturur: kartın diğer bütün
  çiplerinin referansları değişmedi.
- CPU kartı 146 → 194 entegre; en kötü durumda CPU saati 860 → 824 ns (1,21 MHz),
  tipik 470 → 369 ns.
- Denklik testi (tests/kontrol.test.ts): kontrol birimi tek başına bir kartta, gerçek
  çip modelleriyle (LogicSim) 8192 mikrokod adresinin ve 128 ALU adresinin hepsinde
  tabloyla aynı kelimeyi verir.
- roms.ts, cpu16/roms/ ve "roms" komutu kalktı; "kontrol" komutu gömülü mikrokodu
  (micro/cpu16-ucode.ts) yeniler ve devreyi denetler. GateComputer ve GateMachine artık
  mikrokod istemez.
- CPU şeması A0'a sığsın diye dekuplaj kondansatörleri dar sütunlarda; KiCad dosyaları,
  BOM ve deney rehberlerinin otomatik bölümleri yeniden üretildi.

Co-Authored-By: Claude Opus 5.5 (1M context) <noreply@anthropic.com>
Claude-Session: https://claude.ai/code/session_018J8WVuECVRbQJyCbmF6Nsi
Connections:
- net N2804 is gone; now on net N2999: U646.11 (4Y), U654.2 (1B)
- net N2999: no longer U650.11 (4Y), U651.1 (1A)
- net N2650 renamed N2845
- net N2803 renamed N2998
- net N2807 renamed N3002
- net N2808 renamed N3003
- net N2810 renamed N3005
- net N2814 renamed N3009
- net N2815 renamed N3010
- net N2817 renamed N3012
- net N2827 renamed N3022
- net N2829 renamed N3024
- net N2924 renamed N3119
- net N2925 renamed N3120
- net N2994 renamed N3189
- net N2997 renamed N3192
- net N3000 renamed N3195
- net N3197 renamed N3392
- net N3198 renamed N3393
- net N3211 renamed N3406
- net N3212 renamed N3407
- new net N3194: U650.11 (4Y), U651.1 (1A)
