File: cpu16/kicad/gc/gc.kicad_sch (KiCad schematic)
At the start: 137 parts, among them J601 CONN_CH340, J602 CONN_PS2, J603 BACKPLANE_2x32, U601 74HC138, U602 74HC138, U603 74HC138, U604 74HC138, U605 74HC74, U606 74HC14, U607 74HC165, U608 74HC161, U609 74HC161, U610 74HC161, U611 74HC74, U612 74HC74, U613 74HC161, U614 74HC161, U615 74HC161, U616 74HC595, U617 74HC161, U618 74HC595, U619 74HC05, U620 74HC161, U621 74HC161, U622 74HC161, U623 74HC574, U624 74HC574, U625 74HC541, U626 74HC541, U627 74HC175, U628 74HC541, U629 74HC541, U630 74HC74, U631 74HC74, U632 74HC193, U633 74HC193, U634 74HC193, U635 74HC193, U636 74HC688, U637 74HC688, U638 74HC175, U639 74HC148, U640 74HC541, U641 74HC541, U642 74HC541, U643 74HC541, U644 74HC541, U645 74HC74, U646 74HC08, U647 74HC08, U648 74HC08, U649 74HC08, U650 74HC08, U651 74HC08, U652 74HC08, U653 74HC08, U654 74HC32, U655 74HC32, U656 74HC32, U657 74HC32, U658 74HC00, U659 74HC00, U660 74HC00, U661 74HC02, U662 74HC02, U663 74HC04, U664 74HC04, U665 74HC04

Commit message: Anakart yalnız yaygın parçalarla: 28C256 + 4 × 62256, kendin yap bellek kartı
AFU kararı: bilgisayar yalnız yaygın 7400 serisi lojikle ve iki bellek
çipiyle (62256, 28C256) kurulur.

Bellek kartı (31 → 34 entegre):
- SST39SF010A yerine 28C256 (32 KB, fiziksel 0x00000–0x07FFF, bank 0–1)
- AS6C4008 yerine 4 × 62256 (128 KB, 0x80000–0x9FFFF, bank 32–39)
- çip seçimi tek 74HC138; geri kalan bölgeler boş (0xFF, yazma yok sayılır)

Nadir parçalar çıktı:
- önbellek sayaçları 74HC590 → 74HC161 × 8 + 74HC541 × 4 (37 → 46)
- zamanlayıcı 74HC193 → 74HC161 (tümleyeni yukarı sayar)
- kesme öncelik kodlayıcısı 74HC148 → kapılar
- video adres sayacı (VADDR) 74HC193 → 74HC161 × 4 + yükleme bayrakları
- karakter ROM'u 28C256; yavaşlığı font register'ıyla bir aşamalık boru
  hattında karşılanır (V_H2 en kötü 262 ns, font yolu 199 ns ≤ 317,8);
  resim Machine ile aynı (video 69 → 73 entegre)
- 74HC166 kalır: 74HC165'in eşzamansız yüklemesi piksel saatine sığmaz

Kendin yap bellek kartı (kyb, 22 entegre): FF40–FF4F, 16 bayt, her bayt
bir 74HC574; 74HC138 çözücüler ve 74HC245 veri yolu tamponları. Machine
aygıtı, KiCad klasörü, kapı seviyesi kart Machine ile döngü döngüsüne aynı.

Machine'de At28c256 modeli (sayfa yazma, tBLC, yazma döngüsü, DATA
yoklaması, toggle biti, SDP); kapı seviyesi kartlar aynı modeli kullanır.
BIOS: F komutu korumalı sayfa yazmasıyla yalnız bank 1'e, I komutu yazma
korumasını gösterir, T bank 32–39'u sınar. Deney 8 programı 8 bank sayar,
boş bölgeleri denetler; Deney 14 programı ve testi eklendi.

Co-Authored-By: Claude Opus 5.5 (1M context) <noreply@anthropic.com>
Claude-Session: https://claude.ai/code/session_018J8WVuECVRbQJyCbmF6Nsi
Parts:
- removed U631, U645: 74HC74, Package_DIP:DIP-14_W7.62mm, symbol cpu16:74HC74
- removed U632, U633, U634, U635: 74HC193, Package_DIP:DIP-16_W7.62mm, symbol cpu16:74HC193
- removed U637: 74HC688, Package_DIP:DIP-20_W7.62mm, symbol cpu16:74HC688
- removed U638: 74HC175, Package_DIP:DIP-16_W7.62mm, symbol cpu16:74HC175
- removed U639: 74HC148, Package_DIP:DIP-16_W7.62mm, symbol cpu16:74HC148
- removed U643, U644: 74HC541, Package_DIP:DIP-20_W7.62mm, symbol cpu16:74HC541
- removed U652, U653: 74HC08, Package_DIP:DIP-14_W7.62mm, symbol cpu16:74HC08
- removed U657: 74HC32, Package_DIP:DIP-14_W7.62mm, symbol cpu16:74HC32
- removed U659, U660: 74HC00, Package_DIP:DIP-14_W7.62mm, symbol cpu16:74HC00
- removed U661, U662: 74HC02, Package_DIP:DIP-14_W7.62mm, symbol cpu16:74HC02
- added U631, U632, U633, U634: 74HC161, Package_DIP:DIP-16_W7.62mm, symbol cpu16:74HC161
- added U635: 74HC688, Package_DIP:DIP-20_W7.62mm, symbol cpu16:74HC688
- added U637: 74HC175, Package_DIP:DIP-16_W7.62mm, symbol cpu16:74HC175
- added U638, U639: 74HC541, Package_DIP:DIP-20_W7.62mm, symbol cpu16:74HC541
- added U643: 74HC74, Package_DIP:DIP-14_W7.62mm, symbol cpu16:74HC74
- added U644, U645: 74HC08, Package_DIP:DIP-14_W7.62mm, symbol cpu16:74HC08
- added U652, U653: 74HC32, Package_DIP:DIP-14_W7.62mm, symbol cpu16:74HC32
- added U657: 74HC00, Package_DIP:DIP-14_W7.62mm, symbol cpu16:74HC00
- added U659, U660: 74HC02, Package_DIP:DIP-14_W7.62mm, symbol cpu16:74HC02
- added U661, U662: 74HC04, Package_DIP:DIP-14_W7.62mm, symbol cpu16:74HC04
- U630: Gorev yeniden yükleme isteği, EXPIRED (FF07) -> EXPIRED (FF07); resetten sonraki ilk TCLK kenarı
- U636: Gorev sayaç = 1 algılama (düşük bayt = 01) -> c = 1 algılama: u yüksek bayt = FF
- U640: Gorev IRQ_SRC okuma (istek yoksa sürülmez: 0xFF) -> IRQ_MASK okuma
- U641: Gorev IRQ_PEND okuma -> UART_STAT okuma (RX_READY, TX_EMPTY)
- U642: Gorev IRQ_MASK okuma -> KBD_STAT okuma (READY)
- U646: Gorev yapıştırıcı: KBD_DATA okunuyor (READY iken: çerçeve ortasın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 -> yapıştırıcı: bitiş biti bitti, BUSY sonraki değer
- U647: Gorev yapıştırıcı: bit sonu -> yapıştırıcı: örnek anı (bölücü 34), bitiş biti örneği, bayt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
- U648: Gorev yapıştırıcı: bitiş biti bitti, BUSY sonraki değer -> yapıştırıcı: RX_READY sil: UART_DATA okundu, 9 bit alındı: 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
- U649: Gorev yapıştırıcı: örnek anı (bölücü 34), bitiş biti örneği, bayt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 -> yapıştırıcı: sayaç = 10: sonraki kenar bitiş biti, KBD_DATA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
- U650: Gorev yapıştırıcı: RX_READY sil: UART_DATA okundu, 9 bit alındı: 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 -> yapıştırıcı: sayaç yükleme (aktif düşük), TIMER_STAT'a 1 ya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
- U651: Gorev yapıştırıcı: sayaç = 10: sonraki kenar bitiş biti, KBD_DATA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 -> yapıştırıcı: kaynak 1 maskeli, kaynak 2 maskeli, kaynak 3 m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
- U654: Gorev yapıştırıcı: bit ≥ 7: kısa bit (34 döngü), bölücü 33 / 34 a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 -> yapıştırıcı: çıkış register'ı saati (örnek 9), kaydırma saa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
- U655: Gorev yapıştırıcı: başlangıç biti değil, TX hattı: boşta 1, başla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 -> yapıştırıcı: EXPIRED kur / tut, kaynak 0 ya da 1, kaynak 2 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
- U656: Gorev yapıştırıcı: çıkış register'ı saati (örnek 9), kaydırma saa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 -> yapıştırıcı: IRQ_SRC bit 1: kaynak 3 ya da 2, IRQ_SRC bit 0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
- U658: Gorev yapıştırıcı: veri bitleri arasında kaydır, sayaç = 9, azalt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 -> yapıştırıcı lojik
- U663: Gorev yapıştırıcı: reset (aktif yüksek), TCLK tersi, uzun bit (35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 -> yapıştırıcı: RELOAD bit 2 tersi, RELOAD bit 3 tersi, RELOAD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
- U664: Gorev yapıştırıcı: sayaç biti 1 tersi, sayaç ≠ 1 -> yapıştırıcı: RELOAD bit 8 tersi, RELOAD bit 9 tersi, RELOAD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
- U665: Gorev yapıştırıcı: IRQ hattı = OR(bekleyen ∧ maske) -> yapıştırıcı: RELOAD bit 14 tersi, RELOAD bit 15 tersi, iste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
Connections:
- net GC_DECP is gone; now on net GND: U658.12 (4A)
- net GC_TRL is gone; now on net GC_EXPIRED: U630.5 (1Q)
- net N2650 is gone; now on net GC_TXEND: U646.1 (1A)
- net ~{GC_SA0} is gone; now on net GC_R15: U665.3 (2A)
- net ~{GC_SA1} is gone; now on net IRQ: U665.5 (3A)
- net A0: now also U659.3 (1B), U659.6 (2B)
- net DE0: now also U638.18 (Y0), U639.18 (Y0); no longer U640.18 (Y0), U641.18 (Y0), U651.10 (3B)
- net DE1: now also U638.17 (Y1), U639.17 (Y1); no longer U640.17 (Y1), U641.17 (Y1)
- net DE2: now also U638.16 (Y2), U639.16 (Y2); no longer U640.16 (Y2), U641.16 (Y2)
- net DE3: now also U638.15 (Y3), U639.15 (Y3); no longer U640.15 (Y3), U641.15 (Y3)
- net DE4: now also U638.14 (Y4), U639.14 (Y4); no longer U640.14 (Y4), U641.14 (Y4)
- net DE5: now also U638.13 (Y5), U639.13 (Y5); no longer U640.13 (Y5), U641.13 (Y5)
- net DE6: now also U638.12 (Y6), U639.12 (Y6); no longer U640.12 (Y6), U641.12 (Y6)
- net DE7: now also U638.11 (Y7), U639.11 (Y7); no longer U640.11 (Y7), U641.11 (Y7)
- net DO0: now also U640.18 (Y0), U641.18 (Y0), U658.2 (1B), U637.4 (D0)
- net DO1: now also U640.17 (Y1), U641.17 (Y1), U637.5 (D1)
- net DO2: now also U640.16 (Y2), U641.16 (Y2), U637.12 (D2)
- net DO3: now also U640.15 (Y3), U641.15 (Y3), U637.13 (D3)
- net DO4: now also U640.14 (Y4), U641.14 (Y4)
- net DO5: now also U640.13 (Y5), U641.13 (Y5)
- net DO6: now also U640.12 (Y6), U641.12 (Y6)
- net DO7: now also U640.11 (Y7), U641.11 (Y7)
- net GC_EXPIRED: now also U650.9 (3A), U655.2 (1B); no longer U630.9 (2Q)
- net GC_EXP_D: now also U630.2 (1D), U655.3 (1Y); no longer U630.12 (2D)
- net GC_KB0: now also U648.10 (3B), U654.4 (2A), U662.5 (3A); no longer U650.10 (3B), U656.4 (2A), U664.5 (3A)
- net GC_KB1: now also U648.13 (4B), U654.5 (2B), U662.3 (2A); no longer U650.13 (4B), U656.5 (2B), U664.3 (2A)
- net GC_KB3: now also U648.12 (4A), U648.4 (2A), U648.9 (3A); no longer U650.12 (4A), U650.4 (2A), U650.9 (3A)
- net GC_KCLKN: now also U654.12 (4A), U654.9 (3A), U643.11 (2CLK); no longer U656.12 (4A), U656.9 (3A)
- net GC_KEQ10: now also U649.3 (1Y), U643.12 (2D); no longer U651.3 (1Y)
- net GC_KGE9: now also U648.6 (2Y), U654.10 (3B); no longer U650.6 (2Y), U656.10 (3B)
- net GC_KRDY: now also U642.2 (A0), U651.1 (1A), U639.3 (A1), U643.9 (2Q), U644.2 (1B); no longer U641.3 (A1), U646.2 (1B)
- net GC_KSHCP: now also U654.8 (3Y); no longer U656.8 (3Y)
- net GC_KSTCP: now also U654.11 (4Y); no longer U656.11 (4Y)
- net GC_M0: now also U640.2 (A0), U650.13 (4B), U637.2 (Q0); no longer U642.2 (A0)
- net GC_M1: now also U640.3 (A1), U651.2 (1B), U637.7 (Q1); no longer U642.3 (A1)
- net GC_M2: now also U640.4 (A2), U651.5 (2B), U637.10 (Q2); no longer U642.4 (A2)
- net GC_M3: now also U640.5 (A3), U651.10 (3B), U637.15 (Q3); no longer U642.5 (A3)
- net GC_P0: now also U650.12 (4A), U650.8 (3Y), U639.2 (A0); no longer U641.2 (A0)
- net GC_R0: now also U662.11 (5A)
- net GC_R1: now also U662.13 (6A)
- net GC_R10: now also U664.5 (3A)
- net GC_R11: now also U664.9 (4A)
- net GC_R12: now also U664.11 (5A)
- net GC_R13: now also U664.13 (6A)
- net GC_R14: now also U665.1 (1A)
- net GC_R2: now also U663.1 (1A)
- net GC_R3: now also U663.3 (2A)
- net GC_R4: now also U663.5 (3A)
- net GC_R5: now also U663.9 (4A)
- net GC_R6: now also U663.11 (5A)
- net GC_R7: now also U663.13 (6A)
- net GC_R8: now also U664.1 (1A)
- net GC_R9: now also U664.3 (2A)
- net GC_RB0: now also U647.10 (3B); no longer U649.10 (3B)
- net GC_RB3: now also U647.9 (3A); no longer U649.9 (3A)
- net GC_RB9: now also U647.13 (4B), U647.8 (3Y), U662.1 (1A); no longer U649.13 (4B), U649.8 (3Y), U664.1 (1A)
- net GC_RDK: now also U644.3 (1Y); no longer U646.3 (1Y)
- net GC_RDU: now also U659.1 (1Y)
- net GC_RLD: now also U649.11 (4Y), U655.1 (1A); no longer U630.2 (1D)
- net GC_RSTD: now also U630.9 (2Q), U659.12 (4B)
- net GC_RXBUSY: now also U646.12 (4A); no longer U648.12 (4A)
- net GC_RXBUSY_D: now also U653.8 (3Y); no longer U655.8 (3Y)
- net GC_RXD1: now also U647.5 (2B); no longer U649.5 (2B)
- net GC_RXD5: now also U647.4 (2A); no longer U649.4 (2A)
- net GC_RXDONE: now also U647.11 (4Y), U661.13 (6A); no longer U649.11 (4Y), U663.13 (6A)
- net GC_RXEND: now also U647.12 (4A), U647.6 (2Y), U657.4 (2A), U659.8 (3A); no longer U649.12 (4A), U649.6 (2Y), U658.4 (2A)
- net GC_RXRDY: now also U641.2 (A0), U651.4 (2A), U639.4 (A2), U643.5 (1Q); no longer U641.4 (A2)
- net GC_RXSHCP: now also U653.11 (4Y); no longer U655.11 (4Y)
- net GC_RXSTCP: now also U654.3 (1Y), U643.3 (1CLK); no longer U656.3 (1Y)
- net GC_SA0: now also U656.6 (2Y), U638.2 (A0); no longer U640.2 (A0), U665.4 (2Y)
- net GC_SA1: now also U656.3 (1Y), U638.3 (A1); no longer U640.3 (A1), U665.6 (3Y)
- net GC_TB0: now also U644.10 (3B), U645.13 (4B), U652.9 (3A); no longer U646.10 (3B), U647.13 (4B), U654.9 (3A)
- net GC_TB1: now also U644.9 (3A), U652.10 (3B); no longer U646.9 (3A), U654.10 (3B)
- net GC_TB2: now also U644.12 (4A), U652.12 (4A); no longer U646.12 (4A), U654.12 (4A)
- net GC_TB3: now also U645.12 (4A), U652.1 (1A), U652.13 (4B); no longer U647.12 (4A), U654.1 (1A), U654.13 (4B)
- net GC_TBNZ: now also U646.9 (3A), U653.3 (1Y), U657.2 (1B); no longer U648.9 (3A), U655.3 (1Y), U658.2 (1B)
- net GC_TD0: now also U645.2 (1B); no longer U647.2 (1B)
- net GC_TD1: now also U645.5 (2B); no longer U647.5 (2B)
- net GC_TD5: now also U645.9 (3A); no longer U647.9 (3A)
- net GC_TEN: now also U649.10 (3B), U650.1 (1A)
- net GC_TICKP: now also U649.9 (3A), U659.11 (4A)
- net GC_TIRQEN: now also U650.10 (3B)
- net GC_TTICK: now also U649.12 (4A), U649.8 (3Y), U631.7 (CEP), U632.7 (CEP), U633.7 (CEP), U634.7 (CEP), U657.12 (4A)
- net GC_TXBUSY: now also U644.4 (2A); no longer U648.4 (2A)
- net GC_TXBUSY_D: now also U646.6 (2Y); no longer U648.6 (2Y)
- net GC_TXDONE: now also U646.3 (1Y), U661.11 (5A); no longer U648.3 (1Y), U663.11 (5A)
- net GC_TXEMPTY: now also U641.3 (A1), U653.4 (2A); no longer U655.4 (2A)
- net GC_TXEND: now also U645.8 (3Y), U657.1 (1A), U661.9 (4A); no longer U647.8 (3Y), U648.1 (1A), U658.1 (1A), U663.9 (4A)
- net GC_TXLOW: now also U645.10 (3B), U652.6 (2Y); no longer U647.10 (3B), U654.6 (2Y)
- net GC_TXQ: now also U646.10 (3B); no longer U648.10 (3B)
- net GC_TXRUN: now also U644.6 (2Y); no longer U646.6 (2Y)
- net GC_TXS: now also U645.1 (1A), U652.3 (1Y), U661.5 (3A); no longer U647.1 (1A), U654.3 (1Y), U663.5 (3A)
- net GC_Z1: now also U649.13 (4B), U657.13 (4B), U660.1 (1Y); no longer U664.13 (6A)
- net GND: now also U630.12 (2D), U640.19 (~{OE2}), U641.4 (A2), U641.5 (A3), U642.3 (A1), U642.4 (A2), U642.5 (A3), U656.10 (3B), U656.12 (4A), U656.13 (4B), U656.9 (3A), U658.10 (3B), U658.13 (4B), U658.4 (2A), U658.5 (2B), U658.9 (3A), U631.8 (GND), U632.8 (GND), U633.8 (GND), U634.8 (GND), U635.1 (~{E}), U635.10 (GND), U635.3 (Q0), U637.8 (GND), U638.10 (GND), U638.4 (A2), U638.5 (A3), U638.6 (A4), U638.7 (A5), U638.8 (A6), U638.9 (A7), U639.10 (GND), U639.19 (~{OE2}), U639.6 (A4), U639.7 (A5), U639.8 (A6), U639.9 (A7), U643.7 (GND), U644.7 (GND), U645.7 (GND), U652.7 (GND), U653.7 (GND), U657.7 (GND), U659.7 (GND), U660.11 (4A), U660.12 (4B), U660.5 (2A), U660.6 (2B), U660.7 (GND), U660.8 (3A), U660.9 (3B), U661.7 (GND), U662.7 (GND); no longer U636.12 (Q4), U636.14 (Q5), U636.16 (Q6), U636.18 (Q7), U636.5 (Q1), U636.7 (Q2), U636.9 (Q3), U640.4 (A2), U640.5 (A3), U665.9 (4A)
- net IRQ: now also U655.11 (4Y); no longer U665.2 (1Y)
- net TCLK: now also U654.1 (1A), U631.2 (CP), U632.2 (CP), U633.2 (CP), U634.2 (CP), U653.12 (4A), U661.3 (2A); no longer U655.12 (4A), U656.1 (1A), U663.3 (2A)
- net UART_TXD: now also U653.6 (2Y); no longer U655.6 (2Y)
- net VCC: now also U630.13 (~{2CLR}), U636.12 (Q4), U636.14 (Q5), U636.16 (Q6), U636.18 (Q7), U636.5 (Q1), U636.7 (Q2), U636.9 (Q3), U631.10 (CET), U631.16 (VCC), U632.16 (VCC), U633.16 (VCC), U634.16 (VCC), U635.12 (Q4), U635.14 (Q5), U635.16 (Q6), U635.18 (Q7), U635.20 (VCC), U635.5 (Q1), U635.7 (Q2), U635.9 (Q3), U637.16 (VCC), U638.20 (VCC), U639.20 (VCC), U643.10 (~{2PRE}), U643.14 (VCC), U643.2 (1D), U643.4 (~{1PRE}), U644.14 (VCC), U645.14 (VCC), U652.14 (VCC), U653.14 (VCC), U657.14 (VCC), U659.14 (VCC), U660.14 (VCC), U661.14 (VCC), U662.14 (VCC); no longer U630.10 (~{2PRE})
- net VSYNC_REQ: now also U651.9 (3A), U639.5 (A3); no longer U641.5 (A3)
- net ~{GC_EXPCLR}: now also U630.1 (~{1CLR}), U650.6 (2Y); no longer U630.13 (~{2CLR})
- net ~{GC_GS}: now also U665.6 (3Y), U638.19 (~{OE2}); no longer U640.19 (~{OE2}), U665.1 (1A)
- net ~{GC_I2}: now also U651.13 (4B), U665.8 (4Y)
- net ~{GC_KB1}: now also U657.10 (3B), U662.4 (2Y); no longer U658.10 (3B), U664.4 (2Y)
- net ~{GC_KCLR}: now also U649.6 (2Y), U643.13 (~{2CLR}); no longer U651.6 (2Y)
- net ~{GC_KEQ9}: now also U654.13 (4B), U657.8 (3Y); no longer U656.13 (4B), U658.8 (3Y)
- net ~{GC_PLD}: now also U659.13 (4Y)
- net ~{GC_RD0}: now also U641.1 (~{OE1}), U659.2 (1A)
- net ~{GC_RD1}: now also U642.1 (~{OE1}), U659.5 (2A)
- net ~{GC_RD4}: now also U640.1 (~{OE1}), U639.1 (~{OE1}); no longer U641.1 (~{OE1}), U642.1 (~{OE1})
- net ~{GC_RD5}: now also U638.1 (~{OE1}); no longer U640.1 (~{OE1})
- net ~{GC_RDK_Q}: now also U649.5 (2B); no longer U651.5 (2B)
- net ~{GC_RDU_Q}: now also U648.2 (1B); no longer U650.2 (1B)
- net ~{GC_RXBUSY}: now also U647.1 (1A), U659.9 (3B); no longer U649.1 (1A)
- net ~{GC_RXCLR}: now also U648.3 (1Y), U643.1 (~{1CLR}); no longer U650.3 (1Y)
- net ~{GC_RXDONE}: now also U646.13 (4B), U654.2 (1B), U661.12 (6Y); no longer U648.13 (4B), U656.2 (1B), U663.12 (6Y)
- net ~{GC_RXLD}: now also U659.10 (3Y)
- net ~{GC_RXS2}: now also U647.2 (1B); no longer U649.2 (1B)
- net ~{GC_TXDONE}: now also U646.5 (2B), U661.10 (5Y); no longer U648.5 (2B), U663.10 (5Y)
- net ~{GC_TXEND}: now also U661.8 (4Y); no longer U663.8 (4Y)
- net ~{GC_TXSH}: now also U657.3 (1Y); no longer U658.3 (1Y)
- net ~{GC_TXS}: now also U645.4 (2A), U661.6 (3Y); no longer U647.4 (2A), U663.6 (3Y)
- net ~{GC_WE0}: now also U644.5 (2B); no longer U646.5 (2B)
- net ~{GC_WE3}: no longer U664.9 (4A)
- net ~{GC_WO3}: now also U662.9 (4A); no longer U664.11 (5A)
- net ~{GC_WO4}: now also U637.9 (CP)
- net ~{GC_Z1H}: now also U636.19 (~{EQ}), U660.3 (1B)
- net ~{GC_Z1L}: now also U635.19 (~{EQ}), U660.2 (1A); no longer U636.19 (~{EQ})
- net ~{RESET}: now also U630.10 (~{2PRE}), U648.1 (1A), U649.4 (2A), U650.4 (2A), U631.1 (~{MR}), U632.1 (~{MR}), U633.1 (~{MR}), U634.1 (~{MR}), U637.1 (~{MR}), U661.1 (1A); no longer U630.1 (~{1CLR}), U650.1 (1A), U651.4 (2A), U663.1 (1A)
- net GC_C0 renamed GC_U8
- net GC_U8: now also U633.14 (Q0)
- net GC_C1 renamed GC_U9
- net GC_U9: now also U633.13 (Q1)
- net GC_C2 renamed GC_U10
- net GC_U10: now also U633.12 (Q2)
- net GC_C3 renamed GC_U11
- net GC_U11: now also U633.11 (Q3)
- net GC_C4 renamed GC_U12
- net GC_U12: now also U634.14 (Q0)
- net GC_C5 renamed GC_U13
- net GC_U13: now also U634.13 (Q1)
- net GC_C6 renamed GC_U14
- net GC_U14: now also U634.12 (Q2)
- net GC_C7 renamed GC_U15
- net GC_U15: now also U634.11 (Q3)
- net GC_RST renamed ~{GC_R2}
- net ~{GC_R2}: now also U631.5 (D2)
- net GC_TCLKN renamed ~{GC_R3}
- net ~{GC_R3}: now also U631.6 (D3); no longer U658.13 (4B)
- net GC_TDCLK: no longer names the net of U658.11 (4Y)
- net GC_TLDEN renamed N3437
- net N3437: now also U656.5 (2B)
- net N2803 renamed N2871
- net N2871: now also U653.5 (2B); no longer U646.13 (4B)
- net N2804 renamed N2881
- net N2881: now also U653.9 (3A); no longer U654.2 (1B)
- net N2807 renamed N2883
- net N2883: now also U653.10 (3B); no longer U654.4 (2A)
- removed net N2808: U647.6 (2Y), U654.5 (2B)
- removed net N2810: U647.11 (4Y), U648.2 (1B)
- removed net N2814: U654.8 (3Y), U655.1 (1A)
- removed net N2815: U654.11 (4Y), U655.2 (1B)
- net N2817 renamed GC_I1
- net GC_I1: now also U651.12 (4A), U651.3 (1Y); no longer U648.8 (3Y)
- net N2827 renamed GC_I2
- net GC_I2: now also U651.6 (2Y), U656.2 (1B), U665.9 (4A); no longer U648.11 (4Y)
- net N2829 renamed GC_I3
- net GC_I3: now also U651.8 (3Y), U656.1 (1A), U656.4 (2A); no longer U649.3 (1Y)
- net N2924 renamed ~{GC_R8}
- net ~{GC_R8}: now also U633.3 (D0); no longer U658.5 (2B)
- net N2925: no longer names the net of U658.6 (2Y)
- net N2925: no longer U655.13 (4B)
- net N2994 renamed N3258
- net N3258: now also U658.3 (1Y); no longer U656.6 (2Y)
- removed net N2997: U650.8 (3Y), U658.9 (3A)
- net N2999 renamed GC_I0
- net GC_I0: now also U655.4 (2A); no longer U651.1 (1A)
- net N3000 renamed ~{GC_R10}
- net ~{GC_R10}: now also U633.5 (D2); no longer U651.2 (1B)
- net N3197 renamed ~{GC_R11}
- net ~{GC_R11}: now also U633.6 (D3); no longer U651.9 (3A)
- removed net N3198: U651.12 (4A), U651.8 (3Y)
- net N3211 renamed ~{GC_R12}
- net ~{GC_R12}: now also U634.3 (D0)
- net ~{GC_TEN}: no longer names the net of U627.3 (~{Q0})
- net ~{GC_TEN}: no longer U651.13 (4B)
- net ~{GC_Z1} renamed ~{GC_R13}
- net ~{GC_R13}: now also U634.4 (D1)
- new net GC_U0: U631.14 (Q0), U635.2 (P0)
- new net GC_U1: U631.13 (Q1), U635.4 (P1)
- new net GC_U2: U631.12 (Q2), U635.6 (P2)
- new net GC_U3: U631.11 (Q3), U635.8 (P3)
- new net GC_U4: U632.14 (Q0), U635.11 (P4)
- new net GC_U5: U632.13 (Q1), U635.13 (P5)
- new net GC_U6: U632.12 (Q2), U635.15 (P6)
- new net GC_U7: U632.11 (Q3), U635.17 (P7)
- new net GC_UTC0: U631.15 (TC), U632.10 (CET)
- new net GC_UTC1: U632.15 (TC), U633.10 (CET)
- new net GC_UTC2: U633.15 (TC), U634.10 (CET)
- new net N2704: U644.1 (1A), U659.4 (2Y)
- new net N2857: U644.13 (4B), U644.8 (3Y)
- new net N2858: U644.11 (4Y), U652.2 (1B)
- new net N2861: U645.3 (1Y), U652.4 (2A)
- new net N2862: U645.6 (2Y), U652.5 (2B)
- new net N2864: U645.11 (4Y), U646.2 (1B)
- new net N2868: U652.8 (3Y), U653.1 (1A)
- new net N2869: U652.11 (4Y), U653.2 (1B)
- new net N2978: U657.5 (2B), U662.2 (1Y)
- new net N2979: U653.13 (4B), U657.6 (2Y)
- new net N3048: U648.5 (2B), U654.6 (2Y)
- new net N3051: U648.8 (3Y), U657.9 (3A)
- new net N3053: U648.11 (4Y), U649.1 (1A)
- new net N3054: U649.2 (1B), U662.6 (3Y)
- new net N3257: U658.1 (1A), U662.8 (4Y)
- new net N3432: U655.12 (4A), U655.6 (2Y)
- new net N3433: U655.13 (4B), U655.8 (3Y)
- new net ~{GC_R0}: U631.3 (D0), U662.10 (5Y)
- new net ~{GC_R14}: U634.5 (D2), U665.2 (1Y)
- new net ~{GC_R15}: U634.6 (D3), U665.4 (2Y)
- new net ~{GC_R1}: U631.4 (D1), U662.12 (6Y)
- new net ~{GC_R4}: U632.3 (D0), U663.6 (3Y)
- new net ~{GC_R5}: U632.4 (D1), U663.8 (4Y)
- new net ~{GC_R6}: U632.5 (D2), U663.10 (5Y)
- new net ~{GC_R7}: U632.6 (D3), U663.12 (6Y)
- new net ~{GC_R9}: U633.4 (D1), U664.4 (2Y)
- new net ~{GC_RLD}: U650.2 (1B), U657.11 (4Y)
- new net ~{GC_TPE}: U631.9 (~{PE}), U632.9 (~{PE}), U633.9 (~{PE}), U634.9 (~{PE}), U650.3 (1Y)
- no-connect marks 106 -> 98
