File: cpu16/kicad/onbellek/onbellek.kicad_sch (KiCad schematic)
At the start: 76 parts, among them J501 BACKPLANE_2x32, U501 74HC688, U502 74HC139, U503 74HC74, U504 74HC74, U505 74HC74, U506 74HC74, U507 74HC161, U508 74HC161, U509 74HC161, U510 74HC157, U511 74HC157, U512 74HC157, U513 62256, U514 62256, U515 74HC541, U516 74HC541, U517 74HC688, U518 74HC688, U519 62256, U520 62256, U521 74HC590, U522 74HC590, U523 74HC590, U524 74HC590, U525 74HC541, U526 74HC08, U527 74HC08, U528 74HC08, U529 74HC08, U530 74HC08, U531 74HC32, U532 74HC32, U533 74HC32, U534 74HC00, U535 74HC02, U536 74HC02, U537 74HC04

Commit message: Kontrol birimi: mikrokod ve ALU ROM'ları yerine 74HC kapı devresi
CPU kartındaki 7 SST39SF010A (4 mikrokod, 3 ALU kod çözme ROM'u) kalktı. Yerine
board/kontrol.ts, cpu16.ucode'dan (tek kaynak) ve aluControl tablosundan çok seviyeli
bir 74HC devresi üretir ve Board API ile gerçek çipler olarak yerleştirir:

- Mikrokod: adım ve komut çözücüleri (74HC138; INT = 1 iken komutlar pasif, f3'e göre
  dallanan komutlara alt çözücü), aynı mikro programı çalıştıran (op, f3, COND)
  atomları, ortak alt kümeli VEYA ağı, sık kullanılan bitler için adım seçici
  (74HC151), adım 8..15 için SWI hattıyla açılan çözücü.
- ALU kod çözme: işlem çözücüleri (3 × 74HC138), işlem bitleri, h ve C terimleri.
- Yeni kapı çipleri: 74HC11, 74HC20, 74HC21, 74HC27, 74HC30 (veri sayfası pin sırası,
  doğruluk tablosu, zamanlama modeli, KiCad sembolü).
- Board: esnek yapıştırıcı kapılar (kartın diğer kapılarından sonra paketlenir, son
  çipi az dolu türü başka türlerin boş birimlerine taşır) ve defer(). Çözücüler eski
  ROM'ların yuvalarına (U1, U3, U5, U7, U10, U68–U71) oturur: kartın diğer bütün
  çiplerinin referansları değişmedi.
- CPU kartı 146 → 194 entegre; en kötü durumda CPU saati 860 → 824 ns (1,21 MHz),
  tipik 470 → 369 ns.
- Denklik testi (tests/kontrol.test.ts): kontrol birimi tek başına bir kartta, gerçek
  çip modelleriyle (LogicSim) 8192 mikrokod adresinin ve 128 ALU adresinin hepsinde
  tabloyla aynı kelimeyi verir.
- roms.ts, cpu16/roms/ ve "roms" komutu kalktı; "kontrol" komutu gömülü mikrokodu
  (micro/cpu16-ucode.ts) yeniler ve devreyi denetler. GateComputer ve GateMachine artık
  mikrokod istemez.
- CPU şeması A0'a sığsın diye dekuplaj kondansatörleri dar sütunlarda; KiCad dosyaları,
  BOM ve deney rehberlerinin otomatik bölümleri yeniden üretildi.

Co-Authored-By: Claude Opus 5.5 (1M context) <noreply@anthropic.com>
Claude-Session: https://claude.ai/code/session_018J8WVuECVRbQJyCbmF6Nsi
Connections:
- net N2189 is gone; now on net N2384: U531.8 (3Y), U534.4 (2A)
- net N2384: no longer U530.11 (4Y), U534.13 (4B)
- net N2174 renamed N2369
- net N2192 renamed N2387
- net N2198 renamed N2393
- net N2200 renamed N2395
- net N2202 renamed N2397
- net N2203 renamed N2398
- net N2382 renamed N2577
- net N2438 renamed N2633
- net N2539 renamed N2734
- new net N2579: U530.11 (4Y), U534.13 (4B)
