File: cpu16/kicad/onbellek/onbellek.kicad_sch (KiCad schematic)
At the start: 76 parts, among them J501 BACKPLANE_2x32, U501 74HC688, U502 74HC139, U503 74HC74, U504 74HC74, U505 74HC74, U506 74HC74, U507 74HC161, U508 74HC161, U509 74HC161, U510 74HC157, U511 74HC157, U512 74HC157, U513 62256, U514 62256, U515 74HC541, U516 74HC541, U517 74HC688, U518 74HC688, U519 62256, U520 62256, U521 74HC590, U522 74HC590, U523 74HC590, U524 74HC590, U525 74HC541, U526 74HC08, U527 74HC08, U528 74HC08, U529 74HC08, U530 74HC08, U531 74HC32, U532 74HC32, U533 74HC32, U534 74HC00, U535 74HC02, U536 74HC02, U537 74HC04

Commit message: Anakart zamanlama testi; önbellek kartında adlandırılmış ara netler
Bütün anakartın zamanlaması testte: 1 MHz CPU en kötü durumda sığar, tutma payları
≥ 5 ns, kapı açıkken değişebilen izinler yalnızca tasarımı gereği güvenli olanlar
(~WSEL, C_MEMACC; önbellek yazma evresindeki C_CB, C_INVL, C_RAMHIT). Bu izinlerin
netleri önbellek kartında adlandırıldı (C_MEMACC, C_TCB, C_INVWR, C_RAMHIT) ki rapor
ve test kararlı olsun.

Co-Authored-By: Claude Opus 5.5 (1M context) <noreply@anthropic.com>
Claude-Session: https://claude.ai/code/session_018J8WVuECVRbQJyCbmF6Nsi
Connections:
- net N2187 renamed C_MEMACC
- net N2190 renamed C_TCB
- net N2194 renamed C_INVWR
- net N2196 renamed C_RAMHIT
Changed lines of the file:
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@@
   (label "~{C_CLK}" (at 256.54 55.88 180) (fields_autoplaced) (effects (font (size 1.27 1.27)) (justify right bottom)))
   (label "C_MEMNOW" (at 256.54 58.42 180) (fields_autoplaced) (effects (font (size 1.27 1.27)) (justify right bottom)))
-  (label "N2187" (at 256.54 60.96 180) (fields_autoplaced) (effects (font (size 1.27 1.27)) (justify right bottom)))
+  (label "C_MEMACC" (at 256.54 60.96 180) (fields_autoplaced) (effects (font (size 1.27 1.27)) (justify right bottom)))
   (label "TCLK" (at 256.54 63.5 180) (fields_autoplaced) (effects (font (size 1.27 1.27)) (justify right bottom)))
   (label "C_CB" (at 256.54 66.04 180) (fields_autoplaced) (effects (font (size 1.27 1.27)) (justify right bottom)))
-  (label "N2190" (at 256.54 68.58 180) (fields_autoplaced) (effects (font (size 1.27 1.27)) (justify right bottom)))
+  (label "C_TCB" (at 256.54 68.58 180) (fields_autoplaced) (effects (font (size 1.27 1.27)) (justify right bottom)))
   (label "~{C_CBF}" (at 256.54 71.12 180) (fields_autoplaced) (effects (font (size 1.27 1.27)) (justify right bottom)))
   (label "C_MEMNOW" (at 276.86 53.34 0) (fields_autoplaced) (effects (font (size 1.27 1.27)) (justify left bottom)))
   (label "C_NEED" (at 276.86 55.88 0) (fields_autoplaced) (effects (font (size 1.27 1.27)) (justify left bottom)))
-  (label "N2190" (at 276.86 58.42 0) (fields_autoplaced) (effects (font (size 1.27 1.27)) (justify left bottom)))
+  (label "C_TCB" (at 276.86 58.42 0) (fields_autoplaced) (effects (font (size 1.27 1.27)) (justify left bottom)))
   (label "C_TAGPH" (at 276.86 60.96 0) (fields_autoplaced) (effects (font (size 1.27 1.27)) (justify left bottom)))
   (label "GND" (at 266.7 78.74 270) (fields_autoplaced) (effects (font (size 1.27 1.27)) (justify right bottom)))
@@
   (label "N2192" (at 276.86 96.52 0) (fields_autoplaced) (effects (font (size 1.27 1.27)) (justify left bottom)))
   (label "C_FILL" (at 276.86 99.06 0) (fields_autoplaced) (effects (font (size 1.27 1.27)) (justify left bottom)))
-  (label "N2194" (at 276.86 101.6 0) (fields_autoplaced) (effects (font (size 1.27 1.27)) (justify left bottom)))
-  (label "N2196" (at 276.86 104.14 0) (fields_autoplaced) (effects (font (size 1.27 1.27)) (justify left bottom)))
+  (label "C_INVWR" (at 276.86 101.6 0) (fields_autoplaced) (effects (font (size 1.27 1.27)) (justify left bottom)))
+  (label "C_RAMHIT" (at 276.86 104.14 0) (fields_autoplaced) (effects (font (size 1.27 1.27)) (justify left bottom)))
   (label "GND" (at 266.7 121.92 270) (fields_autoplaced) (effects (font (size 1.27 1.27)) (justify right bottom)))
   (label "VCC" (at 266.7 91.44 90) (fields_autoplaced) (effects (font (size 1.27 1.27)) (justify left bottom)))
   (label "C_TAGPH" (at 256.54 139.7 180) (fields_autoplaced) (effects (font (size 1.27 1.27)) (justify right bottom)))
-  (label "N2196" (at 256.54 142.24 180) (fields_autoplaced) (effects (font (size 1.27 1.27)) (justify right bottom)))
+  (label "C_RAMHIT" (at 256.54 142.24 180) (fields_autoplaced) (effects (font (size 1.27 1.27)) (justify right bottom)))
   (label "C_SNP" (at 256.54 144.78 180) (fields_autoplaced) (effects (font (size 1.27 1.27)) (justify right bottom)))
   (label "C_WRL_E" (at 256.54 147.32 180) (fields_autoplaced) (effects (font (size 1.27 1.27)) (justify right bottom)))
@@
   (label "C_CA" (at 256.54 238.76 180) (fields_autoplaced) (effects (font (size 1.27 1.27)) (justify right bottom)))
   (label "C_FILL" (at 256.54 241.3 180) (fields_autoplaced) (effects (font (size 1.27 1.27)) (justify right bottom)))
-  (label "N2194" (at 256.54 243.84 180) (fields_autoplaced) (effects (font (size 1.27 1.27)) (justify right bottom)))
+  (label "C_INVWR" (at 256.54 243.84 180) (fields_autoplaced) (effects (font (size 1.27 1.27)) (justify right bottom)))
   (label "C_WRL" (at 276.86 226.06 0) (fields_autoplaced) (effects (font (size 1.27 1.27)) (justify left bottom)))
-  (label "N2187" (at 276.86 228.6 0) (fields_autoplaced) (effects (font (size 1.27 1.27)) (justify left bottom)))
+  (label "C_MEMACC" (at 276.86 228.6 0) (fields_autoplaced) (effects (font (size 1.27 1.27)) (justify left bottom)))
   (label "N2189" (at 276.86 231.14 0) (fields_autoplaced) (effects (font (size 1.27 1.27)) (justify left bottom)))
   (label "C_TAGWR" (at 276.86 233.68 0) (fields_autoplaced) (effects (font (size 1.27 1.27)) (justify left bottom)))

Commit message: Anakart yalnız yaygın parçalarla: 28C256 + 4 × 62256, kendin yap bellek kartı
AFU kararı: bilgisayar yalnız yaygın 7400 serisi lojikle ve iki bellek
çipiyle (62256, 28C256) kurulur.

Bellek kartı (31 → 34 entegre):
- SST39SF010A yerine 28C256 (32 KB, fiziksel 0x00000–0x07FFF, bank 0–1)
- AS6C4008 yerine 4 × 62256 (128 KB, 0x80000–0x9FFFF, bank 32–39)
- çip seçimi tek 74HC138; geri kalan bölgeler boş (0xFF, yazma yok sayılır)

Nadir parçalar çıktı:
- önbellek sayaçları 74HC590 → 74HC161 × 8 + 74HC541 × 4 (37 → 46)
- zamanlayıcı 74HC193 → 74HC161 (tümleyeni yukarı sayar)
- kesme öncelik kodlayıcısı 74HC148 → kapılar
- video adres sayacı (VADDR) 74HC193 → 74HC161 × 4 + yükleme bayrakları
- karakter ROM'u 28C256; yavaşlığı font register'ıyla bir aşamalık boru
  hattında karşılanır (V_H2 en kötü 262 ns, font yolu 199 ns ≤ 317,8);
  resim Machine ile aynı (video 69 → 73 entegre)
- 74HC166 kalır: 74HC165'in eşzamansız yüklemesi piksel saatine sığmaz

Kendin yap bellek kartı (kyb, 22 entegre): FF40–FF4F, 16 bayt, her bayt
bir 74HC574; 74HC138 çözücüler ve 74HC245 veri yolu tamponları. Machine
aygıtı, KiCad klasörü, kapı seviyesi kart Machine ile döngü döngüsüne aynı.

Machine'de At28c256 modeli (sayfa yazma, tBLC, yazma döngüsü, DATA
yoklaması, toggle biti, SDP); kapı seviyesi kartlar aynı modeli kullanır.
BIOS: F komutu korumalı sayfa yazmasıyla yalnız bank 1'e, I komutu yazma
korumasını gösterir, T bank 32–39'u sınar. Deney 8 programı 8 bank sayar,
boş bölgeleri denetler; Deney 14 programı ve testi eklendi.

Co-Authored-By: Claude Opus 5.5 (1M context) <noreply@anthropic.com>
Claude-Session: https://claude.ai/code/session_018J8WVuECVRbQJyCbmF6Nsi
Parts:
- removed U525: 74HC541, Package_DIP:DIP-20_W7.62mm, symbol cpu16:74HC541
- removed U526, U527, U528, U529, U530: 74HC08, Package_DIP:DIP-14_W7.62mm, symbol cpu16:74HC08
- removed U531, U532, U533: 74HC32, Package_DIP:DIP-14_W7.62mm, symbol cpu16:74HC32
- removed U534: 74HC00, Package_DIP:DIP-14_W7.62mm, symbol cpu16:74HC00
- removed U536: 74HC02, Package_DIP:DIP-14_W7.62mm, symbol cpu16:74HC02
- removed U537: 74HC04, Package_DIP:DIP-14_W7.62mm, symbol cpu16:74HC04
- added C522, C539, C540, C541, C542, C543, C544, C545, C546, C547: C_100N, Capacitor_THT:C_Disc_D5.0mm_W2.5mm_P5.00mm, symbol cpu16:C_100N
- added U525, U526, U527, U528: 74HC161, Package_DIP:DIP-16_W7.62mm, symbol cpu16:74HC161
- added U529, U530, U531, U532: 74HC541, Package_DIP:DIP-20_W7.62mm, symbol cpu16:74HC541
- added U534, U535, U536, U537, U538: 74HC08, Package_DIP:DIP-14_W7.62mm, symbol cpu16:74HC08
- added U540, U541: 74HC32, Package_DIP:DIP-14_W7.62mm, symbol cpu16:74HC32
- added U542: 74HC00, Package_DIP:DIP-14_W7.62mm, symbol cpu16:74HC00
- added U543, U544: 74HC02, Package_DIP:DIP-14_W7.62mm, symbol cpu16:74HC02
- added U545, U546: 74HC04, Package_DIP:DIP-14_W7.62mm, symbol cpu16:74HC04
- U521: value 74HC590 -> 74HC161; symbol cpu16:74HC590 -> cpu16:74HC161; Gorev isabet sayacı düşük bayt (FF30) -> isabet sayacı bit 0–3
- U522: value 74HC590 -> 74HC161; symbol cpu16:74HC590 -> cpu16:74HC161; Gorev isabet sayacı yüksek bayt (FF31) -> isabet sayacı bit 4–7
- U523: value 74HC590 -> 74HC161; symbol cpu16:74HC590 -> cpu16:74HC161; Gorev ıskalama sayacı düşük bayt (FF32) -> isabet sayacı bit 8–11
- U524: value 74HC590 -> 74HC161; symbol cpu16:74HC590 -> cpu16:74HC161; Gorev ıskalama sayacı yüksek bayt (FF33) -> isabet sayacı bit 12–15
- U533: renamed from U535; value 74HC02 -> 74HC541; footprint Package_DIP:DIP-14_W7.62mm -> Package_DIP:DIP-20_W7.62mm; symbol cpu16:74HC02 -> cpu16:74HC541; Gorev yapıştırıcı: veri belleği yazma (çift), veri belleği yazma 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 -> CACHE_CTRL geri okuma (FF34)
- U539: renamed from C522; value C_100N -> 74HC08; footprint Capacitor_THT:C_Disc_D5.0mm_W2.5mm_P5.00mm -> Package_DIP:DIP-14_W7.62mm; symbol cpu16:C_100N -> cpu16:74HC08; Gorev U521 dekuplaj -> yapıştırıcı: ıskalama sayımı
Connections:
- net N2198 is gone; now on net GND: U533.3 (A1)
- net ~{C_RCO_H} is gone; now on net VCC: U521.9 (~{PE})
- net ~{C_RCO_M} is gone; now on net VCC: U523.9 (~{PE})
- net CLK: now also U521.2 (CP), U522.2 (CP), U523.2 (CP), U524.2 (CP), U525.2 (CP), U526.2 (CP), U527.2 (CP), U528.2 (CP), U545.13 (6A); no longer U521.11 (CPC), U522.11 (CPC), U523.11 (CPC), U524.11 (CPC)
- net C_CA: now also U534.1 (1A), U538.13 (4B), U540.10 (3B)
- net C_CB: now also U535.10 (3B)
- net C_CBD: now also U534.3 (1Y)
- net C_CLRWE: now also U543.10 (3Y), U543.12 (4B); no longer U533.10 (3Y), U533.12 (4B)
- net C_EN: now also U533.2 (A0), U536.2 (1B), U538.12 (4A), U542.1 (1A)
- net C_ENCK: now also U541.3 (1Y)
- net C_ENHIT: now also U538.2 (1B), U545.10 (5Y)
- net C_FILL: now also U536.6 (2Y), U540.12 (4A), U543.2 (1A), U543.5 (2A); no longer U533.2 (1A), U533.5 (2A)
- net C_HIT: now also U534.4 (2A), U536.12 (4A), U542.2 (1B), U544.1 (1Y)
- net C_INVD: now also U534.8 (3Y)
- net C_INVL: now also U536.10 (3B)
- net C_INVWR: now also U536.8 (3Y), U540.13 (4B)
- net C_MEMACC: now also U535.5 (2B), U540.6 (2Y)
- net C_MEMNOW: now also U535.3 (1Y), U535.4 (2A)
- net C_MRD: now also U539.1 (1A), U534.12 (4A), U536.1 (1A), U537.13 (4B), U538.4 (2A), U545.2 (1Y); no longer U521.13 (CPR), U522.13 (CPR), U523.13 (CPR), U524.13 (CPR)
- net C_NEED: now also U535.6 (2Y), U540.9 (3A)
- net C_RAMHIT: now also U536.11 (4Y), U537.2 (1B)
- net C_RDMISS: now also U534.11 (4Y), U540.5 (2B)
- net C_SNP: now also U537.3 (1Y), U537.4 (2A), U537.9 (3A)
- net C_TAGPH: now also U535.11 (4Y), U536.4 (2A), U536.9 (3A), U537.1 (1A)
- net C_TAGWR: now also U540.11 (4Y), U543.11 (4A); no longer U533.11 (4A)
- net C_TCB: now also U535.12 (4A), U535.8 (3Y)
- net C_VNEW: now also U538.6 (2Y)
- net C_WAITING: now also U534.2 (1B), U545.4 (2Y)
- net C_WRL: now also U534.9 (3A), U540.3 (1Y), U540.4 (2A)
- net C_WRL_E: now also U537.5 (2B), U540.1 (1A)
- net C_WRL_O: now also U537.10 (3B), U540.2 (1B)
- net DE0: now also U533.18 (Y0), U529.18 (Y0), U531.18 (Y0); no longer U521.15 (Q0), U523.15 (Q0)
- net DE1: now also U533.17 (Y1), U529.17 (Y1), U531.17 (Y1); no longer U521.1 (Q1), U523.1 (Q1)
- net DE2: now also U533.16 (Y2), U529.16 (Y2), U531.16 (Y2); no longer U521.2 (Q2), U523.2 (Q2)
- net DE3: now also U533.15 (Y3), U529.15 (Y3), U531.15 (Y3); no longer U521.3 (Q3), U523.3 (Q3)
- net DE4: now also U533.14 (Y4), U529.14 (Y4), U531.14 (Y4); no longer U521.4 (Q4), U523.4 (Q4)
- net DE5: now also U533.13 (Y5), U529.13 (Y5), U531.13 (Y5); no longer U521.5 (Q5), U523.5 (Q5)
- net DE6: now also U533.12 (Y6), U529.12 (Y6), U531.12 (Y6); no longer U521.6 (Q6), U523.6 (Q6)
- net DE7: now also U533.11 (Y7), U529.11 (Y7), U531.11 (Y7); no longer U521.7 (Q7), U523.7 (Q7)
- net DO0: now also U530.18 (Y0), U532.18 (Y0); no longer U522.15 (Q0), U524.15 (Q0)
- net DO1: now also U530.17 (Y1), U532.17 (Y1); no longer U522.1 (Q1), U524.1 (Q1)
- net DO2: now also U530.16 (Y2), U532.16 (Y2); no longer U522.2 (Q2), U524.2 (Q2)
- net DO3: now also U530.15 (Y3), U532.15 (Y3); no longer U522.3 (Q3), U524.3 (Q3)
- net DO4: now also U530.14 (Y4), U532.14 (Y4); no longer U522.4 (Q4), U524.4 (Q4)
- net DO5: now also U530.13 (Y5), U532.13 (Y5); no longer U522.5 (Q5), U524.5 (Q5)
- net DO6: now also U530.12 (Y6), U532.12 (Y6); no longer U522.6 (Q6), U524.6 (Q6)
- net DO7: now also U530.11 (Y7), U532.11 (Y7); no longer U522.7 (Q7), U524.7 (Q7)
- net GND: now also U521.3 (D0), U521.4 (D1), U521.5 (D2), U521.6 (D3), U522.3 (D0), U522.4 (D1), U522.5 (D2), U522.6 (D3), U523.3 (D0), U523.4 (D1), U523.5 (D2), U523.6 (D3), U524.3 (D0), U524.4 (D1), U524.5 (D2), U524.6 (D3), U533.10 (GND), U533.4 (A2), U533.5 (A3), U533.6 (A4), U533.8 (A6), U533.9 (A7), U539.10 (3B), U539.12 (4A), U539.13 (4B), U539.4 (2A), U539.5 (2B), U539.7 (GND), U539.9 (3A), C522.2, C539.2, C540.2, C541.2, C542.2, C543.2, C544.2, C545.2, C546.2, C547.2, U525.3 (D0), U525.4 (D1), U525.5 (D2), U525.6 (D3), U525.8 (GND), U526.3 (D0), U526.4 (D1), U526.5 (D2), U526.6 (D3), U526.8 (GND), U527.3 (D0), U527.4 (D1), U527.5 (D2), U527.6 (D3), U527.8 (GND), U528.3 (D0), U528.4 (D1), U528.5 (D2), U528.6 (D3), U528.8 (GND), U529.10 (GND), U529.19 (~{OE2}), U530.10 (GND), U530.19 (~{OE2}), U531.10 (GND), U531.19 (~{OE2}), U532.10 (GND), U532.19 (~{OE2}), U534.7 (GND), U535.7 (GND), U536.7 (GND), U537.7 (GND), U538.7 (GND), U540.7 (GND), U541.7 (GND), U542.12 (4A), U542.13 (4B), U542.7 (GND), U543.7 (GND), U544.11 (4A), U544.12 (4B), U544.5 (2A), U544.6 (2B), U544.7 (GND), U544.8 (3A), U544.9 (3B), U545.7 (GND), U546.11 (5A), U546.13 (6A), U546.3 (2A), U546.5 (3A), U546.7 (GND), U546.9 (4A); no longer U539.2
- net N2200: now also U540.8 (3Y), U542.4 (2A); no longer U533.6 (2B)
- net N2203: now also U536.3 (1Y), U536.5 (2B)
- net OSC: now also U543.8 (3A); no longer U533.8 (3A)
- net PA19: now also U536.13 (4B), U545.9 (4A)
- net TCLK: now also U535.9 (3A), U545.5 (3A)
- net VCC: now also U521.10 (CET), U522.9 (~{PE}), U524.9 (~{PE}), U533.20 (VCC), U539.14 (VCC), C522.1, C539.1, C540.1, C541.1, C542.1, C543.1, C544.1, C545.1, C546.1, C547.1, U525.10 (CET), U525.16 (VCC), U525.9 (~{PE}), U526.16 (VCC), U526.9 (~{PE}), U527.16 (VCC), U527.9 (~{PE}), U528.16 (VCC), U528.9 (~{PE}), U529.20 (VCC), U530.20 (VCC), U531.20 (VCC), U532.20 (VCC), U534.14 (VCC), U535.14 (VCC), U536.14 (VCC), U537.14 (VCC), U538.14 (VCC), U540.14 (VCC), U541.14 (VCC), U542.14 (VCC), U543.14 (VCC), U544.14 (VCC), U545.14 (VCC), U546.14 (VCC); no longer U533.14 (VCC), U539.1
- net ~{CS_CTRL}: now also U533.19 (~{OE2}), U541.2 (1B)
- net ~{CS_HITS}: now also U541.10 (3B), U541.5 (2B)
- net ~{CS_MISS}: now also U541.13 (4B)
- net ~{C_CA}: now also U542.10 (3B)
- net ~{C_CBF}: now also U535.13 (4B)
- net ~{C_CB}: now also U542.5 (2B)
- net ~{C_CLK}: now also U535.2 (1B), U545.12 (6Y)
- net ~{C_CLRS}: now also U538.5 (2B), U543.9 (3B); no longer U533.9 (3B)
- net ~{C_CNTCLR}: now also U521.1 (~{MR}), U522.1 (~{MR}), U523.1 (~{MR}), U524.1 (~{MR}), U525.1 (~{MR}), U526.1 (~{MR}), U527.1 (~{MR}), U528.1 (~{MR}), U538.8 (3Y); no longer U521.10 (~{MRC}), U522.10 (~{MRC}), U523.10 (~{MRC}), U524.10 (~{MRC})
- net ~{C_CWE_E}: now also U543.1 (1Y); no longer U533.1 (1Y)
- net ~{C_CWE_O}: now also U543.4 (2Y); no longer U533.4 (2Y)
- net ~{C_ENHIT}: now also U534.13 (4B), U542.3 (1Y), U545.11 (5A)
- net ~{C_HITRD}: now also U542.8 (3Y), U546.1 (1A); no longer U521.12 (~{CEC})
- net ~{C_OE_HITS}: now also U529.1 (~{OE1}), U530.1 (~{OE1}), U541.8 (3Y); no longer U521.14 (~{OE}), U522.14 (~{OE})
- net ~{C_OE_MISS}: now also U531.1 (~{OE1}), U532.1 (~{OE1}), U541.11 (4Y); no longer U523.14 (~{OE}), U524.14 (~{OE})
- net ~{C_TCLK}: now also U545.6 (3Y)
- net ~{C_TEQ_HI}: now also U544.3 (1B)
- net ~{C_TEQ_LO}: now also U544.2 (1A)
- net ~{C_TWE}: now also U543.13 (4Y); no longer U533.13 (4Y)
- net ~{IO}: now also U535.1 (1A), U537.12 (4A)
- net ~{MRD}: now also U533.1 (~{OE1}), U541.12 (4A), U541.9 (3A), U545.1 (1A)
- net ~{MWE_E}: now also U541.1 (1A), U541.4 (2A)
- net ~{RESET}: now also U538.9 (3A)
- net ~{WAIT}: now also U542.6 (2Y), U545.3 (2A)
- net N2438 renamed C_HC6
- net C_HC6: now also U529.8 (A6)
- net N2539 renamed C_HC14
- net C_HC14: now also U530.8 (A6)
- net ~{C_MISS} renamed C_HC10
- net C_HC10: now also U530.4 (A2)
- new net C_HC0: U521.14 (Q0), U529.2 (A0)
- new net C_HC1: U521.13 (Q1), U529.3 (A1)
- new net C_HC11: U523.11 (Q3), U530.5 (A3)
- new net C_HC12: U524.14 (Q0), U530.6 (A4)
- new net C_HC13: U524.13 (Q1), U530.7 (A5)
- new net C_HC15: U524.11 (Q3), U530.9 (A7)
- new net C_HC2: U521.12 (Q2), U529.4 (A2)
- new net C_HC3: U521.11 (Q3), U529.5 (A3)
- new net C_HC4: U522.14 (Q0), U529.6 (A4)
- new net C_HC5: U522.13 (Q1), U529.7 (A5)
- new net C_HC7: U522.11 (Q3), U529.9 (A7)
- new net C_HC8: U523.14 (Q0), U530.2 (A0)
- new net C_HC9: U523.13 (Q1), U530.3 (A1)
- new net C_HC_TC0: U521.15 (TC), U522.10 (CET)
- new net C_HC_TC1: U522.15 (TC), U523.10 (CET)
- new net C_HC_TC2: U523.15 (TC), U524.10 (CET)
- new net C_HITCNT: U521.7 (CEP), U522.7 (CEP), U523.7 (CEP), U524.7 (CEP), U546.2 (1Y)
- new net C_MC0: U525.14 (Q0), U531.2 (A0)
- new net C_MC1: U525.13 (Q1), U531.3 (A1)
- new net C_MC10: U527.12 (Q2), U532.4 (A2)
- new net C_MC11: U527.11 (Q3), U532.5 (A3)
- new net C_MC12: U528.14 (Q0), U532.6 (A4)
- new net C_MC13: U528.13 (Q1), U532.7 (A5)
- new net C_MC14: U528.12 (Q2), U532.8 (A6)
- new net C_MC15: U528.11 (Q3), U532.9 (A7)
- new net C_MC2: U525.12 (Q2), U531.4 (A2)
- new net C_MC3: U525.11 (Q3), U531.5 (A3)
- new net C_MC4: U526.14 (Q0), U531.6 (A4)
- new net C_MC5: U526.13 (Q1), U531.7 (A5)
- new net C_MC6: U526.12 (Q2), U531.8 (A6)
- new net C_MC7: U526.11 (Q3), U531.9 (A7)
- new net C_MC8: U527.14 (Q0), U532.2 (A0)
- new net C_MC9: U527.13 (Q1), U532.3 (A1)
- new net C_MC_TC0: U525.15 (TC), U526.10 (CET)
- new net C_MC_TC1: U526.15 (TC), U527.10 (CET)
- new net C_MC_TC2: U527.15 (TC), U528.10 (CET)
- new net C_MISSCNT: U525.7 (CEP), U526.7 (CEP), U527.7 (CEP), U528.7 (CEP), U539.3 (1Y)
- new net C_ROM: U534.5 (2B), U545.8 (4Y)
- new net N2185: U534.10 (3B), U534.6 (2Y)
- new net N2209: U537.6 (2Y), U543.3 (1B)
- new net N2211: U537.8 (3Y), U543.6 (2B)
- new net N2213: U537.11 (4Y), U538.1 (1A)
- new net N2214: U538.3 (1Y), U542.9 (3A)
- new net N2393: U538.10 (3B), U541.6 (2Y)
- new net N2396: U538.11 (4Y), U539.2 (1B)
- no-connect marks 27 -> 34
