File: cpu16/kicad/video/video.kicad_sch (KiCad schematic)
At the start: 148 parts, among them J701 CONN_VGA, J702 BACKPLANE_2x32, U701 74HC138, U702 74HC138, U703 74HC138, U704 74HC138, U705 74HC161, U706 74HC161, U707 74HC161, U708 74HC161, U709 74HC161, U710 74HC161, U711 74HC74, U712 74HC688, U713 74HC74, U714 74HC393, U715 74HC541, U716 74HC161, U717 74HC161, U718 74HC161, U719 74HC574, U720 74HC574, U721 74HC157, U722 74HC157, U723 74HC157, U724 62256, U725 62256, U726 74HC574, U727 74HC574, U728 74HC574, U729 SST39SF010A, U730 74HC166, U731 74HC175, U732 74HC688, U733 74HC688, U734 74HC157, U735 74HC193, U736 74HC193, U737 74HC193, U738 74HC193, U739 74HC74, U740 74HC74, U741 74HC74, U742 74HC74, U743 74HC574, U744 74HC574, U745 74HC574, U746 74HC574, U747 74HC541, U748 74HC574, U749 74HC574, U750 74HC541, U751 74HC541, U752 74HC08, U753 74HC08, U754 74HC08, U755 74HC08, U756 74HC08, U757 74HC08, U758 74HC08, U759 74HC08, U760 74HC08, U761 74HC32, U762 74HC32, U763 74HC32, U764 74HC00, U765 74HC02, U766 74HC04, U767 74HC04, U768 74HC10, U769 74HC10, X701 OSC_25M175

Commit message: Video kartı zamanlaması: sayaçlar karakter saatinde; piksel saatinde yalnız 74AC161, 74AC74 ve kaydırıcı
Statik zamanlama analizi piksel saatinde (VID_OSC, hedef 39,7 ns) en kötü 127 ns (7,87 MHz),
tipik 89 ns (11,24 MHz) buluyordu: yatay sayaç → satır sonu çözümü → dikey sayacın ~PE'si.

- Piksel fazı ayrı bir 74AC161: 9..15, 0 diye sayar; Q3 hem kendi ~PE'sine hem 74HC166'nın
  ~PE'sine doğrudan gider (çözücü kapı yok).
- 74AC74: H2 = Q2'nin bir piksel gecikmişi (parazitsiz karakter saati), LD7 = TC'nin.
- Karakter sayacı (0..99), dikey sayaç, MA, satır başı ve CPU istekleri H2'de (p4), VBQ ve
  eşzamanlayıcılar H2'nin düşen kenarında (p0); satır sonu çözümü artık 318 ns'lik alanda.
- Karartma, senkronlar ve imleç p4'te ön 74HC175'e, p7 → p0'da (Q3'ün yükselen kenarı) çıkış
  74HC175'ine alınır; VID_OSC ile kapılı karakter sınırı saati kalktı.
- Satır başı saati H2 ∨ ¬ENRS (ENRS yalnız H2 = 1 iken değişir); ENRS'de VBQ yerine VBL.
- VRAM yazma darbesi H2 ∧ Q1 (p5–p6): her kenarda tek giriş değişir.

Sonuç: VID_OSC en kötü 30,5 ns (32,79 MHz), tipik 16,8 ns (59,52 MHz); piksel saatinde kapılı
saat, açıkken değişen izin ya da tutma denetimi yok. Karakter saati (kök H2) en kötü 262 ns
(3,82 MHz; hedef 3,15 MHz), tutma payı 36 ns. Çip sayısı 69 → 69 (+1 74HC175, −1 74HC08), 2'si
74AC. Alanlar arası geçişler belgede elle hesaplandı.

Davranış aynı: VSTAT / VSYNC_REQ aynı piksel kenarında (384 000, 420 000), kilit adım testi
değişmeden geçiyor. Açılışta faz sayacı p7'de olduğu için tezgâhta görüntü bir piksel geç başlar:
testler hc = x + 9 bekler (kartın kendi sayacında hc = x + 8). Yeni test: bütün anakartta iki
kök, iki köşe.

Co-Authored-By: Claude Opus 5.5 (1M context) <noreply@anthropic.com>
Claude-Session: https://claude.ai/code/session_018J8WVuECVRbQJyCbmF6Nsi
Parts:
- removed U706: 74HC161, Package_DIP:DIP-16_W7.62mm, symbol cpu16:74HC161
- removed U711, U739: 74HC74, Package_DIP:DIP-14_W7.62mm, symbol cpu16:74HC74
- removed U732: 74HC688, Package_DIP:DIP-20_W7.62mm, symbol cpu16:74HC688
- removed U734: 74HC157, Package_DIP:DIP-16_W7.62mm, symbol cpu16:74HC157
- removed U743, U748: 74HC574, Package_DIP:DIP-20_W7.62mm, symbol cpu16:74HC574
- removed U747, U750: 74HC541, Package_DIP:DIP-20_W7.62mm, symbol cpu16:74HC541
- removed U752: 74HC08, Package_DIP:DIP-14_W7.62mm, symbol cpu16:74HC08
- added U706: 74AC74, Package_DIP:DIP-14_W7.62mm, symbol cpu16:74HC74
- added U711: 74HC161, Package_DIP:DIP-16_W7.62mm, symbol cpu16:74HC161
- added U732: 74HC175, Package_DIP:DIP-16_W7.62mm, symbol cpu16:74HC175
- added U734: 74HC688, Package_DIP:DIP-20_W7.62mm, symbol cpu16:74HC688
- added U739: 74HC193, Package_DIP:DIP-16_W7.62mm, symbol cpu16:74HC193
- added U743: 74HC74, Package_DIP:DIP-14_W7.62mm, symbol cpu16:74HC74
- added U747, U750: 74HC574, Package_DIP:DIP-20_W7.62mm, symbol cpu16:74HC574
- added U748, U752: 74HC541, Package_DIP:DIP-20_W7.62mm, symbol cpu16:74HC541
- U705: value 74HC161 -> 74AC161; Gorev yatay sayaç H0–H3 (piksel) -> piksel fazı p0..p7 (9..15, 0); Q3 = 0 → p7
- U707: Gorev yatay sayaç H8–H9 -> karakter sayacı H3–H6 (0..99)
- U708: Gorev dikey sayaç V0–V3 (satır) -> karakter sayacı H7–H9
- U709: Gorev dikey sayaç V4–V7 -> dikey sayaç V0–V3 (satır)
- U710: Gorev dikey sayaç V8–V9 -> dikey sayaç V4–V7
- U728: Gorev renk baytı (karakter sınırında, gösterilen karakterinki) -> renk baytı (p7 → p0 kenarında, gösterilen karakterinki)
- U731: Gorev karartma, senkronlar (negatif) ve imleç: piksellerle aynı k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 -> karartma, senkronlar, imleç: ön register (p4)
- U733: Gorev imleç satırı = karakter satırı -> imleç sütunu = karakter sütunu
- U735: value 74HC193 -> 74HC157; symbol cpu16:74HC193 -> cpu16:74HC157; Gorev VADDR bit 0–3 -> IRGB: yazı / zemin rengi, karartmada siyah
- U736: Gorev VADDR bit 4–7 -> VADDR bit 0–3
- U737: Gorev VADDR bit 8–11 -> VADDR bit 4–7
- U738: Gorev VADDR bit 12–12 -> VADDR bit 8–11
- U740: Gorev istek eşzamanlayıcı (p0) -> VDATA yazma isteği, ön okuma isteği
- U741: Gorev bu CPU yuvasında: yazma / ön okuma -> istek eşzamanlayıcı (p0)
- U742: Gorev VDATA okuma yan etkisi (sonraki döngü), VCTRL (FF23) -> bu CPU yuvasında: yazma / ön okuma
- U744: Gorev VDATA yazma verisi → renk şeridi -> VDATA yazma verisi → karakter şeridi
- U745: Gorev VDATA ön okuma (karakter şeridi) -> VDATA yazma verisi → renk şeridi
- U746: Gorev VDATA ön okuma (renk şeridi) -> VDATA ön okuma (karakter şeridi)
- U749: Gorev CURSOR_Y (FF25) -> CURSOR_X (FF24)
- U751: Gorev CURSOR_Y okuma -> CURSOR_X okuma
- U753: Gorev yapıştırıcı: p = 4, 5, hc ≥ 640 (yatay karartma), karakter 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 -> yapıştırıcı: karakter 98 / 99, VRAM yazma darbesi (p5–p6)
- U754: Gorev yapıştırıcı: karakter 80..95, alt 4 bit 2..13, karakter 82.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 -> yapıştırıcı: hc ≥ 640 (yatay karartma), karakter 98: satır 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
- U755: Gorev yapıştırıcı: tarama satırı 14–15 -> yapıştırıcı: alt 4 bit 2..13, karakter 82..93: HSYNC (96 pi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
- U756: Gorev yapıştırıcı: karakter satırının son tarama satırı, VSTAT'a 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 -> yapıştırıcı: tarama satırı 14–15, karakter satırının son ta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
- U761: Gorev yapıştırıcı: karakter sınırı saati (p7 → p0) -> yapıştırıcı: vc ≥ 480 (dikey karartma)
- U762: Gorev yapıştırıcı: vc ≥ 480 (dikey karartma), karartma, yazı reng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 -> yapıştırıcı: karartma, satır başı saati (p4), yazı rengi: p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
- U764: Gorev yapıştırıcı: karakter 99: MA ← satır başı, yazma bitti: VAD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 -> yapıştırıcı: karakter 99 (satır sonu), satır başını güncell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
- U766: Gorev yapıştırıcı: reset (aktif yüksek), satır sonu, CPU yuvası b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 -> yapıştırıcı: reset (aktif yüksek), CPU yuvası bitti (p0), s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
- U768: Gorev yapıştırıcı: hc = 799 (satır sonu), vc = 524 ve satır sonu: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 -> yapıştırıcı: vc = 524 ve satır sonu: kare sonu, karakter şe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
- U769: Gorev yapıştırıcı: karakter şeridine yaz (VADDR çift), renk şerid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 -> yapıştırıcı: renk şeridine yaz (VADDR tek)
Connections:
- net N3689 is gone; now on net V_HEND: U766.6 (3Y)
- net N4148 is gone; now on net N4150: U757.12 (4A), U757.6 (2Y)
- net N4168 is gone; now on net N4170: U758.5 (2B), U765.4 (2Y)
- net V_HTC1 is gone; now on net VCC: U707.10 (CET)
- net V_P45 is gone; now on net V_H89: U753.3 (1Y)
- net ~{V_HC99} is gone; now on net ~{V_HEND}: U716.9 (~{PE}), U717.9 (~{PE}), U718.9 (~{PE}), U764.3 (1Y)
- net CLK: now also U743.3 (1CLK); no longer U742.3 (1CLK)
- net DE0: now also U736.15 (D0), U745.2 (D0), U749.2 (D0), U751.18 (Y0), U747.19 (Q0); no longer U735.15 (D0), U745.19 (Q0)
- net DE1: now also U736.1 (D1), U745.3 (D1), U749.3 (D1), U751.17 (Y1), U747.18 (Q1); no longer U735.1 (D1), U745.18 (Q1)
- net DE2: now also U736.10 (D2), U745.4 (D2), U749.4 (D2), U751.16 (Y2), U747.17 (Q2); no longer U735.10 (D2), U745.17 (Q2)
- net DE3: now also U736.9 (D3), U745.5 (D3), U749.5 (D3), U751.15 (Y3), U747.16 (Q3); no longer U735.9 (D3), U745.16 (Q3)
- net DE4: now also U737.15 (D0), U745.6 (D4), U749.6 (D4), U751.14 (Y4), U747.15 (Q4); no longer U736.15 (D0), U745.15 (Q4)
- net DE5: now also U737.1 (D1), U745.7 (D5), U749.7 (D5), U751.13 (Y5), U747.14 (Q5); no longer U736.1 (D1), U745.14 (Q5)
- net DE6: now also U737.10 (D2), U745.8 (D6), U749.8 (D6), U751.12 (Y6), U747.13 (Q6); no longer U736.10 (D2), U745.13 (Q6)
- net DE7: now also U737.9 (D3), U745.9 (D7), U749.9 (D7), U751.11 (Y7), U747.12 (Q7); no longer U736.9 (D3), U745.12 (Q7)
- net DO0: now also U738.15 (D0), U743.12 (2D), U748.18 (Y0), U750.2 (D0), U752.18 (Y0); no longer U737.15 (D0), U742.12 (2D), U749.2 (D0), U751.18 (Y0)
- net DO1: now also U738.1 (D1), U748.17 (Y1), U750.3 (D1), U752.17 (Y1); no longer U737.1 (D1), U749.3 (D1), U751.17 (Y1)
- net DO2: now also U738.10 (D2), U748.16 (Y2), U750.4 (D2), U752.16 (Y2); no longer U737.10 (D2), U749.4 (D2), U751.16 (Y2)
- net DO3: now also U738.9 (D3), U748.15 (Y3), U750.5 (D3), U752.15 (Y3); no longer U737.9 (D3), U749.5 (D3), U751.15 (Y3)
- net DO4: now also U739.15 (D0), U748.14 (Y4), U750.6 (D4), U752.14 (Y4); no longer U738.15 (D0), U749.6 (D4), U751.14 (Y4)
- net DO5: now also U739.1 (D1), U748.13 (Y5), U750.7 (D5), U752.13 (Y5); no longer U738.1 (D1), U749.7 (D5), U751.13 (Y5)
- net DO6: now also U739.10 (D2), U748.12 (Y6), U750.8 (D6), U752.12 (Y6); no longer U738.10 (D2), U749.8 (D6), U751.12 (Y6)
- net DO7: now also U739.9 (D3), U748.11 (Y7), U750.9 (D7), U752.11 (Y7); no longer U738.9 (D3), U749.9 (D7), U751.11 (Y7)
- net GND: now also U767.11 (5A), U767.13 (6A), U769.3 (2A), U769.4 (2B), U769.5 (2C), U706.7 (GND), U711.3 (D0), U711.4 (D1), U711.5 (D2), U711.6 (D3), U711.8 (GND), U732.8 (GND), U734.1 (~{E}), U734.10 (GND), U734.15 (P6), U734.17 (P7), U739.8 (GND), U743.7 (GND), U747.10 (GND), U748.10 (GND), U748.19 (~{OE2}), U748.3 (A1), U748.4 (A2), U748.5 (A3), U748.6 (A4), U748.7 (A5), U748.8 (A6), U748.9 (A7), U750.1 (~{OE}), U750.10 (GND), U752.10 (GND), U752.19 (~{OE2}); no longer U705.3 (D0), U705.6 (D3), U733.15 (P6), U764.12 (4A), U764.13 (4B)
- net N3704: now also U755.1 (1A), U761.8 (3Y); no longer U753.13 (4B), U767.2 (1Y)
- net N3709: now also U755.11 (4Y), U756.2 (1B); no longer U761.12 (4A), U761.8 (3Y)
- net N3710: now also U756.3 (1Y), U761.13 (4B); no longer U754.9 (3A), U761.11 (4Y)
- net N4150: no longer U757.9 (3A), U765.1 (1Y)
- net N4170: no longer U758.10 (3B), U767.12 (6Y)
- net VCC: now also U705.3 (D0), U705.6 (D3), U708.7 (CEP), U709.10 (CET), U740.12 (2D), U740.2 (1D), U706.1 (~{1CLR}), U706.10 (~{2PRE}), U706.13 (~{2CLR}), U706.14 (VCC), U706.4 (~{1PRE}), U711.1 (~{MR}), U711.16 (VCC), U732.1 (~{MR}), U732.16 (VCC), U734.20 (VCC), U739.16 (VCC), U739.4 (CPD), U743.10 (~{2PRE}), U743.14 (VCC), U743.4 (~{1PRE}), U747.20 (VCC), U748.20 (VCC), U750.20 (VCC), U752.20 (VCC); no longer U708.10 (CET), U735.4 (CPD), U740.10 (~{2PRE})
- net VGA_HSYNC: now also U732.6 (~{Q1}); no longer U731.6 (~{Q1})
- net VGA_VSYNC: now also U732.10 (Q2); no longer U731.10 (Q2)
- net VID_OSC: now also U706.11 (2CLK), U706.3 (1CLK); no longer U707.2 (CP), U708.2 (CP), U709.2 (CP), U710.2 (CP), U713.3 (1CLK), U761.1 (1A)
- net V_AD0: now also U745.19 (Q0), U747.2 (D0); no longer U744.19 (Q0), U746.2 (D0)
- net V_AD1: now also U745.18 (Q1), U747.3 (D1); no longer U744.18 (Q1), U746.3 (D1)
- net V_AD2: now also U745.17 (Q2), U747.4 (D2); no longer U744.17 (Q2), U746.4 (D2)
- net V_AD3: now also U745.16 (Q3), U747.5 (D3); no longer U744.16 (Q3), U746.5 (D3)
- net V_AD4: now also U745.15 (Q4), U747.6 (D4); no longer U744.15 (Q4), U746.6 (D4)
- net V_AD5: now also U745.14 (Q5), U747.7 (D5); no longer U744.14 (Q5), U746.7 (D5)
- net V_AD6: now also U745.13 (Q6), U747.8 (D6); no longer U744.13 (Q6), U746.8 (D6)
- net V_AD7: now also U745.12 (Q7), U747.9 (D7); no longer U744.12 (Q7), U746.9 (D7)
- net V_ADR0: now also U736.3 (Q0), U767.3 (2A), U769.13 (1C); no longer U735.3 (Q0), U767.9 (4A), U769.5 (2C)
- net V_ADR1: now also U736.2 (Q1); no longer U735.2 (Q1)
- net V_ADR10: now also U738.6 (Q2); no longer U737.6 (Q2)
- net V_ADR11: now also U738.7 (Q3); no longer U737.7 (Q3)
- net V_ADR12: now also U739.3 (Q0); no longer U738.3 (Q0)
- net V_ADR2: now also U736.6 (Q2); no longer U735.6 (Q2)
- net V_ADR3: now also U736.7 (Q3); no longer U735.7 (Q3)
- net V_ADR4: now also U737.3 (Q0); no longer U736.3 (Q0)
- net V_ADR5: now also U737.2 (Q1); no longer U736.2 (Q1)
- net V_ADR6: now also U737.6 (Q2); no longer U736.6 (Q2)
- net V_ADR7: now also U737.7 (Q3); no longer U736.7 (Q3)
- net V_ADR8: now also U738.3 (Q0); no longer U737.3 (Q0)
- net V_ADR9: now also U738.2 (Q1); no longer U737.2 (Q1)
- net V_ATD0: now also U735.3 (1I1)
- net V_ATD1: now also U735.6 (2I1)
- net V_ATD2: now also U735.10 (3I1)
- net V_ATD3: now also U735.13 (4I1)
- net V_ATD4: now also U735.2 (1I0)
- net V_ATD5: now also U735.5 (2I0)
- net V_ATD6: now also U735.11 (3I0)
- net V_ATD7: now also U735.14 (4I0)
- net V_B: now also U735.4 (1Y)
- net V_BLANK: now also U762.3 (1Y); no longer U762.6 (2Y)
- net V_BLANKD: now also U735.15 (~{E}), U732.2 (Q0); no longer U731.2 (Q0)
- net V_BLINK: now also U767.5 (3A); no longer U767.11 (5A)
- net V_BROWN: now also U767.9 (4A); no longer U767.13 (6A)
- net V_CD0: now also U744.19 (Q0), U746.2 (D0); no longer U745.2 (D0)
- net V_CD1: now also U744.18 (Q1), U746.3 (D1); no longer U745.3 (D1)
- net V_CD2: now also U744.17 (Q2), U746.4 (D2); no longer U745.4 (D2)
- net V_CD3: now also U744.16 (Q3), U746.5 (D3); no longer U745.5 (D3)
- net V_CD4: now also U744.15 (Q4), U746.6 (D4); no longer U745.6 (D4)
- net V_CD5: now also U744.14 (Q5), U746.7 (D5); no longer U745.7 (D5)
- net V_CD6: now also U744.13 (Q6), U746.8 (D6); no longer U745.8 (D6)
- net V_CD7: now also U744.12 (Q7), U746.9 (D7); no longer U745.9 (D7)
- net V_CURD: now also U732.15 (Q3); no longer U731.15 (Q3)
- net V_CX0: now also U733.3 (Q0), U749.19 (Q0), U751.2 (A0)
- net V_CX1: now also U733.5 (Q1), U749.18 (Q1), U751.3 (A1)
- net V_CX2: now also U733.7 (Q2), U749.17 (Q2), U751.4 (A2)
- net V_CX3: now also U733.9 (Q3), U749.16 (Q3), U751.5 (A3)
- net V_CX4: now also U733.12 (Q4), U749.15 (Q4), U751.6 (A4)
- net V_CX5: now also U733.14 (Q5), U749.14 (Q5), U751.7 (A5)
- net V_CX6: now also U733.16 (Q6), U749.13 (Q6), U751.8 (A6)
- net V_CX7: now also U733.18 (Q7), U749.12 (Q7), U751.9 (A7)
- net V_CY0: now also U734.3 (Q0), U750.19 (Q0), U752.2 (A0); no longer U733.3 (Q0), U749.19 (Q0), U751.2 (A0)
- net V_CY1: now also U734.5 (Q1), U750.18 (Q1), U752.3 (A1); no longer U733.5 (Q1), U749.18 (Q1), U751.3 (A1)
- net V_CY2: now also U734.7 (Q2), U750.17 (Q2), U752.4 (A2); no longer U733.7 (Q2), U749.17 (Q2), U751.4 (A2)
- net V_CY3: now also U734.9 (Q3), U750.16 (Q3), U752.5 (A3); no longer U733.9 (Q3), U749.16 (Q3), U751.5 (A3)
- net V_CY4: now also U734.12 (Q4), U750.15 (Q4), U752.6 (A4); no longer U733.12 (Q4), U749.15 (Q4), U751.6 (A4)
- net V_CY5: now also U734.14 (Q5), U750.14 (Q5), U752.7 (A5); no longer U733.14 (Q5), U749.14 (Q5), U751.7 (A5)
- net V_CY6: now also U734.16 (Q6), U750.13 (Q6), U752.8 (A6); no longer U733.16 (Q6), U749.13 (Q6), U751.8 (A6)
- net V_CY7: now also U734.18 (Q7), U750.12 (Q7), U752.9 (A7); no longer U733.18 (Q7), U749.12 (Q7), U751.9 (A7)
- net V_FGSEL: now also U735.1 (S)
- net V_G: now also U735.7 (2Y)
- net V_H2: now also U707.2 (CP), U708.2 (CP), U709.2 (CP), U710.2 (CP), U731.9 (CP), U742.11 (2CLK), U742.3 (1CLK), U753.12 (4A), U762.9 (3A), U766.3 (2A), U706.5 (1Q), U711.2 (CP); no longer U705.12 (Q2), U741.11 (2CLK), U741.3 (1CLK), U753.1 (1A), U756.12 (4A), U766.11 (5A)
- net V_H2N: now also U713.3 (1CLK), U741.11 (2CLK), U741.3 (1CLK), U766.4 (2Y); no longer U740.11 (2CLK), U740.3 (1CLK), U766.10 (5Y)
- net V_H3: now also U707.14 (Q0), U733.2 (P0), U766.11 (5A); no longer U705.11 (Q3), U767.1 (1A)
- net V_H4: now also U707.13 (Q1), U733.4 (P1), U753.5 (2B), U761.4 (2A), U768.3 (2A); no longer U753.10 (3B), U761.9 (3A), U768.2 (1B), U768.9 (3A)
- net V_H5: now also U707.12 (Q2), U733.6 (P2), U761.5 (2B), U768.4 (2B); no longer U761.10 (3B), U768.10 (3B)
- net V_H6: now also U707.11 (Q3), U733.8 (P3), U761.10 (3B), U768.5 (2C); no longer U761.13 (4B), U768.11 (3C)
- net V_H7: now also U708.14 (Q0), U733.11 (P4), U754.10 (3B), U761.2 (1B); no longer U754.2 (1B), U761.5 (2B)
- net V_H8: now also U708.13 (Q1), U733.13 (P5), U753.1 (1A), U761.1 (1A), U766.13 (6A); no longer U707.14 (Q0), U761.4 (2A), U767.3 (2A)
- net V_H89: now also U753.4 (2A); no longer U753.9 (3A), U768.13 (1C)
- net V_H9: now also U708.12 (Q2), U733.15 (P6), U753.2 (1B), U754.9 (3A); no longer U707.13 (Q1), U753.4 (2A)
- net V_H984: now also U753.6 (2Y), U754.4 (2A); no longer U753.12 (4A), U753.8 (3Y)
- net V_HBL: now also U754.3 (1Y), U762.1 (1A), U766.9 (4A); no longer U753.6 (2Y), U762.4 (2A), U766.13 (6A)
- net V_HC98: now also U754.6 (2Y), U764.9 (3A); no longer U753.11 (4Y), U756.9 (3A)
- net V_HEND: now also U768.1 (1A), U711.7 (CEP); no longer U708.7 (CEP), U766.4 (2Y), U768.3 (2A)
- net V_HSA: now also U754.11 (4Y), U755.4 (2A); no longer U754.12 (4A), U754.6 (2Y)
- net V_HSB: now also U755.3 (1Y), U755.5 (2B); no longer U754.13 (4B), U754.8 (3Y)
- net V_HSYNC_A: now also U755.6 (2Y); no longer U754.11 (4Y)
- net V_HTC0: now also U707.15 (TC), U708.10 (CET); no longer U705.15 (TC), U768.1 (1A)
- net V_HVIS: now also U766.8 (4Y); no longer U766.12 (6Y)
- net V_I: now also U735.12 (4Y)
- net V_INC: now also U736.5 (CPU); no longer U735.5 (CPU)
- net V_LD7: now also U764.13 (4B), U706.9 (2Q); no longer U764.10 (3B)
- net V_OPR: now also U742.9 (2Q); no longer U741.9 (2Q)
- net V_OPR_D: now also U742.12 (2D); no longer U741.12 (2D)
- net V_OPW: now also U742.5 (1Q), U764.12 (4A), U768.9 (3A); no longer U741.5 (1Q), U764.9 (3A), U769.3 (2A)
- net V_PFCLK: now also U740.11 (2CLK)
- net V_PREF: now also U740.9 (2Q), U741.12 (2D); no longer U740.12 (2D)
- net V_PREFS: now also U741.9 (2Q); no longer U740.9 (2Q)
- net V_R: now also U735.9 (3Y)
- net V_RDCLK: now also U747.11 (CP); no longer U745.11 (CP)
- net V_RDD: now also U743.2 (1D); no longer U742.2 (1D)
- net V_RSCLK: now also U762.8 (3Y); no longer U756.11 (4Y)
- net V_RST: now also U739.14 (MR); no longer U735.14 (MR)
- net V_SL15: now also U756.8 (3Y), U762.4 (2A); no longer U756.3 (1Y), U762.9 (3A)
- net V_V0: now also U709.14 (Q0), U756.10 (3B); no longer U708.14 (Q0), U756.2 (1B)
- net V_V1: now also U709.13 (Q1), U756.5 (2B); no longer U708.13 (Q1), U755.13 (4B)
- net V_V2: now also U709.12 (Q2), U753.10 (3B); no longer U708.12 (Q2)
- net V_V3: now also U709.11 (Q3), U753.9 (3A); no longer U708.11 (Q3)
- net V_V32: now also U753.8 (3Y), U756.4 (2A), U768.13 (1C); no longer U755.12 (4A), U768.5 (2C)
- net V_V321: now also U756.6 (2Y), U756.9 (3A); no longer U755.11 (4Y), U756.1 (1A)
- net V_V4: now also U710.14 (Q0), U734.2 (P0); no longer U709.14 (Q0), U733.2 (P0)
- net V_V5: now also U710.13 (Q1), U755.13 (4B), U734.4 (P1); no longer U709.13 (Q1), U733.4 (P1), U755.5 (2B)
- net V_V6: now also U710.12 (Q2), U755.12 (4A), U734.6 (P2); no longer U709.12 (Q2), U733.6 (P2), U755.4 (2A)
- net V_V7: now also U710.11 (Q3), U755.10 (3B), U734.8 (P3); no longer U709.11 (Q3), U733.8 (P3), U755.2 (1B)
- net V_V8: now also U755.9 (3A), U711.14 (Q0), U734.11 (P4); no longer U710.14 (Q0), U733.11 (P4), U755.1 (1A)
- net V_V9: now also U761.12 (4A), U768.2 (1B), U711.13 (Q1), U734.13 (P5); no longer U710.13 (Q1), U733.13 (P5), U762.1 (1A), U768.4 (2B)
- net V_VBL: now also U761.11 (4Y), U762.2 (1B); no longer U762.3 (1Y)
- net V_VBQ: no longer U762.10 (3B)
- net V_VCTL: now also U743.9 (2Q), U748.2 (A0); no longer U742.9 (2Q)
- net V_VTC0: now also U709.15 (TC), U710.10 (CET); no longer U708.15 (TC), U709.10 (CET)
- net V_VTC1: now also U710.15 (TC), U711.10 (CET); no longer U709.15 (TC), U710.10 (CET)
- net V_WREQ: now also U740.5 (1Q), U741.2 (1D); no longer U740.2 (1D)
- net V_WREQS: now also U741.5 (1Q), U742.2 (1D); no longer U740.5 (1Q), U741.2 (1D)
- net V_WRP: now also U753.11 (4Y), U768.10 (3B); no longer U769.4 (2B)
- net ~{RESET}: now also U740.10 (~{2PRE}), U756.12 (4A), U743.1 (~{1CLR}), U743.13 (~{2CLR}); no longer U740.1 (~{1CLR}), U740.13 (~{2CLR}), U756.4 (2A)
- net ~{V_ADR0}: now also U767.4 (2Y), U768.11 (3C); no longer U767.8 (4Y), U769.13 (1C)
- net ~{V_CXEQ}: now also U733.19 (~{EQ})
- net ~{V_CYEQ}: now also U734.19 (~{EQ}); no longer U733.19 (~{EQ})
- net ~{V_FCLR}: now also U756.11 (4Y); no longer U756.6 (2Y)
- net ~{V_HEND}: now also U708.9 (~{PE}), U766.5 (3A); no longer U705.9 (~{PE}), U766.3 (2A), U768.12 (1Y)
- net ~{V_LD7}: now also U705.11 (Q3), U705.9 (~{PE}), U728.11 (CP), U732.9 (CP); no longer U761.2 (1B)
- net ~{V_OPR}: now also U740.13 (~{2CLR}), U742.8 (~{2Q}); no longer U741.8 (~{2Q})
- net ~{V_OPW}: now also U742.6 (~{1Q}); no longer U741.6 (~{1Q})
- net ~{V_RD1}: now also U748.1 (~{OE1})
- net ~{V_RD2}: now also U752.1 (~{OE1})
- net ~{V_RDA}: now also U747.1 (~{OE}); no longer U746.1 (~{OE})
- net ~{V_RDC}: now also U746.1 (~{OE}); no longer U745.1 (~{OE})
- net ~{V_RDDQ}: now also U743.6 (~{1Q}); no longer U742.6 (~{1Q})
- net ~{V_VLD}: now also U768.12 (1Y), U711.9 (~{PE}); no longer U708.9 (~{PE}), U768.6 (2Y)
- net ~{V_VTCU0}: now also U736.12 (~{TCU}), U737.5 (CPU); no longer U735.12 (~{TCU}), U736.5 (CPU)
- net ~{V_VTCU1}: now also U737.12 (~{TCU}), U738.5 (CPU); no longer U736.12 (~{TCU}), U737.5 (CPU)
- net ~{V_VTCU2}: now also U738.12 (~{TCU}), U739.5 (CPU); no longer U737.12 (~{TCU}), U738.5 (CPU)
- net ~{V_WE0}: now also U737.11 (~{PL}); no longer U735.11 (~{PL})
- net ~{V_WE1}: now also U740.3 (1CLK), U745.11 (CP)
- net ~{V_WE2}: now also U749.11 (CP)
- net ~{V_WE3}: now also U767.1 (1A); no longer U767.5 (3A)
- net ~{V_WEA}: now also U745.1 (~{OE}), U769.12 (1Y); no longer U744.1 (~{OE}), U769.6 (2Y)
- net ~{V_WEC}: now also U744.1 (~{OE}), U768.8 (3Y); no longer U769.12 (1Y)
- net ~{V_WINC}: now also U764.11 (4Y); no longer U764.8 (3Y)
- net ~{V_WO0}: now also U739.11 (~{PL}); no longer U737.11 (~{PL})
- net ~{V_WO1}: now also U743.11 (2CLK); no longer U742.11 (2CLK)
- net ~{V_WO2}: now also U750.11 (CP); no longer U749.11 (CP)
- net ~{V_WRCLR}: now also U740.1 (~{1CLR})
- net ~{V_WREQS}: now also U741.6 (~{1Q}); no longer U740.6 (~{1Q})
- net V_HSYNCP: now reaches U731.7 (Q1)
- net V_HSYNCP: now also U732.5 (D1)
- removed net N3691: U753.2 (1B), U766.8 (4Y)
- net N3699 renamed N3703
- net N3703: now also U761.9 (3A); no longer U753.5 (2B)
- removed net N3706: U754.3 (1Y), U754.4 (2A)
- net N3707 renamed N3698
- net N3698: now also U766.10 (5Y); no longer U767.4 (2Y)
- removed net N3711: U754.10 (3B), U768.8 (3Y)
- removed net N3714: U755.3 (1Y), U755.9 (3A)
- removed net N3715: U755.10 (3B), U755.6 (2Y)
- net N3716 renamed N3708
- net N3708: now also U756.1 (1A); no longer U762.2 (1B)
- net N3731 renamed N3725
- net N3725: now also U767.2 (1Y); no longer U767.6 (3Y)
- net N3732 renamed N3726
- net N3726: now also U756.13 (4B); no longer U756.5 (2B)
- removed net N3860: U756.10 (3B), U762.8 (3Y)
- net N4147: no longer names the net of U767.10 (5Y)
- net N4147: no longer U757.5 (2B)
- net N4151 renamed N4153
- net N4167 renamed N4169
- net N4327 renamed N4329
- removed net V_CLKA: U728.11 (CP), U731.9 (CP), U761.3 (1Y)
- removed net V_ENRS: U756.13 (4B), U756.8 (3Y)
- net V_H0: no longer names the net of U705.14 (Q0)
- net V_H0: no longer U766.5 (3A)
- net V_H1 renamed V_Q1
- net V_Q1: now also U753.13 (4B); no longer U766.9 (4A)
- new net N3695: U754.2 (1B), U761.3 (1Y)
- new net N3700: U754.12 (4A), U754.8 (3Y)
- new net N3701: U754.13 (4B), U766.12 (6Y)
- new net N3705: U755.2 (1B), U768.6 (2Y)
- new net N3854: U762.6 (2Y), U764.10 (3B)
- new net N4149: U757.5 (2B), U767.6 (3Y)
- new net N4152: U757.9 (3A), U765.1 (1Y)
- new net N4172: U758.10 (3B), U767.8 (4Y)
- new net V_BLANKP: U731.2 (Q0), U732.4 (D0)
- new net V_CURP: U731.15 (Q3), U732.13 (D3)
- new net V_Q15: U705.15 (TC), U706.12 (2D)
- new net V_Q2: U705.12 (Q2), U706.2 (1D)
- new net ~{V_ENRS}: U762.10 (3B), U764.8 (3Y)
- new net ~{V_VSYNCP}: U731.10 (Q2), U732.12 (D2)
- no-connect marks 76 -> 83
Other:
- moved on the sheet: U712, U713, U714, U715, U716, U717, U718, U735

Commit message: Kontrol birimi: mikrokod ve ALU ROM'ları yerine 74HC kapı devresi
CPU kartındaki 7 SST39SF010A (4 mikrokod, 3 ALU kod çözme ROM'u) kalktı. Yerine
board/kontrol.ts, cpu16.ucode'dan (tek kaynak) ve aluControl tablosundan çok seviyeli
bir 74HC devresi üretir ve Board API ile gerçek çipler olarak yerleştirir:

- Mikrokod: adım ve komut çözücüleri (74HC138; INT = 1 iken komutlar pasif, f3'e göre
  dallanan komutlara alt çözücü), aynı mikro programı çalıştıran (op, f3, COND)
  atomları, ortak alt kümeli VEYA ağı, sık kullanılan bitler için adım seçici
  (74HC151), adım 8..15 için SWI hattıyla açılan çözücü.
- ALU kod çözme: işlem çözücüleri (3 × 74HC138), işlem bitleri, h ve C terimleri.
- Yeni kapı çipleri: 74HC11, 74HC20, 74HC21, 74HC27, 74HC30 (veri sayfası pin sırası,
  doğruluk tablosu, zamanlama modeli, KiCad sembolü).
- Board: esnek yapıştırıcı kapılar (kartın diğer kapılarından sonra paketlenir, son
  çipi az dolu türü başka türlerin boş birimlerine taşır) ve defer(). Çözücüler eski
  ROM'ların yuvalarına (U1, U3, U5, U7, U10, U68–U71) oturur: kartın diğer bütün
  çiplerinin referansları değişmedi.
- CPU kartı 146 → 194 entegre; en kötü durumda CPU saati 860 → 824 ns (1,21 MHz),
  tipik 470 → 369 ns.
- Denklik testi (tests/kontrol.test.ts): kontrol birimi tek başına bir kartta, gerçek
  çip modelleriyle (LogicSim) 8192 mikrokod adresinin ve 128 ALU adresinin hepsinde
  tabloyla aynı kelimeyi verir.
- roms.ts, cpu16/roms/ ve "roms" komutu kalktı; "kontrol" komutu gömülü mikrokodu
  (micro/cpu16-ucode.ts) yeniler ve devreyi denetler. GateComputer ve GateMachine artık
  mikrokod istemez.
- CPU şeması A0'a sığsın diye dekuplaj kondansatörleri dar sütunlarda; KiCad dosyaları,
  BOM ve deney rehberlerinin otomatik bölümleri yeniden üretildi.

Co-Authored-By: Claude Opus 5.5 (1M context) <noreply@anthropic.com>
Claude-Session: https://claude.ai/code/session_018J8WVuECVRbQJyCbmF6Nsi
Connections:
- net N3695 renamed N3890
- net N3698 renamed N3893
- net N3700 renamed N3895
- net N3701 renamed N3896
- net N3703 renamed N3898
- net N3704 renamed N3899
- net N3705 renamed N3900
- net N3708 renamed N3903
- net N3709 renamed N3904
- net N3710 renamed N3905
- net N3725 renamed N3920
- net N3726 renamed N3921
- net N3854 renamed N4049
- net N4149 renamed N4344
- net N4150 renamed N4345
- net N4152 renamed N4347
- net N4153 renamed N4348
- net N4169 renamed N4364
- net N4170 renamed N4365
- net N4172 renamed N4367
- net N4329 renamed N4524
