File: cpu16/kicad/video/video.kicad_sch (KiCad schematic)
At the start: 148 parts, among them J701 CONN_VGA, J702 BACKPLANE_2x32, U701 74HC138, U702 74HC138, U703 74HC138, U704 74HC138, U705 74AC161, U706 74AC74, U707 74HC161, U708 74HC161, U709 74HC161, U710 74HC161, U711 74HC161, U712 74HC688, U713 74HC74, U714 74HC393, U715 74HC541, U716 74HC161, U717 74HC161, U718 74HC161, U719 74HC574, U720 74HC574, U721 74HC157, U722 74HC157, U723 74HC157, U724 62256, U725 62256, U726 74HC574, U727 74HC574, U728 74HC574, U729 SST39SF010A, U730 74HC166, U731 74HC175, U732 74HC175, U733 74HC688, U734 74HC688, U735 74HC157, U736 74HC193, U737 74HC193, U738 74HC193, U739 74HC193, U740 74HC74, U741 74HC74, U742 74HC74, U743 74HC74, U744 74HC574, U745 74HC574, U746 74HC574, U747 74HC574, U748 74HC541, U749 74HC574, U750 74HC574, U751 74HC541, U752 74HC541, U753 74HC08, U754 74HC08, U755 74HC08, U756 74HC08, U757 74HC08, U758 74HC08, U759 74HC08, U760 74HC08, U761 74HC32, U762 74HC32, U763 74HC32, U764 74HC00, U765 74HC02, U766 74HC04, U767 74HC04, U768 74HC10, U769 74HC10, X701 OSC_25M175

Commit message: Anakart yalnız yaygın parçalarla: 28C256 + 4 × 62256, kendin yap bellek kartı
AFU kararı: bilgisayar yalnız yaygın 7400 serisi lojikle ve iki bellek
çipiyle (62256, 28C256) kurulur.

Bellek kartı (31 → 34 entegre):
- SST39SF010A yerine 28C256 (32 KB, fiziksel 0x00000–0x07FFF, bank 0–1)
- AS6C4008 yerine 4 × 62256 (128 KB, 0x80000–0x9FFFF, bank 32–39)
- çip seçimi tek 74HC138; geri kalan bölgeler boş (0xFF, yazma yok sayılır)

Nadir parçalar çıktı:
- önbellek sayaçları 74HC590 → 74HC161 × 8 + 74HC541 × 4 (37 → 46)
- zamanlayıcı 74HC193 → 74HC161 (tümleyeni yukarı sayar)
- kesme öncelik kodlayıcısı 74HC148 → kapılar
- video adres sayacı (VADDR) 74HC193 → 74HC161 × 4 + yükleme bayrakları
- karakter ROM'u 28C256; yavaşlığı font register'ıyla bir aşamalık boru
  hattında karşılanır (V_H2 en kötü 262 ns, font yolu 199 ns ≤ 317,8);
  resim Machine ile aynı (video 69 → 73 entegre)
- 74HC166 kalır: 74HC165'in eşzamansız yüklemesi piksel saatine sığmaz

Kendin yap bellek kartı (kyb, 22 entegre): FF40–FF4F, 16 bayt, her bayt
bir 74HC574; 74HC138 çözücüler ve 74HC245 veri yolu tamponları. Machine
aygıtı, KiCad klasörü, kapı seviyesi kart Machine ile döngü döngüsüne aynı.

Machine'de At28c256 modeli (sayfa yazma, tBLC, yazma döngüsü, DATA
yoklaması, toggle biti, SDP); kapı seviyesi kartlar aynı modeli kullanır.
BIOS: F komutu korumalı sayfa yazmasıyla yalnız bank 1'e, I komutu yazma
korumasını gösterir, T bank 32–39'u sınar. Deney 8 programı 8 bank sayar,
boş bölgeleri denetler; Deney 14 programı ve testi eklendi.

Co-Authored-By: Claude Opus 5.5 (1M context) <noreply@anthropic.com>
Claude-Session: https://claude.ai/code/session_018J8WVuECVRbQJyCbmF6Nsi
Parts:
- removed U728, U744, U745, U746, U747: 74HC574, Package_DIP:DIP-20_W7.62mm, symbol cpu16:74HC574
- removed U729: SST39SF010A, Package_DIP:DIP-32_W15.24mm, symbol cpu16:SST39SF010A
- removed U730: 74HC166, Package_DIP:DIP-16_W7.62mm, symbol cpu16:74HC166
- removed U731, U732: 74HC175, Package_DIP:DIP-16_W7.62mm, symbol cpu16:74HC175
- removed U733, U734: 74HC688, Package_DIP:DIP-20_W7.62mm, symbol cpu16:74HC688
- removed U735: 74HC157, Package_DIP:DIP-16_W7.62mm, symbol cpu16:74HC157
- removed U736, U737, U738, U739: 74HC193, Package_DIP:DIP-16_W7.62mm, symbol cpu16:74HC193
- removed U740, U741, U742, U743: 74HC74, Package_DIP:DIP-14_W7.62mm, symbol cpu16:74HC74
- removed U748, U751: 74HC541, Package_DIP:DIP-20_W7.62mm, symbol cpu16:74HC541
- removed U753, U754, U755, U756: 74HC08, Package_DIP:DIP-14_W7.62mm, symbol cpu16:74HC08
- removed U761, U762, U763: 74HC32, Package_DIP:DIP-14_W7.62mm, symbol cpu16:74HC32
- removed U764: 74HC00, Package_DIP:DIP-14_W7.62mm, symbol cpu16:74HC00
- removed U765: 74HC02, Package_DIP:DIP-14_W7.62mm, symbol cpu16:74HC02
- removed U766, U767: 74HC04, Package_DIP:DIP-14_W7.62mm, symbol cpu16:74HC04
- removed U768, U769: 74HC10, Package_DIP:DIP-14_W7.62mm, symbol cpu16:74HC10
- added C719, C771, C772, C773, C774: C_100N, Capacitor_THT:C_Disc_D5.0mm_W2.5mm_P5.00mm, symbol cpu16:C_100N
- added U728: 28C256, Package_DIP:DIP-28_W15.24mm, symbol cpu16:28C256
- added U729, U730, U731, U748, U751, U753, U754: 74HC574, Package_DIP:DIP-20_W7.62mm, symbol cpu16:74HC574
- added U732: 74HC166, Package_DIP:DIP-16_W7.62mm, symbol cpu16:74HC166
- added U733, U734, U735: 74HC175, Package_DIP:DIP-16_W7.62mm, symbol cpu16:74HC175
- added U736, U737: 74HC688, Package_DIP:DIP-20_W7.62mm, symbol cpu16:74HC688
- added U738: 74HC157, Package_DIP:DIP-16_W7.62mm, symbol cpu16:74HC157
- added U739, U744, U745, U746, U747: 74HC74, Package_DIP:DIP-14_W7.62mm, symbol cpu16:74HC74
- added U740, U741, U742, U743: 74HC161, Package_DIP:DIP-16_W7.62mm, symbol cpu16:74HC161
- added U755, U756: 74HC541, Package_DIP:DIP-20_W7.62mm, symbol cpu16:74HC541
- added U761, U762, U763, U764: 74HC08, Package_DIP:DIP-14_W7.62mm, symbol cpu16:74HC08
- added U765, U766, U767: 74HC32, Package_DIP:DIP-14_W7.62mm, symbol cpu16:74HC32
- added U768: 74HC00, Package_DIP:DIP-14_W7.62mm, symbol cpu16:74HC00
- added U769: 74HC02, Package_DIP:DIP-14_W7.62mm, symbol cpu16:74HC02
- added U770, U771: 74HC04, Package_DIP:DIP-14_W7.62mm, symbol cpu16:74HC04
- added U773: 74HC10, Package_DIP:DIP-14_W7.62mm, symbol cpu16:74HC10
- U749: Gorev CURSOR_X (FF24) -> VDATA yazma verisi → renk şeridi
- U750: Gorev CURSOR_Y (FF25) -> VDATA ön okuma (karakter şeridi)
- U752: Gorev CURSOR_Y okuma -> VCTRL okuma (FF23)
- U757: Gorev yapıştırıcı: VRAM çıkışı kapalı: CPU yazıyor, imleç burada -> yapıştırıcı: karakter 98 / 99, VRAM yazma darbesi (p5–p6)
- U758: Gorev yapıştırıcı: renk 6, yeşil 2/3, VADDR artırma saati -> yapıştırıcı: hc ≥ 640 (yatay karartma), karakter 98: satır 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
- U759: Gorev yapıştırıcı: VADDR değişti: ön okuma iste, yazma isteği alı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 -> yapıştırıcı: alt 4 bit 2..13, karakter 82..93: HSYNC (96 pi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
- U760: Gorev yapıştırıcı: ön okuma latch saati (p7) -> yapıştırıcı: tarama satırı 14–15, karakter satırının son ta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
- U772: renamed from C719; value C_100N -> 74HC10; footprint Capacitor_THT:C_Disc_D5.0mm_W2.5mm_P5.00mm -> Package_DIP:DIP-14_W7.62mm; symbol cpu16:C_100N -> cpu16:74HC10; Gorev U718 dekuplaj -> yapıştırıcı: vc = 524 ve satır sonu: kare sonu, karakter şe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
Connections:
- net N4149 is gone; now on net V_H4: U757.5 (2B)
- net N4152 is gone; now on net V_V3: U757.9 (3A)
- net N4170 is gone; now on net N3698: U758.5 (2B)
- net N4172 is gone; now on net V_H7: U758.10 (3B)
- net A0: now also U769.9 (3B)
- net CLK: now also U747.3 (1CLK)
- net DE0: now also U750.19 (Q0), U740.3 (D0), U748.2 (D0), U751.19 (Q0), U753.2 (D0), U755.18 (Y0)
- net DE1: now also U750.18 (Q1), U740.4 (D1), U748.3 (D1), U751.18 (Q1), U753.3 (D1), U755.17 (Y1), U768.5 (2B)
- net DE2: now also U750.17 (Q2), U740.5 (D2), U748.4 (D2), U751.17 (Q2), U753.4 (D2), U755.16 (Y2)
- net DE3: now also U750.16 (Q3), U740.6 (D3), U748.5 (D3), U751.16 (Q3), U753.5 (D3), U755.15 (Y3)
- net DE4: now also U750.15 (Q4), U741.3 (D0), U748.6 (D4), U751.15 (Q4), U753.6 (D4), U755.14 (Y4)
- net DE5: now also U750.14 (Q5), U741.4 (D1), U748.7 (D5), U751.14 (Q5), U753.7 (D5), U755.13 (Y5)
- net DE6: now also U750.13 (Q6), U741.5 (D2), U748.8 (D6), U751.13 (Q6), U753.8 (D6), U755.12 (Y6)
- net DE7: now also U750.12 (Q7), U741.6 (D3), U748.9 (D7), U751.12 (Q7), U753.9 (D7), U755.11 (Y7)
- net DO0: now also U742.3 (D0), U747.12 (2D), U754.2 (D0), U756.18 (Y0); no longer U750.2 (D0)
- net DO1: now also U742.4 (D1), U754.3 (D1), U756.17 (Y1); no longer U750.3 (D1)
- net DO2: now also U742.5 (D2), U754.4 (D2), U756.16 (Y2); no longer U750.4 (D2)
- net DO3: now also U742.6 (D3), U754.5 (D3), U756.15 (Y3); no longer U750.5 (D3)
- net DO4: now also U743.3 (D0), U754.6 (D4), U756.14 (Y4); no longer U750.6 (D4)
- net DO5: now also U743.4 (D1), U754.7 (D5), U756.13 (Y5); no longer U750.7 (D5)
- net DO6: now also U743.5 (D2), U754.8 (D6), U756.12 (Y6); no longer U750.8 (D6)
- net DO7: now also U743.6 (D3), U754.9 (D7), U756.11 (Y7); no longer U750.9 (D7)
- net GND: now also U752.3 (A1), U752.4 (A2), U752.5 (A3), U752.6 (A4), U752.7 (A5), U752.8 (A6), U752.9 (A7), U772.7 (GND), C719.2, C771.2, C772.2, C773.2, C774.2, U728.1 (A14), U728.14 (GND), U728.2 (A12), U728.20 (~{CE}), U728.22 (~{OE}), U728.26 (A13), U729.1 (~{OE}), U729.10 (GND), U730.1 (~{OE}), U730.10 (GND), U731.1 (~{OE}), U731.10 (GND), U732.1 (DS), U732.6 (~{CE}), U732.8 (GND), U733.8 (GND), U734.8 (GND), U735.8 (GND), U736.1 (~{E}), U736.10 (GND), U736.17 (P7), U737.1 (~{E}), U737.10 (GND), U737.15 (P6), U737.17 (P7), U738.8 (GND), U739.12 (2D), U739.2 (1D), U739.7 (GND), U740.8 (GND), U741.8 (GND), U742.8 (GND), U743.8 (GND), U744.7 (GND), U745.7 (GND), U746.7 (GND), U747.7 (GND), U748.10 (GND), U751.10 (GND), U753.1 (~{OE}), U753.10 (GND), U754.1 (~{OE}), U754.10 (GND), U755.10 (GND), U755.19 (~{OE2}), U756.10 (GND), U756.19 (~{OE2}), U761.7 (GND), U762.7 (GND), U763.7 (GND), U764.10 (3B), U764.12 (4A), U764.13 (4B), U764.4 (2A), U764.5 (2B), U764.7 (GND), U764.9 (3A), U765.7 (GND), U766.7 (GND), U767.12 (4A), U767.13 (4B), U767.7 (GND), U768.7 (GND), U769.11 (4A), U769.12 (4B), U769.7 (GND), U770.7 (GND), U771.11 (5A), U771.13 (6A), U771.7 (GND), U771.9 (4A), U773.10 (3B), U773.11 (3C), U773.3 (2A), U773.4 (2B), U773.5 (2C), U773.7 (GND), U773.9 (3A); no longer U749.1 (~{OE}), U750.1 (~{OE}), U760.10 (3B), U760.12 (4A), U760.13 (4B), U760.4 (2A), U760.5 (2B), U760.9 (3A), U772.2
- net N3695: now also U758.2 (1B), U765.3 (1Y)
- net N3698: now also U770.8 (4Y)
- net N3700: now also U758.12 (4A), U758.8 (3Y)
- net N3701: now also U758.13 (4B), U770.10 (5Y)
- net N3703: now also U765.6 (2Y), U765.9 (3A)
- net N3704: now also U759.1 (1A), U765.8 (3Y)
- net N3705: now also U759.2 (1B), U772.6 (2Y)
- net N3708: now also U759.8 (3Y), U760.1 (1A)
- net N3709: now also U759.11 (4Y), U760.2 (1B)
- net N3710: now also U760.3 (1Y), U765.13 (4B)
- net N3725: now also U768.4 (2A), U770.12 (6Y)
- net N3726: now also U760.13 (4B), U768.6 (2Y)
- net N3854: now also U766.6 (2Y), U768.10 (3B)
- net VCC: now also U772.14 (VCC), C719.1, C771.1, C772.1, C773.1, C774.1, U728.27 (~{WE}), U728.28 (VCC), U729.20 (VCC), U730.20 (VCC), U731.20 (VCC), U732.16 (VCC), U732.9 (~{MR}), U733.1 (~{MR}), U733.16 (VCC), U734.1 (~{MR}), U734.16 (VCC), U735.1 (~{MR}), U735.16 (VCC), U736.20 (VCC), U737.20 (VCC), U738.16 (VCC), U739.14 (VCC), U740.10 (CET), U740.16 (VCC), U741.16 (VCC), U742.16 (VCC), U743.16 (VCC), U744.12 (2D), U744.14 (VCC), U744.2 (1D), U744.4 (~{1PRE}), U745.10 (~{2PRE}), U745.14 (VCC), U745.4 (~{1PRE}), U746.10 (~{2PRE}), U746.14 (VCC), U746.4 (~{1PRE}), U747.10 (~{2PRE}), U747.14 (VCC), U747.4 (~{1PRE}), U748.20 (VCC), U751.20 (VCC), U753.20 (VCC), U754.20 (VCC), U755.20 (VCC), U756.20 (VCC), U761.14 (VCC), U762.14 (VCC), U763.14 (VCC), U764.14 (VCC), U765.14 (VCC), U766.14 (VCC), U767.14 (VCC), U768.14 (VCC), U769.14 (VCC), U770.14 (VCC), U771.14 (VCC), U773.14 (VCC); no longer U772.1
- net VGA_HSYNC: now also U735.6 (~{Q1})
- net VGA_VSYNC: now also U735.10 (Q2)
- net VID_OSC: now also U732.7 (CP)
- net V_AD0: now also U749.19 (Q0), U751.2 (D0)
- net V_AD1: now also U749.18 (Q1), U751.3 (D1)
- net V_AD2: now also U749.17 (Q2), U751.4 (D2)
- net V_AD3: now also U749.16 (Q3), U751.5 (D3)
- net V_AD4: now also U749.15 (Q4), U751.6 (D4)
- net V_AD5: now also U749.14 (Q5), U751.7 (D5)
- net V_AD6: now also U749.13 (Q6), U751.8 (D6)
- net V_AD7: now also U749.12 (Q7), U751.9 (D7)
- net V_ADR0: now also U740.14 (Q0), U767.5 (2B), U771.1 (1A), U773.13 (1C)
- net V_ADR1: now also U740.13 (Q1)
- net V_ADR10: now also U742.12 (Q2)
- net V_ADR11: now also U742.11 (Q3)
- net V_ADR12: now also U743.14 (Q0)
- net V_ADR2: now also U740.12 (Q2)
- net V_ADR3: now also U740.11 (Q3)
- net V_ADR4: now also U741.14 (Q0)
- net V_ADR5: now also U741.13 (Q1)
- net V_ADR6: now also U741.12 (Q2)
- net V_ADR7: now also U741.11 (Q3)
- net V_ADR8: now also U742.14 (Q0)
- net V_ADR9: now also U742.13 (Q1)
- net V_AT0: now also U730.2 (D0)
- net V_AT1: now also U730.3 (D1)
- net V_AT2: now also U730.4 (D2)
- net V_AT3: now also U730.5 (D3)
- net V_AT4: now also U730.6 (D4)
- net V_AT5: now also U730.7 (D5)
- net V_AT6: now also U730.8 (D6)
- net V_AT7: now also U730.9 (D7)
- net V_ATD0: now also U731.19 (Q0), U738.3 (1I1)
- net V_ATD1: now also U731.18 (Q1), U738.6 (2I1)
- net V_ATD2: now also U731.17 (Q2), U738.10 (3I1)
- net V_ATD3: now also U731.16 (Q3), U738.13 (4I1)
- net V_ATD4: now also U731.15 (Q4), U738.2 (1I0)
- net V_ATD5: now also U731.14 (Q5), U738.5 (2I0)
- net V_ATD6: now also U731.13 (Q6), U738.11 (3I0)
- net V_ATD7: now also U731.12 (Q7), U738.14 (4I0)
- net V_B: now also U738.4 (1Y), U769.6 (2B)
- net V_BLANK: now also U733.4 (D0), U766.3 (1Y)
- net V_BLANKD: now also U735.2 (Q0), U738.15 (~{E})
- net V_BLANKP: now also U733.2 (Q0), U734.4 (D0)
- net V_BLINK: now also U771.3 (2A)
- net V_BROWN: now also U762.6 (2Y), U767.2 (1B), U771.5 (3A); no longer U758.6 (2Y)
- net V_CD0: now also U750.2 (D0), U748.19 (Q0)
- net V_CD1: now also U750.3 (D1), U748.18 (Q1)
- net V_CD2: now also U750.4 (D2), U748.17 (Q2)
- net V_CD3: now also U750.5 (D3), U748.16 (Q3)
- net V_CD4: now also U750.6 (D4), U748.15 (Q4)
- net V_CD5: now also U750.7 (D5), U748.14 (Q5)
- net V_CD6: now also U750.8 (D6), U748.13 (Q6)
- net V_CD7: now also U750.9 (D7), U748.12 (Q7)
- net V_CHR0: now also U728.6 (A4)
- net V_CHR1: now also U728.5 (A5)
- net V_CHR2: now also U728.4 (A6)
- net V_CHR3: now also U728.3 (A7)
- net V_CHR4: now also U728.25 (A8)
- net V_CHR5: now also U728.24 (A9)
- net V_CHR6: now also U728.21 (A10)
- net V_CHR7: now also U728.23 (A11)
- net V_CURD: now also U735.15 (Q3), U766.13 (4B)
- net V_CURP: now also U733.15 (Q3), U734.13 (D3)
- net V_CURR: now also U733.13 (D3), U761.11 (4Y); no longer U757.11 (4Y)
- net V_CX0: now also U736.3 (Q0), U753.19 (Q0), U755.2 (A0); no longer U749.19 (Q0)
- net V_CX1: now also U736.5 (Q1), U753.18 (Q1), U755.3 (A1); no longer U749.18 (Q1)
- net V_CX2: now also U736.7 (Q2), U753.17 (Q2), U755.4 (A2); no longer U749.17 (Q2)
- net V_CX3: now also U736.9 (Q3), U753.16 (Q3), U755.5 (A3); no longer U749.16 (Q3)
- net V_CX4: now also U736.12 (Q4), U753.15 (Q4), U755.6 (A4); no longer U749.15 (Q4)
- net V_CX5: now also U736.14 (Q5), U753.14 (Q5), U755.7 (A5); no longer U749.14 (Q5)
- net V_CX6: now also U736.16 (Q6), U753.13 (Q6), U755.8 (A6); no longer U749.13 (Q6)
- net V_CX7: now also U736.18 (Q7), U753.12 (Q7), U755.9 (A7); no longer U749.12 (Q7)
- net V_CY0: now also U737.3 (Q0), U754.19 (Q0), U756.2 (A0); no longer U750.19 (Q0), U752.2 (A0)
- net V_CY1: now also U737.5 (Q1), U754.18 (Q1), U756.3 (A1); no longer U750.18 (Q1), U752.3 (A1)
- net V_CY2: now also U737.7 (Q2), U754.17 (Q2), U756.4 (A2); no longer U750.17 (Q2), U752.4 (A2)
- net V_CY3: now also U737.9 (Q3), U754.16 (Q3), U756.5 (A3); no longer U750.16 (Q3), U752.5 (A3)
- net V_CY4: now also U737.12 (Q4), U754.15 (Q4), U756.6 (A4); no longer U750.15 (Q4), U752.6 (A4)
- net V_CY5: now also U737.14 (Q5), U754.14 (Q5), U756.7 (A5); no longer U750.14 (Q5), U752.7 (A5)
- net V_CY6: now also U737.16 (Q6), U754.13 (Q6), U756.8 (A6); no longer U750.13 (Q6), U752.8 (A6)
- net V_CY7: now also U737.18 (Q7), U754.12 (Q7), U756.9 (A7); no longer U750.12 (Q7), U752.9 (A7)
- net V_FD0: now also U728.11 (IO0), U729.2 (D0)
- net V_FD1: now also U728.12 (IO1), U729.3 (D1)
- net V_FD2: now also U728.13 (IO2), U729.4 (D2)
- net V_FD3: now also U728.15 (IO3), U729.5 (D3)
- net V_FD4: now also U728.16 (IO4), U729.6 (D4)
- net V_FD5: now also U728.17 (IO5), U729.7 (D5)
- net V_FD6: now also U728.18 (IO6), U729.8 (D6)
- net V_FD7: now also U728.19 (IO7), U729.9 (D7)
- net V_FGSEL: now also U738.1 (S), U766.11 (4Y)
- net V_G: now also U738.7 (2Y), U762.2 (1B), U762.9 (3A); no longer U758.2 (1B), U758.9 (3A)
- net V_GH: now also U762.8 (3Y); no longer U758.8 (3Y)
- net V_GL: now also U767.3 (1Y)
- net V_H2: now also U757.12 (4A), U729.11 (CP), U730.11 (CP), U733.9 (CP), U734.9 (CP), U746.11 (2CLK), U746.3 (1CLK), U761.2 (1B), U766.9 (3A), U770.1 (1A); no longer U757.2 (1B)
- net V_H2N: now also U745.11 (2CLK), U745.3 (1CLK), U770.2 (1Y)
- net V_H3: now also U736.2 (P0), U768.2 (1B), U770.9 (4A)
- net V_H4: now also U772.3 (2A), U736.4 (P1), U765.4 (2A)
- net V_H5: now also U772.4 (2B), U736.6 (P2), U765.5 (2B)
- net V_H6: now also U772.5 (2C), U736.8 (P3), U765.10 (3B)
- net V_H7: now also U736.11 (P4), U765.2 (1B)
- net V_H8: now also U757.1 (1A), U736.13 (P5), U765.1 (1A), U770.11 (5A)
- net V_H89: now also U757.3 (1Y), U757.4 (2A)
- net V_H9: now also U757.2 (1B), U758.1 (1A), U758.9 (3A), U736.15 (P6)
- net V_H984: now also U757.6 (2Y), U758.4 (2A), U768.1 (1A)
- net V_HBL: now also U758.3 (1Y), U766.1 (1A), U770.5 (3A)
- net V_HC98: now also U758.6 (2Y), U768.9 (3A)
- net V_HEND: now also U772.1 (1A), U770.4 (2Y)
- net V_HSA: now also U758.11 (4Y), U759.4 (2A)
- net V_HSB: now also U759.3 (1Y), U759.5 (2B)
- net V_HSYNCP: now also U733.7 (Q1), U734.5 (D1)
- net V_HSYNC_A: now also U759.6 (2Y), U733.5 (D1)
- net V_HVIS: now also U770.6 (3Y)
- net V_I: now also U738.12 (4Y), U767.1 (1A), U769.5 (2A)
- net V_INC: now also U762.11 (4Y), U763.5 (2B); no longer U758.11 (4Y), U759.5 (2B)
- net V_LD7: now also U764.2 (1B), U768.13 (4B); no longer U760.2 (1B)
- net V_OPR: now also U746.9 (2Q), U764.1 (1A); no longer U760.1 (1A)
- net V_OPR_D: now also U746.12 (2D), U763.11 (4Y); no longer U759.11 (4Y)
- net V_OPW: now also U772.9 (3A), U746.5 (1Q), U761.1 (1A), U768.12 (4A), U773.1 (1A); no longer U757.1 (1A)
- net V_PFCLK: now also U739.11 (2CLK), U739.3 (1CLK), U740.2 (CP), U741.2 (CP), U742.2 (CP), U743.2 (CP), U744.11 (2CLK), U763.6 (2Y); no longer U759.6 (2Y)
- net V_PIX: now also U732.13 (Q7), U766.12 (4A)
- net V_PREF: now also U744.9 (2Q), U745.12 (2D)
- net V_PREFS: now also U745.9 (2Q), U763.12 (4A); no longer U759.12 (4A)
- net V_Q1: now also U757.13 (4B)
- net V_R: now also U738.9 (3Y), U762.1 (1A); no longer U758.1 (1A)
- net V_RDCLK: now also U750.11 (CP), U751.11 (CP), U764.3 (1Y); no longer U760.3 (1Y)
- net V_RDD: now also U747.2 (1D), U769.10 (3Y)
- net V_RSCLK: now also U766.8 (3Y)
- net V_SL15: now also U760.8 (3Y), U766.4 (2A)
- net V_SOE: now also U761.3 (1Y); no longer U757.3 (1Y)
- net V_V0: now also U760.10 (3B), U728.10 (A0)
- net V_V1: now also U760.5 (2B), U728.9 (A1)
- net V_V2: now also U757.10 (3B), U728.8 (A2)
- net V_V3: now also U728.7 (A3)
- net V_V32: now also U757.8 (3Y), U760.4 (2A), U772.13 (1C)
- net V_V321: now also U760.6 (2Y), U760.9 (3A), U761.10 (3B); no longer U757.10 (3B)
- net V_V4: now also U737.2 (P0)
- net V_V5: now also U759.13 (4B), U737.4 (P1)
- net V_V6: now also U759.12 (4A), U737.6 (P2)
- net V_V7: now also U759.10 (3B), U737.8 (P3)
- net V_V8: now also U759.9 (3A), U737.11 (P4)
- net V_V9: now also U772.2 (1B), U737.13 (P5), U765.12 (4A)
- net V_VBL: now also U765.11 (4Y), U766.2 (1B), U766.5 (2B)
- net V_VCTL: now also U752.2 (A0), U747.9 (2Q), U761.4 (2A); no longer U757.4 (2A)
- net V_WREQ: now also U744.5 (1Q), U745.2 (1D)
- net V_WREQS: now also U745.5 (1Q), U746.2 (1D)
- net V_WRP: now also U757.11 (4Y), U772.10 (3B), U773.2 (1B)
- net ~{RESET}: now also U760.12 (4A), U739.1 (~{1CLR}), U739.13 (~{2CLR}), U740.1 (~{MR}), U741.1 (~{MR}), U742.1 (~{MR}), U743.1 (~{MR}), U744.10 (~{2PRE}), U745.1 (~{1CLR}), U745.13 (~{2CLR}), U746.1 (~{1CLR}), U746.13 (~{2CLR}), U747.1 (~{1CLR}), U747.13 (~{2CLR}), U763.10 (3B); no longer U759.10 (3B)
- net ~{V_ADR0}: now also U772.11 (3C), U767.10 (3B), U771.2 (1Y)
- net ~{V_CXEQ}: now also U736.19 (~{EQ}), U769.2 (1A)
- net ~{V_CYEQ}: now also U737.19 (~{EQ}), U769.3 (1B)
- net ~{V_ENRS}: now also U766.10 (3B), U768.8 (3Y)
- net ~{V_FCLR}: now also U760.11 (4Y)
- net ~{V_HEND}: now also U768.3 (1Y), U770.3 (2A)
- net ~{V_LD7}: now also U731.11 (CP), U732.15 (~{PE}), U735.9 (CP)
- net ~{V_OPR}: now also U744.13 (~{2CLR}), U746.8 (~{2Q})
- net ~{V_OPW}: now also U746.6 (~{1Q}), U763.9 (3A); no longer U759.9 (3A)
- net ~{V_RD1}: now also U752.1 (~{OE1}), U767.4 (2A), U767.9 (3A), U769.8 (3A)
- net ~{V_RD2}: now also U755.1 (~{OE1}), U756.1 (~{OE1}); no longer U752.1 (~{OE1})
- net ~{V_RDA}: now also U751.1 (~{OE}), U767.8 (3Y)
- net ~{V_RDC}: now also U750.1 (~{OE}), U767.6 (2Y)
- net ~{V_RDDQ}: now also U747.6 (~{1Q}), U762.12 (4A); no longer U758.12 (4A)
- net ~{V_VLD}: now also U772.12 (1Y)
- net ~{V_VSYNCP}: now also U733.10 (Q2), U734.12 (D2)
- net ~{V_VSYNC_A}: now also U733.12 (D2)
- net ~{V_WE0}: now also U739.4 (~{1PRE}), U763.1 (1A); no longer U759.1 (1A)
- net ~{V_WE1}: now also U749.11 (CP), U744.3 (1CLK), U748.11 (CP)
- net ~{V_WE2}: now also U753.11 (CP); no longer U749.11 (CP)
- net ~{V_WE3}: now also U770.13 (6A)
- net ~{V_WEA}: now also U749.1 (~{OE}), U773.12 (1Y)
- net ~{V_WEC}: now also U772.8 (3Y), U748.1 (~{OE})
- net ~{V_WINC}: now also U762.13 (4B), U768.11 (4Y); no longer U758.13 (4B)
- net ~{V_WO0}: now also U739.10 (~{2PRE}), U763.2 (1B); no longer U759.2 (1B)
- net ~{V_WO1}: now also U747.11 (2CLK)
- net ~{V_WO2}: now also U754.11 (CP); no longer U750.11 (CP)
- net ~{V_WRCLR}: now also U744.1 (~{1CLR}), U763.8 (3Y); no longer U759.8 (3Y)
- net ~{V_WREQS}: now also U745.6 (~{1Q}), U763.13 (4B); no longer U759.13 (4B)
- removed net N4150: U757.12 (4A), U757.6 (2Y)
- removed net N4153: U757.13 (4B), U757.8 (3Y)
- removed net N4169: U758.3 (1Y), U758.4 (2A)
- removed net N4329: U759.3 (1Y), U759.4 (2A)
- new net N4207: U761.5 (2B), U771.4 (2Y)
- new net N4208: U761.12 (4A), U761.6 (2Y)
- new net N4210: U761.9 (3A), U769.1 (1Y)
- new net N4211: U761.13 (4B), U761.8 (3Y)
- new net N4227: U762.3 (1Y), U762.4 (2A)
- new net N4228: U762.5 (2B), U769.4 (2Y)
- new net N4230: U762.10 (3B), U771.6 (3Y)
- new net N4240: U763.3 (1Y), U763.4 (2A)
- new net V_AT20: U730.19 (Q0), U731.2 (D0)
- new net V_AT21: U730.18 (Q1), U731.3 (D1)
- new net V_AT22: U730.17 (Q2), U731.4 (D2)
- new net V_AT23: U730.16 (Q3), U731.5 (D3)
- new net V_AT24: U730.15 (Q4), U731.6 (D4)
- new net V_AT25: U730.14 (Q5), U731.7 (D5)
- new net V_AT26: U730.13 (Q6), U731.8 (D6)
- new net V_AT27: U730.12 (Q7), U731.9 (D7)
- new net V_ATC0: U740.15 (TC), U741.10 (CET)
- new net V_ATC1: U741.15 (TC), U742.10 (CET)
- new net V_ATC2: U742.15 (TC), U743.10 (CET)
- new net V_BLANKQ: U734.2 (Q0), U735.4 (D0)
- new net V_CURQ: U734.15 (Q3), U735.13 (D3)
- new net V_FP0: U729.19 (Q0), U732.2 (D0)
- new net V_FP1: U729.18 (Q1), U732.3 (D1)
- new net V_FP2: U729.17 (Q2), U732.4 (D2)
- new net V_FP3: U729.16 (Q3), U732.5 (D3)
- new net V_FP4: U729.15 (Q4), U732.10 (D4)
- new net V_FP5: U729.14 (Q5), U732.11 (D5)
- new net V_FP6: U729.13 (Q6), U732.12 (D6)
- new net V_FP7: U729.12 (Q7), U732.14 (D7)
- new net V_HSYNCQ: U734.7 (Q1), U735.5 (D1)
- new net ~{V_LHI}: U739.8 (~{2Q}), U740.7 (CEP), U741.7 (CEP), U742.9 (~{PE}), U743.9 (~{PE})
- new net ~{V_LLO}: U739.6 (~{1Q}), U740.9 (~{PE}), U741.9 (~{PE}), U742.7 (CEP), U743.7 (CEP)
- new net ~{V_VSYNCQ}: U734.10 (Q2), U735.12 (D2)
- no-connect marks 83 -> 84
