File: cpu16/kicad/prog/prog.kicad_sch (KiCad schematic)
At the start: 8 parts, among them U1 74HC595, U2 74HC595, U3 SST39SF010A

Commit message: Programlayıcı 28C256 için: korumalı sayfa yazma, DATA yoklaması, SDP
- Arduino taslağı: Intel HEX kaydı sayfa parçalarına bölünür, her parça
  bir korumalı sayfa yazmasıdır (AA 55 A0 + baytlar, tBLC içinde), sonra
  D7 yoklamasıyla beklenir; zaten aynı olan parçalar atlanır. SDP sorgu,
  aç ve kapat komutları; 28C256 dışındaki adresler reddedilir.
- yaz.py: --koruma, --koruma-ac, --koruma-kapat; --sil ve --id artık
  gerekmez (uyarı verir).
- Kart: 2 × 74HC595 + ZIF-28; KiCad şeması yeniden üretildi.
- Test: taslak gerçek kapı seviyesi kartla ve 28C256 modeliyle çalışır;
  pin işlemleri ve gecikmeler zaman olarak sayılır (sayfa penceresi,
  yazma döngüsü, zaman aşımı sınanır).
- Deney 3 rehberi yeni programlayıcıya göre yazıldı.

Co-Authored-By: Claude Opus 5.5 (1M context) <noreply@anthropic.com>
Claude-Session: https://claude.ai/code/session_018J8WVuECVRbQJyCbmF6Nsi
Parts:
- removed U3: SST39SF010A, Package_DIP:DIP-32_W15.24mm_Socket, symbol cpu16:SST39SF010A
- added U3: 28C256, Package_DIP:DIP-28_W15.24mm_Socket, symbol cpu16:28C256
- U2: Gorev adres A8..A15 (zincirin ikincisi) -> adres A8..A14 (zincirin ikincisi)
Connections:
- net FA0: now also U3.10 (A0)
- net FA1: now also U3.9 (A1)
- net FA10: now also U3.21 (A10)
- net FA11: now also U3.23 (A11)
- net FA12: now also U3.2 (A12)
- net FA13: now also U3.26 (A13)
- net FA14: now also U3.1 (A14)
- net FA2: now also U3.8 (A2)
- net FA3: now also U3.7 (A3)
- net FA4: now also U3.6 (A4)
- net FA5: now also U3.5 (A5)
- net FA6: now also U3.4 (A6)
- net FA7: now also U3.3 (A7)
- net FA8: now also U3.25 (A8)
- net FA9: now also U3.24 (A9)
- net FD0: now also U3.11 (IO0)
- net FD1: now also U3.12 (IO1)
- net FD2: now also U3.13 (IO2)
- net FD3: now also U3.15 (IO3)
- net FD4: now also U3.16 (IO4)
- net FD5: now also U3.17 (IO5)
- net FD6: now also U3.18 (IO6)
- net FD7: now also U3.19 (IO7)
- net GND: now also U3.14 (GND)
- net VCC: now also U3.28 (VCC)
- net ~{FCE}: now also U3.20 (~{CE})
- net ~{FOE}: now also U3.22 (~{OE})
- net ~{FWE}: now also U3.27 (~{WE})
- net FA15: no longer names the net of U2.7 (Q7)
- net FA16: no longer names the net of A1.19 (A0)
Other:
- title: CPU16 — Flash programlayıcı (Arduino Nano + 2 × 74HC595) -> CPU16 — EEPROM programlayıcı (Arduino Nano + 2 × 74HC595)
Changed lines of the file:
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@@
 (kicad_sch (version 20230121) (generator cpu16_board)
   (paper "A3")
-  (title_block (title "CPU16 — Flash programlayıcı (Arduino Nano + 2 × 74HC595)") (date "2026-10-11") (rev "1") (company "CPU16") (comment 1 "Bu dosya cpu16/board kaynak kodundan üretildi: npm run cpu16 -- board kicad"))
+  (title_block (title "CPU16 — EEPROM programlayıcı (Arduino Nano + 2 × 74HC595)") (date "2026-10-11") (rev "1") (company "CPU16") (comment 1 "Bu dosya cpu16/board kaynak kodundan üretildi: npm run cpu16 -- board kicad"))
   (symbol (lib_id "cpu16:74HC595") (at 55.88 66.04 0) (unit 1)
     (in_bom yes) (on_board yes) (dnp no)
@@
     (property "Footprint" "Package_DIP:DIP-16_W7.62mm" (at 55.88 114.3 0) (effects (font (size 1.27 1.27)) hide))
     (property "Datasheet" "" (at 55.88 114.3 0) (effects (font (size 1.27 1.27)) hide))
-    (property "Gorev" "adres A8..A15 (zincirin ikincisi)" (at 55.88 114.3 0) (effects (font (size 1.27 1.27)) hide))
+    (property "Gorev" "adres A8..A14 (zincirin ikincisi)" (at 55.88 114.3 0) (effects (font (size 1.27 1.27)) hide))
     (pin "1")
     (pin "2")
@@
     (instances (project "prog" (path "/3216aaaf-0000-4000-8000-000000000001" (reference "U2") (unit 1))))
   )
-  (symbol (lib_id "cpu16:SST39SF010A") (at 55.88 177.8 0) (unit 1)
+  (symbol (lib_id "cpu16:28C256") (at 55.88 172.72 0) (unit 1)
     (in_bom yes) (on_board yes) (dnp no)
     (property "Reference" "U3" (at 55.88 146.05 0) (effects (font (size 1.27 1.27))))
-    (property "Value" "SST39SF010A" (at 55.88 209.55 0) (effects (font (size 1.27 1.27))))
-    (property "Footprint" "Package_DIP:DIP-32_W15.24mm_Socket" (at 55.88 177.8 0) (effects (font (size 1.27 1.27)) hide))
-    (property "Datasheet" "" (at 55.88 177.8 0) (effects (font (size 1.27 1.27)) hide))
-    (property "Gorev" "programlanan Flash (ZIF soket)" (at 55.88 177.8 0) (effects (font (size 1.27 1.27)) hide))
+    (property "Value" "28C256" (at 55.88 199.39 0) (effects (font (size 1.27 1.27))))
+    (property "Footprint" "Package_DIP:DIP-28_W15.24mm_Socket" (at 55.88 172.72 0) (effects (font (size 1.27 1.27)) hide))
+    (property "Datasheet" "" (at 55.88 172.72 0) (effects (font (size 1.27 1.27)) hide))
+    (property "Gorev" "programlanan EEPROM (ZIF-28 soket)" (at 55.88 172.72 0) (effects (font (size 1.27 1.27)) hide))
     (pin "1")
     (pin "2")
@@
     (pin "27")
     (pin "28")
-    (pin "29")
-    (pin "30")
-    (pin "31")
-    (pin "32")
     (instances (project "prog" (path "/3216aaaf-0000-4000-8000-000000000001" (reference "U3") (unit 1))))
   )
@@
   (label "FA13" (at 66.04 111.76 0) (fields_autoplaced) (effects (font (size 1.27 1.27)) (justify left bottom)))
   (label "FA14" (at 66.04 114.3 0) (fields_autoplaced) (effects (font (size 1.27 1.27)) (justify left bottom)))
-  (label "FA15" (at 66.04 116.84 0) (fields_autoplaced) (effects (font (size 1.27 1.27)) (justify left bottom)))
+  (no_connect (at 66.04 116.84))
   (no_connect (at 66.04 119.38))
   (label "FA8" (at 66.04 121.92 0) (fields_autoplaced) (effects (font (size 1.27 1.27)) (justify left bottom)))
   (label "GND" (at 55.88 132.08 270) (fields_autoplaced) (effects (font (size 1.27 1.27)) (justify right bottom)))
   (label "VCC" (at 55.88 96.52 90) (fields_autoplaced) (effects (font (size 1.27 1.27)) (justify left bottom)))
-  (no_connect (at 45.72 149.86))
-  (label "FA16" (at 45.72 152.4 180) (fields_autoplaced) (effects (font (size 1.27 1.27)) (justify right bottom)))
-  (label "FA15" (at 45.72 154.94 180) (fields_autoplaced) (effects (font (size 1.27 1.27)) (justify right bottom)))
-  (label "FA12" (at 45.72 157.48 180) (fields_autoplaced) (effects (font (size 1.27 1.27)) (justify right bottom)))
-  (label "FA7" (at 45.72 160.02 180) (fields_autoplaced) (effects (font (size 1.27 1.27)) (justify right bottom)))
-  (label "FA6" (at 45.72 162.56 180) (fields_autoplaced) (effects (font (size 1.27 1.27)) (justify right bottom)))
-  (label "FA5" (at 45.72 165.1 180) (fields_autoplaced) (effects (font (size 1.27 1.27)) (justify right bottom)))
-  (label "FA4" (at 45.72 167.64 180) (fields_autoplaced) (effects (font (size 1.27 1.27)) (justify right bottom)))
-  (label "FA3" (at 45.72 170.18 180) (fields_autoplaced) (effects (font (size 1.27 1.27)) (justify right bottom)))
-  (label "FA2" (at 45.72 172.72 180) (fields_autoplaced) (effects (font (size 1.27 1.27)) (justify right bottom)))
-  (label "FA1" (at 45.72 175.26 180) (fields_autoplaced) (effects (font (size 1.27 1.27)) (justify right bottom)))
-  (label "FA0" (at 45.72 177.8 180) (fields_autoplaced) (effects (font (size 1.27 1.27)) (justify right bottom)))
-  (label "~{FCE}" (at 45.72 180.34 180) (fields_autoplaced) (effects (font (size 1.27 1.27)) (justify right bottom)))
-  (label "FA10" (at 45.72 182.88 180) (fields_autoplaced) (effects (font (size 1.27 1.27)) (justify right bottom)))
-  (label "~{FOE}" (at 45.72 185.42 180) (fields_autoplaced) (effects (font (size 1.27 1.27)) (justify right bottom)))
-  (label "FA11" (at 45.72 187.96 180) (fields_autoplaced) (effects (font (size 1.27 1.27)) (justify right bottom)))
-  (label "FA9" (at 45.72 190.5 180) (fields_autoplaced) (effects (font (size 1.27 1.27)) (justify right bottom)))
-  (label "FA8" (at 45.72 193.04 180) (fields_autoplaced) (effects (font (size 1.27 1.27)) (justify right bottom)))
-  (label "FA13" (at 45.72 195.58 180) (fields_autoplaced) (effects (font (size 1.27 1.27)) (justify right bottom)))
-  (label "FA14" (at 45.72 198.12 180) (fields_autoplaced) (effects (font (size 1.27 1.27)) (justify right bottom)))
-  (no_connect (at 45.72 200.66))
-  (label "~{FWE}" (at 45.72 203.2 180) (fields_autoplaced) (effects (font (size 1.27 1.27)) (justify right bottom)))
+  (label "FA14" (at 45.72 149.86 180) (fields_autoplaced) (effects (font (size 1.27 1.27)) (justify right bottom)))
+  (label "FA12" (at 45.72 152.4 180) (fields_autoplaced) (effects (font (size 1.27 1.27)) (justify right bottom)))
+  (label "FA7" (at 45.72 154.94 180) (fields_autoplaced) (effects (font (size 1.27 1.27)) (justify right bottom)))
+  (label "FA6" (at 45.72 157.48 180) (fields_autoplaced) (effects (font (size 1.27 1.27)) (justify right bottom)))
+  (label "FA5" (at 45.72 160.02 180) (fields_autoplaced) (effects (font (size 1.27 1.27)) (justify right bottom)))
+  (label "FA4" (at 45.72 162.56 180) (fields_autoplaced) (effects (font (size 1.27 1.27)) (justify right bottom)))
+  (label "FA3" (at 45.72 165.1 180) (fields_autoplaced) (effects (font (size 1.27 1.27)) (justify right bottom)))
+  (label "FA2" (at 45.72 167.64 180) (fields_autoplaced) (effects (font (size 1.27 1.27)) (justify right bottom)))
+  (label "FA1" (at 45.72 170.18 180) (fields_autoplaced) (effects (font (size 1.27 1.27)) (justify right bottom)))
+  (label "FA0" (at 45.72 172.72 180) (fields_autoplaced) (effects (font (size 1.27 1.27)) (justify right bottom)))
+  (label "~{FCE}" (at 45.72 175.26 180) (fields_autoplaced) (effects (font (size 1.27 1.27)) (justify right bottom)))
+  (label "FA10" (at 45.72 177.8 180) (fields_autoplaced) (effects (font (size 1.27 1.27)) (justify right bottom)))
+  (label "~{FOE}" (at 45.72 180.34 180) (fields_autoplaced) (effects (font (size 1.27 1.27)) (justify right bottom)))
+  (label "FA11" (at 45.72 182.88 180) (fields_autoplaced) (effects (font (size 1.27 1.27)) (justify right bottom)))
+  (label "FA9" (at 45.72 185.42 180) (fields_autoplaced) (effects (font (size 1.27 1.27)) (justify right bottom)))
+  (label "FA8" (at 45.72 187.96 180) (fields_autoplaced) (effects (font (size 1.27 1.27)) (justify right bottom)))
+  (label "FA13" (at 45.72 190.5 180) (fields_autoplaced) (effects (font (size 1.27 1.27)) (justify right bottom)))
+  (label "~{FWE}" (at 45.72 193.04 180) (fields_autoplaced) (effects (font (size 1.27 1.27)) (justify right bottom)))
   (label "FD0" (at 66.04 149.86 0) (fields_autoplaced) (effects (font (size 1.27 1.27)) (justify left bottom)))
   (label "FD1" (at 66.04 152.4 0) (fields_autoplaced) (effects (font (size 1.27 1.27)) (justify left bottom)))
@@
   (label "FD6" (at 66.04 165.1 0) (fields_autoplaced) (effects (font (size 1.27 1.27)) (justify left bottom)))
   (label "FD7" (at 66.04 167.64 0) (fields_autoplaced) (effects (font (size 1.27 1.27)) (justify left bottom)))
-  (label "GND" (at 55.88 210.82 270) (fields_autoplaced) (effects (font (size 1.27 1.27)) (justify right bottom)))
+  (label "GND" (at 55.88 200.66 270) (fields_autoplaced) (effects (font (size 1.27 1.27)) (justify right bottom)))
   (label "VCC" (at 55.88 144.78 90) (fields_autoplaced) (effects (font (size 1.27 1.27)) (justify left bottom)))
   (no_connect (at 114.3 53.34))
@@
   (label "FD7" (at 114.3 71.12 180) (fields_autoplaced) (effects (font (size 1.27 1.27)) (justify right bottom)))
   (no_connect (at 114.3 73.66))
-  (label "FA16" (at 114.3 76.2 180) (fields_autoplaced) (effects (font (size 1.27 1.27)) (justify right bottom)))
+  (no_connect (at 114.3 76.2))
   (label "~{FWE}" (at 114.3 78.74 180) (fields_autoplaced) (effects (font (size 1.27 1.27)) (justify right bottom)))
   (no_connect (at 114.3 81.28))
