File: cpu16/kicad/hesap/hesap-onluk-kalan.kicad_sch (KiCad schematic)
At the start: 24 parts, among them U173 74HC283, U174 74HC283, U175 74HC283, U176 74HC283, U177 74HC283, U178 74HC283, U179 74HC283, U180 74HC08, U181 74HC08, U182 74HC32, U183 74HC32, U184 74HC32

Commit message: Hesap makinesi: eksi işareti sonucun solunda, lamba testinde de yanar; HATA LED'i göstergelerin yanında
- işaret hanesi (DS7) sonucun hanelerinden önce yerleşir: 3D kartta ve
  şemada en solda
- ISARET_g = NEG + lamba testi (boş kapı birimleriyle, çip sayısı aynı)
- HATA LED'i Bölme bloğundan "Gösterge: Sonuç" bloğuna
- rehber ve tasarım belgesi güncellendi

Co-Authored-By: Claude Opus 5.5 (1M context) <noreply@anthropic.com>
Claude-Session: https://claude.ai/code/session_018J8WVuECVRbQJyCbmF6Nsi
Connections:
- net N3066 is gone; now on net N3065: U173.2 (B2), U173.6 (B1), U180.3 (1Y)
- net N3098 is gone; now on net N3097: U180.6 (2Y), U182.10 (3B)
- net N3131 is gone; now on net N3130: U180.8 (3Y), U183.2 (1B)
- net N3164 is gone; now on net N3163: U180.11 (4Y), U183.10 (3B)
- net N3197 is gone; now on net N3196: U177.2 (B2), U177.6 (B1), U181.3 (1Y)
- net N3229 is gone; now on net N3228: U181.6 (2Y), U184.5 (2B)
- net N3262 is gone; now on net N3261: U181.8 (3Y), U184.13 (4B)
- net N3065: no longer U180.2 (1B), U182.3 (1Y)
- net N3097: no longer U180.5 (2B), U182.6 (2Y)
- net N3130: no longer U180.10 (3B), U182.11 (4Y)
- net N3163: no longer U180.13 (4B), U183.6 (2Y)
- net N3196: no longer U181.2 (1B), U183.11 (4Y)
- net N3228: no longer U181.5 (2B), U184.3 (1Y)
- net N3261: no longer U181.10 (3B), U184.8 (3Y)
- new net N3064: U180.2 (1B), U182.3 (1Y)
- new net N3096: U180.5 (2B), U182.6 (2Y)
- new net N3129: U180.10 (3B), U182.11 (4Y)
- new net N3162: U180.13 (4B), U183.6 (2Y)
- new net N3195: U181.2 (1B), U183.11 (4Y)
- new net N3227: U181.5 (2B), U184.3 (1Y)
- new net N3260: U181.10 (3B), U184.8 (3Y)
