File: cpu16/kicad/hesap/hesap-onluk-sonuc.kicad_sch (KiCad schematic)
At the start: 116 parts, among them U115 74HC283, U116 74HC283, U117 74HC283, U118 74HC283, U119 74HC283, U120 74HC283, U121 74HC283, U122 74HC283, U123 74HC283, U124 74HC283, U125 74HC283, U126 74HC283, U127 74HC283, U128 74HC283, U129 74HC283, U130 74HC283, U131 74HC283, U132 74HC283, U133 74HC283, U134 74HC283, U135 74HC283, U136 74HC283, U137 74HC283, U138 74HC283, U139 74HC283, U140 74HC283, U141 74HC283, U142 74HC283, U143 74HC283, U144 74HC283, U145 74HC283, U146 74HC283, U147 74HC283, U148 74HC08, U149 74HC08, U150 74HC08, U151 74HC08, U152 74HC08, U153 74HC08, U154 74HC08, U155 74HC08, U156 74HC08, U157 74HC32, U158 74HC32, U159 74HC32, U160 74HC32, U161 74HC32, U162 74HC32, U163 74HC32, U164 74HC32, U165 74HC32, U166 74HC32, U167 74HC32, U168 74HC32, U169 74HC32, U170 74HC32, U171 74HC32, U172 74HC32

Commit message: Hesap makinesi: eksi işareti sonucun solunda, lamba testinde de yanar; HATA LED'i göstergelerin yanında
- işaret hanesi (DS7) sonucun hanelerinden önce yerleşir: 3D kartta ve
  şemada en solda
- ISARET_g = NEG + lamba testi (boş kapı birimleriyle, çip sayısı aynı)
- HATA LED'i Bölme bloğundan "Gösterge: Sonuç" bloğuna
- rehber ve tasarım belgesi güncellendi

Co-Authored-By: Claude Opus 5.5 (1M context) <noreply@anthropic.com>
Claude-Session: https://claude.ai/code/session_018J8WVuECVRbQJyCbmF6Nsi
Connections:
- net N1976 is gone; now on net N1975: U115.2 (B2), U115.6 (B1), U148.3 (1Y)
- net N2008 is gone; now on net N2007: U148.6 (2Y), U157.10 (3B)
- net N2041 is gone; now on net N2040: U148.8 (3Y), U158.2 (1B)
- net N2074 is gone; now on net N2073: U148.11 (4Y), U158.10 (3B)
- net N2107 is gone; now on net N2106: U119.2 (B2), U119.6 (B1), U149.3 (1Y)
- net N2139 is gone; now on net N2138: U149.6 (2Y), U159.5 (2B)
- net N2172 is gone; now on net N2171: U149.8 (3Y), U159.13 (4B)
- net N2205 is gone; now on net N2204: U149.11 (4Y), U160.5 (2B)
- net N2238 is gone; now on net N2237: U150.3 (1Y), U160.13 (4B)
- net N2271 is gone; now on net N2270: U150.6 (2Y), U161.5 (2B)
- net N2304 is gone; now on net N2303: U150.8 (3Y), U161.13 (4B)
- net N2337 is gone; now on net N2336: U126.2 (B2), U126.6 (B1), U150.11 (4Y)
- net N2369 is gone; now on net N2368: U151.3 (1Y), U162.10 (3B)
- net N2402 is gone; now on net N2401: U151.6 (2Y), U163.2 (1B)
- net N2435 is gone; now on net N2434: U151.8 (3Y), U163.10 (3B)
- net N2468 is gone; now on net N2467: U151.11 (4Y), U164.2 (1B)
- net N2501 is gone; now on net N2500: U152.3 (1Y), U164.10 (3B)
- net N2534 is gone; now on net N2533: U152.6 (2Y), U165.2 (1B)
- net N2567 is gone; now on net N2566: U152.8 (3Y), U165.10 (3B)
- net N2600 is gone; now on net N2599: U152.11 (4Y), U166.2 (1B)
- net N2633 is gone; now on net N2632: U153.3 (1Y), U166.10 (3B)
- net N2666 is gone; now on net N2665: U153.6 (2Y), U167.2 (1B)
- net N2699 is gone; now on net N2698: U153.8 (3Y), U167.10 (3B)
- net N2732 is gone; now on net N2731: U153.11 (4Y), U168.2 (1B)
- net N2765 is gone; now on net N2764: U154.3 (1Y), U168.10 (3B)
- net N2798 is gone; now on net N2797: U154.6 (2Y), U169.2 (1B)
- net N2831 is gone; now on net N2830: U154.8 (3Y), U169.10 (3B)
- net N2864 is gone; now on net N2863: U154.11 (4Y), U170.2 (1B)
- net N2897 is gone; now on net N2896: U155.3 (1Y), U170.10 (3B)
- net N2930 is gone; now on net N2929: U155.6 (2Y), U171.2 (1B)
- net N2963 is gone; now on net N2962: U155.8 (3Y), U171.10 (3B)
- net N2996 is gone; now on net N2995: U155.11 (4Y), U172.2 (1B)
- net N3029 is gone; now on net N3028: U156.3 (1Y), U172.10 (3B)
- net N1975: no longer U148.2 (1B), U157.3 (1Y)
- net N2007: no longer U148.5 (2B), U157.6 (2Y)
- net N2040: no longer U148.10 (3B), U157.11 (4Y)
- net N2073: no longer U148.13 (4B), U158.6 (2Y)
- net N2106: no longer U149.2 (1B), U158.11 (4Y)
- net N2138: no longer U149.5 (2B), U159.3 (1Y)
- net N2171: no longer U149.10 (3B), U159.8 (3Y)
- net N2204: no longer U149.13 (4B), U160.3 (1Y)
- net N2237: no longer U150.2 (1B), U160.8 (3Y)
- net N2270: no longer U150.5 (2B), U161.3 (1Y)
- net N2303: no longer U150.10 (3B), U161.8 (3Y)
- net N2336: no longer U150.13 (4B), U162.3 (1Y)
- net N2368: no longer U151.2 (1B), U162.6 (2Y)
- net N2401: no longer U151.5 (2B), U162.11 (4Y)
- net N2434: no longer U151.10 (3B), U163.6 (2Y)
- net N2467: no longer U151.13 (4B), U163.11 (4Y)
- net N2500: no longer U152.2 (1B), U164.6 (2Y)
- net N2533: no longer U152.5 (2B), U164.11 (4Y)
- net N2566: no longer U152.10 (3B), U165.6 (2Y)
- net N2599: no longer U152.13 (4B), U165.11 (4Y)
- net N2632: no longer U153.2 (1B), U166.6 (2Y)
- net N2665: no longer U153.5 (2B), U166.11 (4Y)
- net N2698: no longer U153.10 (3B), U167.6 (2Y)
- net N2731: no longer U153.13 (4B), U167.11 (4Y)
- net N2764: no longer U154.2 (1B), U168.6 (2Y)
- net N2797: no longer U154.5 (2B), U168.11 (4Y)
- net N2830: no longer U154.10 (3B), U169.6 (2Y)
- net N2863: no longer U154.13 (4B), U169.11 (4Y)
- net N2896: no longer U155.2 (1B), U170.6 (2Y)
- net N2929: no longer U155.5 (2B), U170.11 (4Y)
- net N2962: no longer U155.10 (3B), U171.6 (2Y)
- net N2995: no longer U155.13 (4B), U171.11 (4Y)
- net N3028: no longer U156.2 (1B), U172.6 (2Y)
- new net N1974: U148.2 (1B), U157.3 (1Y)
- new net N2006: U148.5 (2B), U157.6 (2Y)
- new net N2039: U148.10 (3B), U157.11 (4Y)
- new net N2072: U148.13 (4B), U158.6 (2Y)
- new net N2105: U149.2 (1B), U158.11 (4Y)
- new net N2137: U149.5 (2B), U159.3 (1Y)
- new net N2170: U149.10 (3B), U159.8 (3Y)
- new net N2203: U149.13 (4B), U160.3 (1Y)
- new net N2236: U150.2 (1B), U160.8 (3Y)
- new net N2269: U150.5 (2B), U161.3 (1Y)
- new net N2302: U150.10 (3B), U161.8 (3Y)
- new net N2335: U150.13 (4B), U162.3 (1Y)
- new net N2367: U151.2 (1B), U162.6 (2Y)
- new net N2400: U151.5 (2B), U162.11 (4Y)
- new net N2433: U151.10 (3B), U163.6 (2Y)
- new net N2466: U151.13 (4B), U163.11 (4Y)
- new net N2499: U152.2 (1B), U164.6 (2Y)
- new net N2532: U152.5 (2B), U164.11 (4Y)
- new net N2565: U152.10 (3B), U165.6 (2Y)
- new net N2598: U152.13 (4B), U165.11 (4Y)
- new net N2631: U153.2 (1B), U166.6 (2Y)
- new net N2664: U153.5 (2B), U166.11 (4Y)
- new net N2697: U153.10 (3B), U167.6 (2Y)
- new net N2730: U153.13 (4B), U167.11 (4Y)
- new net N2763: U154.2 (1B), U168.6 (2Y)
- new net N2796: U154.5 (2B), U168.11 (4Y)
- new net N2829: U154.10 (3B), U169.6 (2Y)
- new net N2862: U154.13 (4B), U169.11 (4Y)
- new net N2895: U155.2 (1B), U170.6 (2Y)
- new net N2928: U155.5 (2B), U170.11 (4Y)
- new net N2961: U155.10 (3B), U171.6 (2Y)
- new net N2994: U155.13 (4B), U171.11 (4Y)
- new net N3027: U156.2 (1B), U172.6 (2Y)
