File: cpu16/kicad/hesap/hesap-anahtarlar.kicad_sch (KiCad schematic)
At the start: 23 parts, among them SW1 SW_DIP_8, SW2 SW_DIP_8, SW3 SW_DIP_2, SW4 SW_PUSH, U1 74HC08, U2 74HC02, U3 74HC04

Commit message: Hesap makinesi: 5 V besleme girişi, en uzun yol analizi, kurulum belgesi metinleri
- CONN_5V parçası; hesap kartı 2 pinli girişten beslenir
- zamanlama: 74HC4511 modeli ve saatsiz devre için en uzun yol
  (anahtar → segment: tipik 887 ns, en kötü 2,05 µs)
- kurulum: "hepsi" yalnız bilgisayarın kartları; hesap kendi adıyla,
  çok sayfalı şema, DIP-16 direnç dizisi ve gösterge notları
- kurulum testleri çok sayfalı şemayı ve bağımsız kartları tanır

Co-Authored-By: Claude Opus 5.5 (1M context) <noreply@anthropic.com>
Claude-Session: https://claude.ai/code/session_018J8WVuECVRbQJyCbmF6Nsi
Parts:
- removed C1: C_100U, Capacitor_THT:CP_Radial_D6.3mm_P2.50mm, symbol cpu16:C_100U
- removed R3: R_330, Resistor_THT:R_Axial_DIN0207_L6.3mm_D2.5mm_P7.62mm_Horizontal, symbol cpu16:R_330
- added D4: LED, LED_THT:LED_D3.0mm, symbol cpu16:LED
- added J1: CONN_5V, Connector_PinHeader_2.54mm:PinHeader_1x02_P2.54mm_Vertical, symbol cpu16:CONN_5V
- added R5: R_330, Resistor_THT:R_Axial_DIN0207_L6.3mm_D2.5mm_P7.62mm_Horizontal, symbol cpu16:R_330
- C1: renamed from C2; value C_100N -> C_100U; footprint Capacitor_THT:C_Disc_D5.0mm_W2.5mm_P5.00mm -> Capacitor_THT:CP_Radial_D6.3mm_P2.50mm; symbol cpu16:C_100N -> cpu16:C_100U; Gorev U1 dekuplaj -> besleme girişi
- C2: renamed from C3; Gorev U2 dekuplaj -> U1 dekuplaj
- C3: renamed from C4; Gorev U3 dekuplaj -> U2 dekuplaj
- C4: renamed from D1; value LED -> C_100N; footprint LED_THT:LED_D3.0mm -> Capacitor_THT:C_Disc_D5.0mm_W2.5mm_P5.00mm; symbol cpu16:LED -> cpu16:C_100N; Gorev ISLEM_TOPLA LED'i -> U3 dekuplaj
- D1: renamed from D2; Gorev ISLEM_CIKAR LED'i -> ISLEM_TOPLA LED'i
- D2: renamed from D3; Gorev ISLEM_CARP LED'i -> ISLEM_CIKAR LED'i
- D3: renamed from D4; Gorev ISLEM_BOL LED'i -> ISLEM_CARP LED'i
- R3: renamed from R4; Gorev ISLEM_CARP LED direnci -> ISLEM_CIKAR LED direnci
- R4: renamed from R5; Gorev ISLEM_BOL LED direnci -> ISLEM_CARP LED direnci
Connections:
- net BOL: now also R5.1; no longer R4.1
- net CARP: now also R4.1; no longer R3.1
- net CIKAR: now also R3.1
- net GND: now also D4.2 (K), J1.2 (GND)
- net LED_ISLEM_BOL: now also D4.1 (A), R5.2; no longer D3.1 (A), R4.2
- net LED_ISLEM_CARP: now also D3.1 (A), R4.2; no longer D2.1 (A), R3.2
- net LED_ISLEM_CIKAR: now also D2.1 (A), R3.2; no longer D1.1 (A)
- net LED_ISLEM_TOPLA: now also D1.1 (A); no longer C4.1 (A)
- net VCC: now also C4.1, J1.1 (+5V)
