File: cpu16/kicad/hesap/hesap-gosterge-sonuc.kicad_sch (KiCad schematic)
At the start: 54 parts, among them U199 74HC08, U200 74HC32, U201 74HC32, U202 74HC02, U203 74HC02, U204 74HC04, U205 74HC4511, U206 74HC4511, U207 74HC4511, U208 74HC4511, U209 74HC4511, U210 74HC08, U211 74HC32, U212 74HC02, U213 74HC04, U214 74HC4511, U215 74HC4511, U216 74HC4511

Commit message: Hesap makinesi: eksi işareti sonucun solunda, lamba testinde de yanar; HATA LED'i göstergelerin yanında
- işaret hanesi (DS7) sonucun hanelerinden önce yerleşir: 3D kartta ve
  şemada en solda
- ISARET_g = NEG + lamba testi (boş kapı birimleriyle, çip sayısı aynı)
- HATA LED'i Bölme bloğundan "Gösterge: Sonuç" bloğuna
- rehber ve tasarım belgesi güncellendi

Co-Authored-By: Claude Opus 5.5 (1M context) <noreply@anthropic.com>
Claude-Session: https://claude.ai/code/session_018J8WVuECVRbQJyCbmF6Nsi
Parts:
- added D5: LED, LED_THT:LED_D3.0mm, symbol cpu16:LED
- added R6: R_330, Resistor_THT:R_Axial_DIN0207_L6.3mm_D2.5mm_P7.62mm_Horizontal, symbol cpu16:R_330
- DS10: Gorev Sonuç: 1. hane -> Sonuç: 2. hane
- DS11: Gorev Sonuç: 0. hane -> Sonuç: 1. hane
- DS12: Gorev Sonuç: eksi işareti (yalnız g segmenti) -> Sonuç: 0. hane
- DS7: Gorev Sonuç: 4. hane -> Sonuç: eksi işareti (yalnız g segmenti)
- DS8: Gorev Sonuç: 3. hane -> Sonuç: 4. hane
- DS9: Gorev Sonuç: 2. hane -> Sonuç: 3. hane
- R7: Gorev Sonuç: eksi işareti direnci -> HATA LED direnci
- U201: Gorev Sonuç: baştaki sıfırları söndürme -> Sonuç: baştaki sıfırları söndürme: eksi işareti ya da lamba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
- U204: Gorev Sonuç: baştaki sıfırları söndürme: Sonuç: grup sönük -> Sonuç: baştaki sıfırları söndürme: Sonuç: grup sönük, lamba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
Connections:
- net N3634 is gone; now on net N3633: U199.8 (3Y), U203.2 (1A)
- net N3892 is gone; now on net N3891: U210.3 (1Y), U212.8 (3A)
- net GND: now also D5.2 (K); no longer U201.12 (4A), U201.13 (4B), U204.3 (2A)
- net HATA: now also R7.1
- net ISARET_g_LED: now also DS7.10 (g), R6.2; no longer DS12.10 (g), R7.2
- net LT_N: now also U204.3 (2A)
- net N3621: now also U200.6 (2Y), U202.3 (1B); no longer U200.3 (1Y), U202.2 (1A)
- net N3622: now also U199.10 (3B), U202.1 (1Y); no longer U200.6 (2Y), U202.3 (1B)
- net N3623: now also U200.8 (3Y), U202.5 (2A); no longer U199.10 (3B), U202.1 (1Y)
- net N3624: now also U200.11 (4Y), U202.6 (2B); no longer U200.8 (3Y), U202.5 (2A)
- net N3625: now also U199.5 (2B), U202.4 (2Y); no longer U200.11 (4Y), U202.6 (2B)
- net N3626: now also U201.3 (1Y), U202.8 (3A); no longer U199.5 (2B), U202.4 (2Y)
- net N3627: now also U201.6 (2Y), U202.9 (3B); no longer U201.3 (1Y), U202.8 (3A)
- net N3628: now also U199.2 (1B), U202.10 (3Y); no longer U201.6 (2Y), U202.9 (3B)
- net N3629: now also U201.8 (3Y), U202.11 (4A); no longer U199.2 (1B), U202.10 (3Y)
- net N3630: now also U199.1 (1A), U202.13 (4Y), U203.11 (4A); no longer U201.8 (3Y), U202.11 (4A)
- net N3631: now also U199.3 (1Y), U199.4 (2A), U203.8 (3A); no longer U199.1 (1A), U202.13 (4Y), U203.11 (4A)
- net N3632: now also U199.6 (2Y), U199.9 (3A), U203.5 (2A); no longer U199.3 (1Y), U199.4 (2A), U203.8 (3A)
- net N3633: no longer U199.6 (2Y), U199.9 (3A), U203.5 (2A)
- net N3888: now also U211.6 (2Y), U212.3 (1B); no longer U211.3 (1Y), U212.2 (1A)
- net N3889: now also U210.2 (1B), U212.1 (1Y); no longer U211.6 (2Y), U212.3 (1B)
- net N3890: now also U210.1 (1A), U212.11 (4A), U212.4 (2Y); no longer U210.2 (1B), U212.1 (1Y)
- net N3891: no longer U210.1 (1A), U212.11 (4A), U212.4 (2Y)
- net NEG: now also U201.12 (4A); no longer R7.1
- net SONUC0_a_LED: now also DS12.7 (a); no longer DS11.7 (a)
- net SONUC0_b_LED: now also DS12.6 (b); no longer DS11.6 (b)
- net SONUC0_c_LED: now also DS12.4 (c); no longer DS11.4 (c)
- net SONUC0_d_LED: now also DS12.2 (d); no longer DS11.2 (d)
- net SONUC0_e_LED: now also DS12.1 (e); no longer DS11.1 (e)
- net SONUC0_f_LED: now also DS12.9 (f); no longer DS11.9 (f)
- net SONUC0_g_LED: now also DS12.10 (g); no longer DS11.10 (g)
- net SONUC1_a_LED: now also DS11.7 (a); no longer DS10.7 (a)
- net SONUC1_b_LED: now also DS11.6 (b); no longer DS10.6 (b)
- net SONUC1_c_LED: now also DS11.4 (c); no longer DS10.4 (c)
- net SONUC1_d_LED: now also DS11.2 (d); no longer DS10.2 (d)
- net SONUC1_e_LED: now also DS11.1 (e); no longer DS10.1 (e)
- net SONUC1_f_LED: now also DS11.9 (f); no longer DS10.9 (f)
- net SONUC1_g_LED: now also DS11.10 (g); no longer DS10.10 (g)
- net SONUC2_a_LED: now also DS10.7 (a); no longer DS9.7 (a)
- net SONUC2_b_LED: now also DS10.6 (b); no longer DS9.6 (b)
- net SONUC2_c_LED: now also DS10.4 (c); no longer DS9.4 (c)
- net SONUC2_d_LED: now also DS10.2 (d); no longer DS9.2 (d)
- net SONUC2_e_LED: now also DS10.1 (e); no longer DS9.1 (e)
- net SONUC2_f_LED: now also DS10.9 (f); no longer DS9.9 (f)
- net SONUC2_g_LED: now also DS10.10 (g); no longer DS9.10 (g)
- net SONUC3_a_LED: now also DS9.7 (a); no longer DS8.7 (a)
- net SONUC3_b_LED: now also DS9.6 (b); no longer DS8.6 (b)
- net SONUC3_c_LED: now also DS9.4 (c); no longer DS8.4 (c)
- net SONUC3_d_LED: now also DS9.2 (d); no longer DS8.2 (d)
- net SONUC3_e_LED: now also DS9.1 (e); no longer DS8.1 (e)
- net SONUC3_f_LED: now also DS9.9 (f); no longer DS8.9 (f)
- net SONUC3_g_LED: now also DS9.10 (g); no longer DS8.10 (g)
- net SONUC4_a_LED: now also DS8.7 (a); no longer DS7.7 (a)
- net SONUC4_b_LED: now also DS8.6 (b); no longer DS7.6 (b)
- net SONUC4_c_LED: now also DS8.4 (c); no longer DS7.4 (c)
- net SONUC4_d_LED: now also DS8.2 (d); no longer DS7.2 (d)
- net SONUC4_e_LED: now also DS8.1 (e); no longer DS7.1 (e)
- net SONUC4_f_LED: now also DS8.9 (f); no longer DS7.9 (f)
- net SONUC4_g_LED: now also DS8.10 (g); no longer DS7.10 (g)
- net N3639: now reaches U204.4 (2Y)
- net N3639: now also U201.13 (4B)
- net ISARET_g: now reaches U201.11 (4Y)
- net ISARET_g: now also R6.1
- new net LED_HATA: D5.1 (A), R7.2
- new net N3620: U200.3 (1Y), U202.2 (1A)
- new net N3887: U211.3 (1Y), U212.2 (1A)
- no-connect marks 48 -> 46
